File: td-deflect/power_supply.sch (KiCad schematic (older format))
At the start: 19 parts

Commit message: add lots of stuff
Parts:
- removed R?: 1M, symbol Device:R
- removed R?: 37.4k, symbol Device:R
- added C19, C30, C43: 0.1uF, Capacitor_SMD:C_0805_2012Metric_Pad1.15x1.40mm_HandSolder, symbol Device:C
- added C24: 0.0073uF, Capacitor_SMD:C_1210_3225Metric_Pad1.42x2.65mm_HandSolder, symbol Device:C
- added C27: 22uF, Capacitor_SMD:C_0805_2012Metric_Pad1.15x1.40mm_HandSolder, symbol Device:C
- added C28: 22uF, symbol Device:C
- added C29, C33: 2.2uF, Capacitor_SMD:C_0805_2012Metric_Pad1.15x1.40mm_HandSolder, symbol Device:C
- added C31: 0.01uF, Capacitor_SMD:C_0805_2012Metric_Pad1.15x1.40mm_HandSolder, symbol Device:C
- added C32: 100uF, symbol Device:C
- added C34: 10uF, Capacitor_SMD:C_0805_2012Metric_Pad1.15x1.40mm_HandSolder, symbol Device:C
- added C44: 0.033uF, Capacitor_SMD:C_0805_2012Metric_Pad1.15x1.40mm_HandSolder, symbol Device:C
- added C45: 22pF, Capacitor_SMD:C_0805_2012Metric_Pad1.15x1.40mm_HandSolder, symbol Device:C
- added C46: 47uF, symbol Device:C
- added D4: C3D10170H, Package_TO_SOT_THT:TO-247-2_Vertical, symbol Diode:C3D10170H
- added D5: B220, Diode_SMD:D_SMB, symbol Diode:B220
- added E2: SPARK_GAP, Capacitor_SMD:C_1825_4564Metric_Pad1.88x6.70mm_HandSolder, symbol Device:SPARK_GAP
- added J13, J14, J2, J8, J9: Conn_01x02_Male, Connector_Phoenix_MSTB:PhoenixContact_MSTBVA_2,5_2-G_1x02_P5.00mm_Vertical, symbol Connector:Conn_01x02_Male
- added L4: 7.8uH, symbol Device:L
- added L5: 100uH, symbol Device:L
- added Q12: C2M0045170D, Package_TO_SOT_THT:TO-247-3_Vertical, symbol Transistor_FET:C2M0045170D
- added R29: 1M, Resistor_SMD:R_0805_2012Metric_Pad1.15x1.40mm_HandSolder, symbol Device:R
- added R30: 37.4k, Resistor_SMD:R_0805_2012Metric_Pad1.15x1.40mm_HandSolder, symbol Device:R
- added R33, R34, R43: 10k, Resistor_SMD:R_0805_2012Metric_Pad1.15x1.40mm_HandSolder, symbol Device:R
- added R35: 1, Resistor_SMD:R_0805_2012Metric_Pad1.15x1.40mm_HandSolder, symbol Device:R
- added R36: 0.01, Resistor_SMD:R_0603_1608Metric_Pad1.05x0.95mm_HandSolder, symbol Device:R
- added R38: 1M, Resistor_THT:R_Axial_DIN0309_L9.0mm_D3.2mm_P15.24mm_Horizontal, symbol Device:R
- added R41, R45: 100k, Resistor_SMD:R_0805_2012Metric_Pad1.15x1.40mm_HandSolder, symbol Device:R
- added R42: 1k, Resistor_SMD:R_0805_2012Metric_Pad1.15x1.40mm_HandSolder, symbol Device:R
- added R44: 39k, Resistor_SMD:R_0805_2012Metric_Pad1.15x1.40mm_HandSolder, symbol Device:R
- added R46: 240k, Resistor_SMD:R_0805_2012Metric_Pad1.15x1.40mm_HandSolder, symbol Device:R
- added R47: 249k, Resistor_SMD:R_0805_2012Metric_Pad1.15x1.40mm_HandSolder, symbol Device:R
- added R48: 15.4k, Resistor_SMD:R_0805_2012Metric_Pad1.15x1.40mm_HandSolder, symbol Device:R
- added R49: 147k, Resistor_SMD:R_0805_2012Metric_Pad1.15x1.40mm_HandSolder, symbol Device:R
- added R50: 10.5k, Resistor_SMD:R_0805_2012Metric_Pad1.15x1.40mm_HandSolder, symbol Device:R
- added U13: MCP1416, Package_TO_SOT_SMD:SOT-23-5, symbol Driver_FET:MCP1416
- added U15: LM1117-ADJ, Package_TO_SOT_SMD:TO-252-2, symbol Regulator_Linear:LM1117-ADJ
- added U16: LTC7149FE, Package_SO:HTSSOP-28-1EP_4.4x9.7mm_P0.65mm_EP2.85x5.4mm, symbol td-deflect:LTC7149FE
- added U17: TPS54360DDA, Package_SO:TI_SO-PowerPAD-8_ThermalVias, symbol Regulator_Switching:TPS54360DDA
- C18: renamed from C?; footprint (none) -> Capacitor_SMD:C_1210_3225Metric_Pad1.42x2.65mm_HandSolder; Voltage (none) -> 100V
- C20, C21, C23: renamed from C?; footprint (none) -> Capacitor_SMD:C_0805_2012Metric_Pad1.15x1.40mm_HandSolder; Voltage (none) -> 10V
- C22, C25, C26: renamed from C?; footprint (none) -> Capacitor_SMD:C_1210_3225Metric_Pad1.42x2.65mm_HandSolder; Voltage (none) -> 200V
- R31, R32, R37, R40: renamed from R?; footprint (none) -> Resistor_SMD:R_0805_2012Metric_Pad1.15x1.40mm_HandSolder
- R39: renamed from R?; footprint (none) -> Resistor_SMD:R_1206_3216Metric_Pad1.42x1.75mm_HandSolder
- RV1: renamed from RV?; footprint (none) -> Potentiometer_THT:Potentiometer_Bourns_3339P_Vertical_HandSoldering
- gave numbers to parts that had none: 4
Connections:
- net +48V: now also C28.1, C34.1, R29.1, U16.6 (Vin), U16.7 (Vin), U16.8 (RUN), U17.2 (VIN)
- net GND: now also C19.2, C24.2, C27.2, C29.2, C32.1, C33.2, C34.2, C44.2, C45.2, C46.2, D4.2 (A), D5.2 (A), E2.2, J13.1 (Pin_1), J14.1 (Pin_1), J2.2 (Pin_2), J9.1 (Pin_1), L4.2, R30.2, R33.2, R34.2, R36.2, R38.2, R42.2, R44.2, R47.2, R50.2, U13.4 (GND), U16.10 (MODE/SYNC), U16.16 (Voutsns), U16.19 (EXTVcc), U16.9 (GND), U17.7 (GND), U17.9 (GNDPAD)
- net HT: now also J2.1 (Pin_1), J8.1 (Pin_1)
- net at U14.9 (~SHDN~/UVLO): now also R29.2, R30.1
- new net: R43.2, R44.1, U15.1 (ADJ)
- new net: C27.1, J9.2 (Pin_2), R43.1, U15.2 (VO)
- new net: R34.1, R35.2, U13.5 (OUT)
- new net: Q12.1 (G), R35.1
- new net: C29.1, C33.1, U16.14 (Vinreg), U16.18 (ITH), U16.20 (INTVcc)
- new net: R45.1, U16.15 (Rt)
- new net: C31.1, R46.1, U16.17 (ISET)
- new net: C30.2, U16.21 (BOOST)
- new net: C30.1, L4.1, U16.22 (SW), U16.23 (SW), U16.24 (SW), U16.25 (SW), U16.26 (SW), U16.27 (SW), U16.28 (SW)
- new net: C43.1, U17.1 (BOOT)
- new net: R47.1, U17.4 (RT/CLK)
- new net: R49.2, R50.1, U17.5 (FB)
- new net: C45.1, R48.1, U17.6 (COMP)
- new net: C43.2, D5.1 (K), L5.1, U17.8 (SW)
- new net: C44.1, R48.2
- new net +12V: C19.1, C46.1, J14.2 (Pin_2), L5.2, R49.1, U13.2 (Vdd), U15.3 (VI)
- new net -12V: C31.2, C32.2, J13.2 (Pin_2), R45.2, R46.2, U16.1 (Vout-), U16.13 (SVout-), U16.2 (Vout-), U16.29 (SVout-), U16.3 (Vout-), U16.4 (Vout-), U16.5 (Vout-)
- new net EHT_CURRENT: Q12.3 (S), R36.1
- new net EHT_FLYBACK_VOLTAGE: R41.2, R42.1
- new net EHT_PWM: R33.1, U13.3 (IN)
- new net eht out: C24.1, D4.1 (K), E2.1, J8.2 (Pin_2), Q12.2 (D), R38.1, R41.1
Other:
- note added: "HEATER"
- moved on the sheet: C18, C20, C21, C22, C23, C25, C26, D3, L3, Q13, R30, R31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

Commit message: more stuff
Parts:
- C28: footprint (none) -> Capacitor_THT:CP_Radial_D8.0mm_P3.50mm; Digikey (none) -> 493-3872-1-ND
- C32: footprint (none) -> Capacitor_THT:CP_Radial_D8.0mm_P3.50mm; Digikey (none) -> 493-3716-ND; Voltage (none) -> 16V
- C46: value 47uF -> 100uF; footprint (none) -> Capacitor_THT:CP_Radial_D8.0mm_P3.50mm; Digikey (none) -> 493-3716-ND; Voltage (none) -> 16V
- L3: footprint (none) -> Inductor_SMD:L_Bourns_SRR1260; Digikey (none) -> SRR1260-330MCT-ND
- L4: footprint (none) -> Inductor_SMD:L_Bourns_SRR1260; Digikey (none) -> SRR1260-7R6YCT-ND
- L5: footprint (none) -> Inductor_SMD:L_Bourns_SRR1260; Digikey (none) -> SRR1260-101MCT-ND
Connections:
- net GND: now also C28.2
Changed lines of the file:
@@
 F 0 "L3" V 3840 1150 50  0000 C CNN
 F 1 "33uH" V 3749 1150 50  0000 C CNN
-F 2 "" H 3650 1150 50  0001 C CNN
+F 2 "Inductor_SMD:L_Bourns_SRR1260" H 3650 1150 50  0001 C CNN
 F 3 "~" H 3650 1150 50  0001 C CNN
+F 4 " SRR1260-330MCT-ND " V 3650 1150 50  0001 C CNN "Digikey"
 	1    3650 1150
 	0    -1   -1   0
@@
 F 0 "L4" V 4690 3450 50  0000 C CNN
 F 1 "7.8uH" V 4599 3450 50  0000 C CNN
-F 2 "" H 4500 3450 50  0001 C CNN
+F 2 "Inductor_SMD:L_Bourns_SRR1260" H 4500 3450 50  0001 C CNN
 F 3 "~" H 4500 3450 50  0001 C CNN
+F 4 " SRR1260-7R6YCT-ND " V 4500 3450 50  0001 C CNN "Digikey"
 	1    4500 3450
 	0    -1   -1   0
@@
 F 0 "C32" H 5015 3646 50  0000 L CNN
 F 1 "100uF" H 5015 3555 50  0000 L CNN
-F 2 "" H 4938 3450 50  0001 C CNN
+F 2 "Capacitor_THT:CP_Radial_D8.0mm_P3.50mm" H 4938 3450 50  0001 C CNN
 F 3 "~" H 4900 3600 50  0001 C CNN
+F 4 " 493-3716-ND " H 4900 3600 50  0001 C CNN "Digikey"
+F 5 "16V" H 4900 3600 50  0001 C CNN "Voltage"
 	1    4900 3600
 	1    0    0    -1
@@
 $EndComp
 Wire Wire Line
-	2750 4250 2250 4250
+	2750 4250 2350 4250
 Wire Wire Line
 	2750 4350 2750 4250
@@
 F 0 "C28" H 2465 4146 50  0000 L CNN
 F 1 "22uF" H 2465 4055 50  0000 L CNN
-F 2 "" H 2388 3950 50  0001 C CNN
+F 2 "Capacitor_THT:CP_Radial_D8.0mm_P3.50mm" H 2388 3950 50  0001 C CNN
 F 3 "~" H 2350 4100 50  0001 C CNN
 F 4 "100V" H 2350 4100 50  0001 C CNN "Voltage"
+F 5 " 493-3872-1-ND " H 2350 4100 50  0001 C CNN "Digikey"
 	1    2350 4100
 	1    0    0    -1
@@
 P 9600 2950
 F 0 "C46" H 9715 2996 50  0000 L CNN
-F 1 "47uF" H 9715 2905 50  0000 L CNN
-F 2 "" H 9638 2800 50  0001 C CNN
+F 1 "100uF" H 9715 2905 50  0000 L CNN
+F 2 "Capacitor_THT:CP_Radial_D8.0mm_P3.50mm" H 9638 2800 50  0001 C CNN
 F 3 "~" H 9600 2950 50  0001 C CNN
+F 4 "16V" H 9600 2950 50  0001 C CNN "Voltage"
+F 5 " 493-3716-ND " H 9600 2950 50  0001 C CNN "Digikey"
 	1    9600 2950
 	1    0    0    -1
@@
 F 0 "L5" V 9040 2800 50  0000 C CNN
 F 1 "100uH" V 8949 2800 50  0000 C CNN
-F 2 "" H 8850 2800 50  0001 C CNN
+F 2 "Inductor_SMD:L_Bourns_SRR1260" H 8850 2800 50  0001 C CNN
 F 3 "~" H 8850 2800 50  0001 C CNN
+F 4 " SRR1260-101MCT-ND " H 8850 2800 50  0001 C CNN "Digikey"
 	1    8850 2800
 	0    -1   -1   0
@@
 Wire Wire Line
 	9850 2800 10100 2800
+Connection ~ 2350 3950
+Connection ~ 2350 4250
+Wire Wire Line
+	2350 4250 2250 4250
 $EndSCHEMATC

Commit message: asdf
Parts:
- added C61: 0.033uF, Capacitor_SMD:C_1206_3216Metric_Pad1.42x1.75mm_HandSolder, symbol Device:C
- added J15: Conn_01x02_Male, td-deflect:sony_monitor_2p, symbol Connector:Conn_01x02_Male
- added J18: Conn_01x02_Male, Connector_Phoenix_MSTB:PhoenixContact_MSTBVA_2,5_2-G_1x02_P5.00mm_Vertical, symbol Connector:Conn_01x02_Male
- added L6: 1mH, Inductor_THT:L_Toroid_Vertical_L31.8mm_W15.9mm_P13.50mm_Bourns_5700, symbol Device:L
- added R97: 1, Resistor_SMD:R_0805_2012Metric_Pad1.15x1.40mm_HandSolder, symbol Device:R
- C19, C30, C43: Digikey (none) -> 1276-1099-1-ND
- C20: value 10nF -> 0.01uF; Digikey (none) -> 1276-2434-1-ND
- C21: Digikey (none) -> 1276-2569-1-ND
- C22: footprint Capacitor_SMD:C_1210_3225Metric_Pad1.42x2.65mm_HandSolder -> Capacitor_SMD:C_1206_3216Metric_Pad1.42x1.75mm_HandSolder; Digikey (none) -> 1276-6641-1-ND; Voltage 200V -> 10V
- C23: Digikey (none) -> 1276-3177-1-ND
- C24: footprint Capacitor_SMD:C_1210_3225Metric_Pad1.42x2.65mm_HandSolder -> Capacitor_THT:C_Rect_L18.0mm_W6.0mm_P15.00mm_FKS3_FKP3; Digikey 495-3231-ND -> 495-3231-ND
- C25: footprint Capacitor_SMD:C_1210_3225Metric_Pad1.42x2.65mm_HandSolder -> Capacitor_THT:CP_Radial_D8.0mm_P3.50mm; symbol Device:C -> Device:CP; Digikey (none) -> UVK2D100MPD-ND
- C26: value 4.7uF -> 0.1uF; footprint Capacitor_SMD:C_1210_3225Metric_Pad1.42x2.65mm_HandSolder -> Capacitor_SMD:C_1206_3216Metric_Pad1.42x1.75mm_HandSolder; Digikey (none) -> 1276-3084-1-ND
- C27: footprint Capacitor_SMD:C_0805_2012Metric_Pad1.15x1.40mm_HandSolder -> Capacitor_SMD:C_1206_3216Metric_Pad1.42x1.75mm_HandSolder; Digikey (none) -> 1276-2769-1-ND
- C28: symbol Device:C -> Device:CP; Digikey 493-3872-1-ND -> 493-3872-1-ND
- C29, C33: Digikey (none) -> 1276-2953-1-ND
- C31: Digikey (none) -> 1276-2434-1-ND; Voltage (none) -> 10V
- C32, C46: symbol Device:C -> Device:CP; Digikey 493-3716-ND -> 493-3716-ND
- C34: footprint Capacitor_SMD:C_0805_2012Metric_Pad1.15x1.40mm_HandSolder -> Capacitor_THT:CP_Radial_D8.0mm_P3.50mm; symbol Device:C -> Device:CP; Digikey (none) -> 493-4578-1-ND; Voltage (none) -> 100V
- C44: Digikey (none) -> 1276-1796-1-ND; Voltage (none) -> 10V
- C45: Digikey (none) -> 1276-2605-1-ND
- D3: Digikey (none) -> 1N5402GOS-ND
- D4: Digikey (none) -> C3D10170H-ND
- D5: Digikey (none) -> B220A-FDICT-ND
- E2: footprint Capacitor_SMD:C_1825_4564Metric_Pad1.88x6.70mm_HandSolder -> Resistor_THT:R_Axial_DIN0309_L9.0mm_D3.2mm_P12.70mm_Horizontal; Digikey F7596TR-ND -> F3681-ND
- J13, J14, J2, J8, J9: Digikey (none) -> 277-1150-ND
- Q12: Digikey (none) -> C2M0045170D-ND
- Q13: Digikey (none) -> BSC082N10LSGATMA1CT-ND
- R32: value 50k -> 49.9k
- R36: footprint Resistor_SMD:R_0603_1608Metric_Pad1.05x0.95mm_HandSolder -> Resistor_SMD:R_0805_2012Metric_Pad1.15x1.40mm_HandSolder
- R41: value 100k -> 1M; footprint Resistor_SMD:R_0805_2012Metric_Pad1.15x1.40mm_HandSolder -> Resistor_THT:R_Axial_DIN0309_L9.0mm_D3.2mm_P15.24mm_Horizontal
Connections:
- net +48V: now also J18.2 (Pin_2)
- net GND: now also J2.1 (Pin_1), C61.2, J15.1 (Pin_1), J18.1 (Pin_1); no longer J2.2 (Pin_2)
- net HT: now also J2.2 (Pin_2), L6.1; no longer J2.1 (Pin_1), J8.1 (Pin_1)
- net eht out: now also L6.2
- net at J9.2 (Pin_2), R43.1, U15.2 (VO): now also J15.2 (Pin_2), R97.1; no longer C27.1
- new net: C27.1, R97.2
- new net: C61.1, J8.1 (Pin_1)
- no-connect marks 0 -> 3
Other:
- moved on the sheet: C24, C27, D4, E2, J2, J8, R38, R41, R42

Commit message: asdf
Parts:
- C18: value 4.7uF -> 22uF; footprint Capacitor_SMD:C_1210_3225Metric_Pad1.42x2.65mm_HandSolder -> Capacitor_THT:CP_Radial_D8.0mm_P3.50mm; Digikey (none) -> 493-3872-1-ND; Voltage 100V -> 63V
- R29: Digikey (none) -> 311-1.00MCRCT-ND
- R30: Digikey (none) -> 311-37.4KCRCT-ND
- R31, R32: Digikey (none) -> 311-49.9KCRCT-ND
- R33, R34, R35, R43, R97: Digikey (none) -> 311-1.00CRCT-ND
- R36, R37: Digikey (none) -> 311-0.01NUCT-ND
- R38, R41: Digikey (none) -> BC4422CT-ND
- R39: Digikey (none) -> 311-68.0KFRCT-ND
- R40: Digikey (none) -> 311-470CRCT-ND
- R42: Digikey (none) -> 311-1.00KCRCT-ND
- R44: Digikey (none) -> 311-39.0KCRCT-ND
- R45: Digikey (none) -> 311-100KCRCT-ND
- R46: Digikey (none) -> 311-240KCRCT-ND
- R47: Digikey (none) -> 311-249KCRCT-ND
- R48: Digikey (none) -> 311-15.4KCRCT-ND
- R49: Digikey (none) -> 311-147KCRCT-ND
- R50: Digikey (none) -> 311-10.5KCRCT-ND
- RV1: footprint Potentiometer_THT:Potentiometer_Bourns_3339P_Vertical_HandSoldering -> Potentiometer_THT:Potentiometer_Bourns_3386P_Vertical; Digikey (none) -> 3386P-102LF-ND
- U13: Digikey (none) -> MCP1416T-E/OTCT-ND
- U14: Digikey (none) -> LT3758AEMSE#TRPBFCT-ND
- U15: Digikey (none) -> LM1117IDTX-ADJ/NOPBCT-ND
- U16: Digikey (none) -> LTC7149IFE#PBF-ND
- U17: Digikey (none) -> 296-37676-1-ND
Changed lines of the file:
@@
 F 2 "Resistor_SMD:R_0805_2012Metric_Pad1.15x1.40mm_HandSolder" V 1430 1350 50  0001 C CNN
 F 3 "~" H 1500 1350 50  0001 C CNN
+F 4 " 311-1.00MCRCT-ND" H 1500 1350 50  0001 C CNN "Digikey"
 	1    1500 1350
 	1    0    0    -1
@@
 F 2 "Resistor_SMD:R_0805_2012Metric_Pad1.15x1.40mm_HandSolder" V 1430 1700 50  0001 C CNN
 F 3 "~" H 1500 1700 50  0001 C CNN
+F 4 " 	311-37.4KCRCT-ND " H 1500 1700 50  0001 C CNN "Digikey"
 	1    1500 1700
 	1    0    0    -1
@@
 F 2 "Package_SO:MSOP-10-1EP_3x3mm_P0.5mm_EP1.68x1.88mm" H 3100 1100 50  0001 L CNN
 F 3 "https://www.analog.com/media/en/technical-documentation/data-sheets/3757Afe.pdf" H 3050 1650 50  0001 C CNN
+F 4 "LT3758AEMSE#TRPBFCT-ND" H 3050 1650 50  0001 C CNN "Digikey"
 	1    3050 1650
 	1    0    0    -1
@@
 F 2 "Resistor_SMD:R_0805_2012Metric_Pad1.15x1.40mm_HandSolder" V 1930 2050 50  0001 C CNN
 F 3 "~" H 2000 2050 50  0001 C CNN
+F 4 " 311-49.9KCRCT-ND" H 2000 2050 50  0001 C CNN "Digikey"
 	1    2000 2050
 	0    1    1    0
@@
 F 2 "Resistor_SMD:R_0805_2012Metric_Pad1.15x1.40mm_HandSolder" V 1580 2200 50  0001 C CNN
 F 3 "~" H 1650 2200 50  0001 C CNN
+F 4 " 311-49.9KCRCT-ND" H 1650 2200 50  0001 C CNN "Digikey"
 	1    1650 2200
 	1    0    0    -1
@@
 F 2 "Resistor_SMD:R_0805_2012Metric_Pad1.15x1.40mm_HandSolder" V 4030 2150 50  0001 C CNN
 F 3 "~" H 4100 2150 50  0001 C CNN
+F 4 "311-0.01NUCT-ND" H 4100 2150 50  0001 C CNN "Digikey"
 	1    4100 2150
 	1    0    0    -1
@@
 F 2 "Resistor_SMD:R_1206_3216Metric_Pad1.42x1.75mm_HandSolder" V 4830 1300 50  0001 C CNN
 F 3 "~" H 4900 1300 50  0001 C CNN
+F 4 " 311-68.0KFRCT-ND" H 4900 1300 50  0001 C CNN "Digikey"
 	1    4900 1300
 	1    0    0    -1
@@
 F 2 "Resistor_SMD:R_0805_2012Metric_Pad1.15x1.40mm_HandSolder" V 4830 2050 50  0001 C CNN
 F 3 "~" H 4900 2050 50  0001 C CNN
+F 4 " 311-470CRCT-ND" H 4900 2050 50  0001 C CNN "Digikey"
 	1    4900 2050
 	1    0    0    -1
@@
 P 1000 1650
 F 0 "C18" H 1115 1696 50  0000 L CNN
-F 1 "4.7uF" H 1115 1605 50  0000 L CNN
-F 2 "Capacitor_SMD:C_1210_3225Metric_Pad1.42x2.65mm_HandSolder" H 1038 1500 50  0001 C CNN
+F 1 "22uF" H 1115 1605 50  0000 L CNN
+F 2 "Capacitor_THT:CP_Radial_D8.0mm_P3.50mm" H 1038 1500 50  0001 C CNN
 F 3 "~" H 1000 1650 50  0001 C CNN
-F 4 "100V" H 1000 1650 50  0001 C CNN "Voltage"
+F 4 "63V" H 1000 1650 50  0001 C CNN "Voltage"
+F 5 "493-3872-1-ND " H 1000 1650 50  0001 C CNN "Digikey"
 	1    1000 1650
 	1    0    0    -1
@@
 F 0 "RV1" H 4830 1704 50  0000 R CNN
 F 1 "1k" H 4830 1795 50  0000 R CNN
-F 2 "Potentiometer_THT:Potentiometer_Bourns_3339P_Vertical_HandSoldering" H 4900 1750 50  0001 C CNN
+F 2 "Potentiometer_THT:Potentiometer_Bourns_3386P_Vertical" H 4900 1750 50  0001 C CNN
 F 3 "~" H 4900 1750 50  0001 C CNN
+F 4 "3386P-102LF-ND" H 4900 1750 50  0001 C CNN "Digikey"
 	1    4900 1750
 	-1   0    0    1
@@
 F 2 "Package_TO_SOT_SMD:TO-252-2" H 8950 5350 50  0001 C CNN
 F 3 "http://www.ti.com/lit/ds/symlink/lm1117.pdf" H 8950 5350 50  0001 C CNN
+F 4 "LM1117IDTX-ADJ/NOPBCT-ND " H 8950 5350 50  0001 C CNN "Digikey"
 	1    8950 5350
 	1    0    0    -1
@@
 F 2 "Resistor_SMD:R_0805_2012Metric_Pad1.15x1.40mm_HandSolder" V 9330 5500 50  0001 C CNN
 F 3 "~" H 9400 5500 50  0001 C CNN
+F 4 "311-1.00CRCT-ND" H 9400 5500 50  0001 C CNN "Digikey"
 	1    9400 5500
 	1    0    0    -1
@@
 F 2 "Resistor_SMD:R_0805_2012Metric_Pad1.15x1.40mm_HandSolder" V 9330 5850 50  0001 C CNN
 F 3 "~" H 9400 5850 50  0001 C CNN
+F 4 " 311-39.0KCRCT-ND" H 9400 5850 50  0001 C CNN "Digikey"
 	1    9400 5850
 	1    0    0    -1
@@
 F 2 "Resistor_SMD:R_0805_2012Metric_Pad1.15x1.40mm_HandSolder" V 3630 6750 50  0001 C CNN
 F 3 "~" H 3700 6750 50  0001 C CNN
+F 4 "311-0.01NUCT-ND" H 3700 6750 50  0001 C CNN "Digikey"
 	1    3700 6750
 	1    0    0    -1
@@
 F 2 "Resistor_SMD:R_0805_2012Metric_Pad1.15x1.40mm_HandSolder" V 1930 6550 50  0001 C CNN
 F 3 "~" H 2000 6550 50  0001 C CNN
+F 4 "311-1.00CRCT-ND" H 2000 6550 50  0001 C CNN "Digikey"
 	1    2000 6550
 	1    0    0    -1
@@
 F 2 "Resistor_SMD:R_0805_2012Metric_Pad1.15x1.40mm_HandSolder" V 2730 6550 50  0001 C CNN
 F 3 "~" H 2800 6550 50  0001 C CNN
+F 4 "311-1.00CRCT-ND" H 2800 6550 50  0001 C CNN "Digikey"
 	1    2800 6550
 	1    0    0    -1
@@
 F 2 "Resistor_SMD:R_0805_2012Metric_Pad1.15x1.40mm_HandSolder" V 2980 6400 50  0001 C CNN
 F 3 "~" H 3050 6400 50  0001 C CNN
+F 4 " 311-1.00CRCT-ND" H 3050 6400 50  0001 C CNN "Digikey"
 	1    3050 6400
 	0    1    1    0
@@
 F 2 "Resistor_THT:R_Axial_DIN0309_L9.0mm_D3.2mm_P15.24mm_Horizontal" V 4130 6400 50  0001 C CNN
 F 3 "~" H 4200 6400 50  0001 C CNN
+F 4 "BC4422CT-ND" H 4200 6400 50  0001 C CNN "Digikey"
 	1    4200 6400
 	1    0    0    -1
@@
 F 2 "Resistor_THT:R_Axial_DIN0309_L9.0mm_D3.2mm_P15.24mm_Horizontal" V 5730 6400 50  0001 C CNN
 F 3 "~" H 5800 6400 50  0001 C CNN
+F 4 "BC4422CT-ND" H 5800 6400 50  0001 C CNN "Digikey"
 	1    5800 6400
 	1    0    0    -1
@@
 F 2 "Resistor_SMD:R_0805_2012Metric_Pad1.15x1.40mm_HandSolder" V 5730 6800 50  0001 C CNN
 F 3 "~" H 5800 6800 50  0001 C CNN
+F 4 " 311-1.00KCRCT-ND" H 5800 6800 50  0001 C CNN "Digikey"
 	1    5800 6800
 	1    0    0    -1
@@
 F 2 "Package_TO_SOT_SMD:SOT-23-5" H 2400 6000 50  0001 C CIN
 F 3 "http://ww1.microchip.com/downloads/en/DeviceDoc/20002092F.pdf" H 2200 6650 50  0001 C CNN
+F 4 "MCP1416T-E/OTCT-ND" H 2400 6400 50  0001 C CNN "Digikey"
 	1    2400 6400
 	1    0    0    -1
@@
 F 2 "Package_SO:HTSSOP-28-1EP_4.4x9.7mm_P0.65mm_EP2.85x5.4mm" H 3350 4100 50  0001 C CNN
 F 3 "" H 2850 3700 50  0001 C CNN
+F 4 "LTC7149IFE#PBF-ND" H 3350 4100 50  0001 C CNN "Digikey"
 	1    3350 4100
 	1    0    0    -1
@@
 F 2 "Resistor_SMD:R_0805_2012Metric_Pad1.15x1.40mm_HandSolder" V 4030 4900 50  0001 C CNN
 F 3 "~" H 4100 4900 50  0001 C CNN
+F 4 " 311-100KCRCT-ND" H 4100 4900 50  0001 C CNN "Digikey"
 	1    4100 4900
 	1    0    0    -1
@@
 F 2 "Resistor_SMD:R_0805_2012Metric_Pad1.15x1.40mm_HandSolder" V 4380 4900 50  0001 C CNN
 F 3 "~" H 4450 4900 50  0001 C CNN
+F 4 "311-240KCRCT-ND " H 4450 4900 50  0001 C CNN "Digikey"
 	1    4450 4900
 	1    0    0    -1
@@
 F 2 "Resistor_SMD:R_0805_2012Metric_Pad1.15x1.40mm_HandSolder" V 9030 3350 50  0001 C CNN
 F 3 "~" H 9100 3350 50  0001 C CNN
+F 4 "311-10.5KCRCT-ND " H 9100 3350 50  0001 C CNN "Digikey"
 	1    9100 3350
 	1    0    0    -1
@@
 F 2 "Package_SO:TI_SO-PowerPAD-8_ThermalVias" H 7250 2350 50  0001 L CIN
 F 3 "http://www.ti.com/lit/ds/symlink/tps54360.pdf" H 7200 2800 50  0001 C CNN
+F 4 "296-37676-1-ND" H 7200 2800 50  0001 C CNN "Digikey"
 	1    7200 2800
 	1    0    0    -1
@@
 F 2 "Resistor_SMD:R_0805_2012Metric_Pad1.15x1.40mm_HandSolder" V 6430 2950 50  0001 C CNN
 F 3 "~" H 6500 2950 50  0001 C CNN
+F 4 " 	311-249KCRCT-ND" H 6500 2950 50  0001 C CNN "Digikey"
 	1    6500 2950
 	1    0    0    -1
@@
 F 2 "Resistor_SMD:R_0805_2012Metric_Pad1.15x1.40mm_HandSolder" V 9030 2950 50  0001 C CNN
 F 3 "~" H 9100 2950 50  0001 C CNN
+F 4 "311-147KCRCT-ND" H 9100 2950 50  0001 C CNN "Digikey"
 	1    9100 2950
 	1    0    0    -1
@@
 F 2 "Resistor_SMD:R_0805_2012Metric_Pad1.15x1.40mm_HandSolder" V 7780 3050 50  0001 C CNN
 F 3 "~" H 7850 3050 50  0001 C CNN
+F 4 " 	311-15.4KCRCT-ND " H 7850 3050 50  0001 C CNN "Digikey"
 	1    7850 3050
 	1    0    0    -1
@@
 F 2 "Resistor_SMD:R_0805_2012Metric_Pad1.15x1.40mm_HandSolder" V 9680 5550 50  0001 C CNN
 F 3 "~" H 9750 5550 50  0001 C CNN
+F 4 " 311-1.00CRCT-ND" H 9750 5550 50  0001 C CNN "Digikey"
 	1    9750 5550
 	1    0    0    -1
