File: td-deflect/td-deflect.sch (KiCad schematic (older format))
At the start: 53 parts, among them J1 Conn_01x02_Male, J2 Conn_01x02_Male, J3 Conn_01x02_Male, Q1 LMG5200, Q2 C2M0045170D, Q3 LMG5200, Q4 LMG5200, Q5 LMG5200, U1 MCP1416

Commit message: drop some of the old GaNs
Parts:
- removed C1, C10, C2, C9: 0.1uF, Capacitor_SMD:C_0603_1608Metric_Pad1.05x0.95mm_HandSolder, symbol Device:C
- removed C17, C18: 47uF, Capacitor_THT:CP_Radial_D10.0mm_P5.00mm, symbol Device:C
- removed L2: 47uH, Inductor_SMD:L_Bourns_SRP1245A, symbol Device:L
- removed Q1, Q3: LMG5200, Package_DFN_QFN:Texas_MOF0009A, symbol Power_Management:LMG5200
- added C? (x2): 0.1uF, Capacitor_SMD:C_0603_1608Metric_Pad1.05x0.95mm_HandSolder, symbol Device:C
- added C?: 1000pF, Capacitor_SMD:C_0603_1608Metric_Pad1.05x0.95mm_HandSolder, symbol Device:C
- added C?: 8200pF, Capacitor_SMD:C_0603_1608Metric_Pad1.05x0.95mm_HandSolder, symbol Device:C
- added C?: 330uF, Capacitor_SMD:C_0603_1608Metric_Pad1.05x0.95mm_HandSolder, symbol Device:C
- added C?: 20uF, Capacitor_SMD:C_0603_1608Metric_Pad1.05x0.95mm_HandSolder, symbol Device:C
- added C?: 1uF, Capacitor_SMD:C_0603_1608Metric_Pad1.05x0.95mm_HandSolder, symbol Device:C
- added D?: D, symbol Device:D
- added L?: 33uH, symbol Device:L
- added Q?: Q_NMOS_GDS, symbol Device:Q_NMOS_GDS
- added R?: 0.01, symbol Device:R
- added R?: 100, symbol Device:R
- added R?: 3.57k, symbol Device:R
- added R?: 20k, symbol Device:R
- added R?: 221, symbol Device:R
- added R?: 86.6k, symbol Device:R
- added R?: 10k, symbol Device:R
- added R?: 1.69k, symbol Device:R
- added U?: LM5022MM, Package_SO:MSOP-10_3x3mm_P0.5mm, symbol Regulator_Switching:LM5022MM
Connections:
- net labels removed: B_HI, B_LI, S_HI, S_LI
- wire segments 78 -> 108
Other:
- moved on the sheet: C3, C4, C5, C7, C8

Commit message: Add power supplies
Parts:
- removed C12, C13, C14, C19, C20, C21, C22, C25, C26, C27, C28, C29, C3, C30, C4, C5: 0.1uF, Capacitor_SMD:C_0603_1608Metric_Pad1.05x0.95mm_HandSolder, symbol Device:C
- removed C15, C16, C31, C32, C33, C34, C7, C8: 4.7uF, Capacitor_SMD:C_1210_3225Metric_Pad1.42x2.65mm_HandSolder, symbol Device:C
- removed C23, C24: 2uF, Capacitor_SMD:C_1210_3225Metric_Pad1.42x2.65mm_HandSolder, symbol Device:C
- removed J3: Conn_01x02_Male, Connector_Wire:SolderWirePad_1x02_P7.62mm_Drill2mm, symbol Connector:Conn_01x02_Male
- removed L3, L4: 10uH, Inductor_SMD:L_Bourns_SRP1245A, symbol Device:L
- removed Q4, Q5: LMG5200, Package_DFN_QFN:Texas_MOF0009A, symbol Power_Management:LMG5200
- removed R1, R3: 1M, Capacitor_SMD:C_0603_1608Metric_Pad1.05x0.95mm_HandSolder, symbol Device:R
- added C?: 0.015uF, Capacitor_SMD:C_1210_3225Metric_Pad1.42x2.65mm_HandSolder, symbol Device:C
- added C?: 0.12uF, Capacitor_SMD:C_1210_3225Metric_Pad1.42x2.65mm_HandSolder, symbol Device:C
- added C? (x2): C, symbol Device:C
- added C?: 0.033uF, Capacitor_SMD:C_1210_3225Metric_Pad1.42x2.65mm_HandSolder, symbol Device:C
- added C?: 0.068uF, Capacitor_SMD:C_1210_3225Metric_Pad1.42x2.65mm_HandSolder, symbol Device:C
- added D?: D_TVS, symbol Device:D_TVS
- added L?: LTRIM, symbol Device:LTRIM
- added Q? (x4): IPD50R380CE, Package_TO_SOT_SMD:TO-252-2, symbol Transistor_FET:IPD50R380CE
- added R?: 1M, Capacitor_SMD:C_0603_1608Metric_Pad1.05x0.95mm_HandSolder, symbol Device:R
- added R? (x2): 10k, symbol Device:R
- added R? (x4): R, symbol Device:R
- added U? (x2): MIC4427, symbol Driver_FET:MIC4427
- C11: value 2uF -> 0.033uF
- C6: value 0.01uF -> 0.0073uF
- R2: value 2 -> 1
Connections:
- net labels added: S0, S1, S2, S3
- net labels removed: +5V, V1_HI, V1_LI, V2_HI, V2_LI, h.return
- wire segments 108 -> 89
Other:
- moved on the sheet: C11, R5

Commit message: drop LM5022 boost
Parts:
- removed C? (x2): 0.1uF, Capacitor_SMD:C_0603_1608Metric_Pad1.05x0.95mm_HandSolder, symbol Device:C
- removed C?: 1000pF, Capacitor_SMD:C_0603_1608Metric_Pad1.05x0.95mm_HandSolder, symbol Device:C
- removed C?: 8200pF, Capacitor_SMD:C_0603_1608Metric_Pad1.05x0.95mm_HandSolder, symbol Device:C
- removed C?: 330uF, Capacitor_SMD:C_0603_1608Metric_Pad1.05x0.95mm_HandSolder, symbol Device:C
- removed C?: 20uF, Capacitor_SMD:C_0603_1608Metric_Pad1.05x0.95mm_HandSolder, symbol Device:C
- removed C?: 1uF, Capacitor_SMD:C_0603_1608Metric_Pad1.05x0.95mm_HandSolder, symbol Device:C
- removed D?: D, symbol Device:D
- removed L?: 33uH, symbol Device:L
- removed Q?: Q_NMOS_GDS, symbol Device:Q_NMOS_GDS
- removed R?: 0.01, symbol Device:R
- removed R?: 100, symbol Device:R
- removed R?: 3.57k, symbol Device:R
- removed R?: 20k, symbol Device:R
- removed R?: 221, symbol Device:R
- removed R?: 86.6k, symbol Device:R
- removed R?: 10k, symbol Device:R
- removed R?: 1.69k, symbol Device:R
- removed U?: LM5022MM, Package_SO:MSOP-10_3x3mm_P0.5mm, symbol Regulator_Switching:LM5022MM
Connections:
- wire segments 89 -> 46

Commit message: Update firmware to not use a git version of hal
Parts:
- removed D?: D_TVS, symbol Device:D_TVS
- added C?: C, symbol Device:C
- added J?: DB15_Female_HighDensity, symbol Connector:DB15_Female_HighDensity
- added U?: AD813, symbol Amplifier_Video:AD813
- added U?: 24LC08, symbol Memory_EEPROM:24LC08
Connections:
- net labels added: blue, green, hsync, red, vsync
- wire segments 46 -> 72
Changed lines of the file:
@@
 S3
-$Comp
-L Device:D_TVS D?
-U 1 1 5D9EBF26
-P 9800 3650
-F 0 "D?" V 9754 3729 50  0000 L CNN
-F 1 "D_TVS" V 9845 3729 50  0000 L CNN
-F 2 "" H 9800 3650 50  0001 C CNN
-F 3 "~" H 9800 3650 50  0001 C CNN
-	1    9800 3650
-	0    1    1    0
-$EndComp
-Wire Wire Line
-	9100 3500 9800 3500
-Connection ~ 9100 3500
-$Comp
-L power:GND #PWR?
-U 1 1 5D9ECF79
-P 9800 3800
-F 0 "#PWR?" H 9800 3550 50  0001 C CNN
-F 1 "GND" H 9805 3627 50  0000 C CNN
-F 2 "" H 9800 3800 50  0001 C CNN
-F 3 "" H 9800 3800 50  0001 C CNN
-	1    9800 3800
-	1    0    0    -1
-$EndComp
 $Comp
 L Device:R R?
@@
 	9250 3800 9250 3850
 Connection ~ 9100 3800
+$Comp
+L Amplifier_Video:AD813 U?
+U 1 1 5D9F2C9A
+P 4450 1200
+F 0 "U?" H 4450 1567 50  0000 C CNN
+F 1 "AD813" H 4450 1476 50  0000 C CNN
+F 2 "" H 4450 1200 50  0001 C CNN
+F 3 "https://www.analog.com/media/en/technical-documentation/data-sheets/AD813.pdf" H 4450 1200 50  0001 C CNN
+	1    4450 1200
+	1    0    0    -1
+$EndComp
+$Comp
+L Connector:DB15_Female_HighDensity J?
+U 1 1 5D9F6269
+P 1800 1750
+F 0 "J?" H 1800 2617 50  0000 C CNN
+F 1 "DB15_Female_HighDensity" H 1800 2526 50  0000 C CNN
+F 2 "" H 850 2150 50  0001 C CNN
+F 3 " ~" H 850 2150 50  0001 C CNN
+	1    1800 1750
+	1    0    0    -1
+$EndComp
+Text Label 1500 1350 2    50   ~ 0
+red
+Text Label 1500 1550 2    50   ~ 0
+green
+Text Label 1500 1750 2    50   ~ 0
+blue
+Text Label 2100 1750 0    50   ~ 0
+hsync
+Text Label 2100 1950 0    50   ~ 0
+vsync
+$Comp
+L power:GND #PWR?
+U 1 1 5D9F853D
+P 1100 2250
+F 0 "#PWR?" H 1100 2000 50  0001 C CNN
+F 1 "GND" H 1105 2077 50  0000 C CNN
+F 2 "" H 1100 2250 50  0001 C CNN
+F 3 "" H 1100 2250 50  0001 C CNN
+	1    1100 2250
+	1    0    0    -1
+$EndComp
+Wire Wire Line
+	1100 1250 1500 1250
+Wire Wire Line
+	1500 1450 1100 1450
+Connection ~ 1100 1450
+Wire Wire Line
+	1100 1450 1100 1250
+Wire Wire Line
+	1500 1650 1100 1650
+Wire Wire Line
+	1100 1450 1100 1650
+Connection ~ 1100 1650
+Wire Wire Line
+	1500 2150 1100 2150
+Connection ~ 1100 2150
+Wire Wire Line
+	1100 2150 1100 2250
+Wire Wire Line
+	1500 2050 1100 2050
+Wire Wire Line
+	1100 1650 1100 2050
+Connection ~ 1100 2050
+Wire Wire Line
+	1100 2050 1100 2150
+$Comp
+L Memory_EEPROM:24LC08 U?
+U 1 1 5D9FB930
+P 3200 1400
+F 0 "U?" H 3200 1881 50  0000 C CNN
+F 1 "24LC08" H 3200 1790 50  0000 C CNN
+F 2 "" H 3200 1400 50  0001 C CNN
+F 3 "http://ww1.microchip.com/downloads/en/DeviceDoc/21710J.pdf" H 3200 1400 50  0001 C CNN
+	1    3200 1400
+	1    0    0    -1
+$EndComp
+Wire Wire Line
+	1150 700  3200 700
+Wire Wire Line
+	3200 700  3200 1100
+Wire Wire Line
+	1150 1850 1500 1850
+Wire Wire Line
+	1150 700  1150 1850
+$Comp
+L power:GND #PWR?
+U 1 1 5D9FE30E
+P 3200 1700
+F 0 "#PWR?" H 3200 1450 50  0001 C CNN
+F 1 "GND" H 3205 1527 50  0000 C CNN
+F 2 "" H 3200 1700 50  0001 C CNN
+F 3 "" H 3200 1700 50  0001 C CNN
+	1    3200 1700
+	1    0    0    -1
+$EndComp
+Connection ~ 3200 1700
+Wire Wire Line
+	3600 1500 3600 1700
+Wire Wire Line
+	3600 1700 3200 1700
+Wire Wire Line
+	2800 1300 2800 1400
+Wire Wire Line
+	2800 1400 2800 1500
+Connection ~ 2800 1400
+Wire Wire Line
+	2800 1500 2800 1700
+Wire Wire Line
+	2800 1700 3200 1700
+Connection ~ 2800 1500
+Wire Wire Line
+	3600 1300 3600 1050
+Wire Wire Line
+	3600 1050 2450 1050
+Wire Wire Line
+	2450 1050 2450 1550
+Wire Wire Line
+	2450 1550 2100 1550
+Wire Wire Line
+	2100 2150 3700 2150
+Wire Wire Line
+	3700 2150 3700 1400
+Wire Wire Line
+	3700 1400 3600 1400
+$Comp
+L power:+12V #PWR?
+U 1 1 5D9FF195
+P 2200 3650
+F 0 "#PWR?" H 2200 3500 50  0001 C CNN
+F 1 "+12V" H 2215 3823 50  0000 C CNN
+F 2 "" H 2200 3650 50  0001 C CNN
+F 3 "" H 2200 3650 50  0001 C CNN
+	1    2200 3650
+	1    0    0    -1
+$EndComp
+$Comp
+L Device:C C?
+U 1 1 5D9FF1A3
+P 2200 3800
+F 0 "C?" H 2315 3846 50  0000 L CNN
+F 1 "C" H 2315 3755 50  0000 L CNN
+F 2 "" H 2238 3650 50  0001 C CNN
+F 3 "~" H 2200 3800 50  0001 C CNN
+	1    2200 3800
+	1    0    0    -1
+$EndComp
+$Comp
+L power:GND #PWR?
+U 1 1 5D9FF1B4
+P 2200 3950
+F 0 "#PWR?" H 2200 3700 50  0001 C CNN
+F 1 "GND" H 2205 3777 50  0000 C CNN
+F 2 "" H 2200 3950 50  0001 C CNN
+F 3 "" H 2200 3950 50  0001 C CNN
+	1    2200 3950
+	1    0    0    -1
+$EndComp
 $EndSCHEMATC

Commit message: add lots of stuff
Parts:
- removed C? (x2): C, symbol Device:C
- removed C?: 0.033uF, Capacitor_SMD:C_1210_3225Metric_Pad1.42x2.65mm_HandSolder, symbol Device:C
- removed C?: 0.068uF, Capacitor_SMD:C_1210_3225Metric_Pad1.42x2.65mm_HandSolder, symbol Device:C
- removed J2: Conn_01x02_Male, Connector_Wire:SolderWirePad_1x02_P7.62mm_Drill2mm, symbol Connector:Conn_01x02_Male
- removed J?: DB15_Female_HighDensity, symbol Connector:DB15_Female_HighDensity
- removed Q? (x2): IPD50R380CE, Package_TO_SOT_SMD:TO-252-2, symbol Transistor_FET:IPD50R380CE
- removed R5: 1M, Capacitor_SMD:C_0603_1608Metric_Pad1.05x0.95mm_HandSolder, symbol Device:R
- removed R? (x2): R, symbol Device:R
- removed U?: AD813, symbol Amplifier_Video:AD813
- removed U?: 24LC08, symbol Memory_EEPROM:24LC08
- added C1, C10, C3, C4, C5, C7, C8, C9: 0.1uF, Capacitor_SMD:C_0805_2012Metric_Pad1.15x1.40mm_HandSolder, symbol Device:C
- added C12: 0.01uF, Capacitor_SMD:C_0805_2012Metric_Pad1.15x1.40mm_HandSolder, symbol Device:C
- added C14: 0.033uF, Capacitor_SMD:C_1210_3225Metric_Pad1.42x2.65mm_HandSolder, symbol Device:C
- added C15: 0.068uF, Capacitor_SMD:C_1210_3225Metric_Pad1.42x2.65mm_HandSolder, symbol Device:C
- added D1: BA157, Diode_THT:D_DO-41_SOD81_P10.16mm_Horizontal, symbol Diode:BA157
- added D2: C3D10170H, Package_TO_SOT_THT:TO-247-2_Vertical, symbol Diode:C3D10170H
- added J10, J11, J3: Conn_01x02_Male, Connector_Phoenix_MSTB:PhoenixContact_MSTBVA_2,5_2-G_1x02_P5.00mm_Vertical, symbol Connector:Conn_01x02_Male
- added J12: Conn_01x06_Male, symbol Connector:Conn_01x06_Male
- added Q1, Q3: BSC082N10LSG, Package_TO_SOT_SMD:TDSON-8-1, symbol Transistor_FET:BSC082N10LSG
- added Q4: BCP56, Package_TO_SOT_SMD:SOT-223-3_TabPin2, symbol Transistor_BJT:BCP56
- added Q5: BCP53, Package_TO_SOT_SMD:SOT-223-3_TabPin2, symbol Transistor_BJT:BCP53
- added Q6: MJD44, Package_TO_SOT_SMD:TO-252-2, symbol Transistor_BJT:BD249A
- added Q7: MJD45, Package_TO_SOT_SMD:TO-252-2, symbol Transistor_BJT:BD250A
- added Q8, Q9: IPD50R380CE, Package_TO_SOT_SMD:TO-252-2, symbol Transistor_FET:IPD50R380CE
- added R1, R11, R14, R3, R7, R8, R9: 10k, Resistor_SMD:R_0805_2012Metric_Pad1.15x1.40mm_HandSolder, symbol Device:R
- added R13, R15, R16: 100, Resistor_SMD:R_0805_2012Metric_Pad1.15x1.40mm_HandSolder, symbol Device:R
- added R17, R18, R19, R22: 1, Resistor_SMD:R_0805_2012Metric_Pad1.15x1.40mm_HandSolder, symbol Device:R
- added R20: 220k, Resistor_SMD:R_0805_2012Metric_Pad1.15x1.40mm_HandSolder, symbol Device:R
- added R21: 1k, Resistor_SMD:R_0805_2012Metric_Pad1.15x1.40mm_HandSolder, symbol Device:R
- added R23, R24, R27: 100k, Resistor_SMD:R_1206_3216Metric_Pad1.42x1.75mm_HandSolder, symbol Device:R
- added R28: 1k, Resistor_SMD:R_1206_3216Metric_Pad1.42x1.75mm_HandSolder, symbol Device:R
- added T1: CST1, Transformer_SMD:Transformer_Coilcraft_CST1, symbol Transformer:CST1
- added U5: TL082, Package_SO:SOIC-8_3.9x4.9mm_P1.27mm, symbol Amplifier_Operational:TL082
- added U6: IRS2005S, Package_SO:SOIC-8_3.9x4.9mm_P1.27mm, symbol Driver_FET:IRS2005S
- added U7: LTC6090, Package_SO:SOIC-8-1EP_3.9x4.9mm_P1.27mm_EP2.29x3mm, symbol td-deflect:LTC6090
- added U8: INA181, Package_TO_SOT_SMD:SOT-23-6, symbol Amplifier_Current:INA181
- C11: Voltage (none) -> 200V
- C13, C16: renamed from C?; Voltage (none) -> 200V
- C2: renamed from C?; value C -> 0.1uF; footprint (none) -> Capacitor_SMD:C_0805_2012Metric_Pad1.15x1.40mm_HandSolder
- C6: footprint Capacitor_SMD:C_1210_3225Metric_Pad1.42x2.65mm_HandSolder -> Capacitor_THT:C_Rect_L18.0mm_W6.0mm_P15.00mm_FKS3_FKP3; Digikey (none) -> 495-3231-ND; Voltage (none) -> 2000V
- E1: Voltage (none) -> 1800V
- J1: footprint Connector_Wire:SolderWirePad_1x02_P7.62mm_Drill2mm -> Connector_Phoenix_MSTB:PhoenixContact_MSTBVA_2,5_2-G_1x02_P5.00mm_Vertical
- R10, R5: renamed from R?; footprint (none) -> Resistor_SMD:R_0805_2012Metric_Pad1.15x1.40mm_HandSolder
- R12: renamed from R?; footprint Capacitor_SMD:C_0603_1608Metric_Pad1.05x0.95mm_HandSolder -> Resistor_THT:R_Axial_DIN0309_L9.0mm_D3.2mm_P15.24mm_Horizontal; Digikey (none) -> BC4422CT-ND; Voltage (none) -> 1700V
- R2: footprint Resistor_SMD:R_MELF_MMB-0207 -> Resistor_SMD:R_0805_2012Metric_Pad1.15x1.40mm_HandSolder
- R25, R26: renamed from R?; value R -> 100k; footprint (none) -> Resistor_SMD:R_1206_3216Metric_Pad1.42x1.75mm_HandSolder
- U10, U9: renamed from U?; footprint (none) -> Package_SO:SOIC-8_3.9x4.9mm_P1.27mm
- gave numbers to parts that had none: 3
Connections:
- net labels added: +1V5, +3.3V, +48V, -12V, H_CURRENT, PIN_HI, PIN_LO, S_VOLTAGE, V_DAC, h.ret, hsupply, v.out, v.ret
- net labels removed: blue, green, hsync, red, vsync
- wire segments 72 -> 129
Other:
- note added: "H.LIN"
- note added: "H.YOKE"
- note added: "MS9 connector"
- note added: "PVM-1390 connector"
- note added: "V.YOKE"
- note added: "saturable\nreactor"
- moved on the sheet: C10, C11, C13, C15, C16, C2, C6, E1, J1, L1, L2, Q10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

Commit message: more stuff
Parts:
- added H? (x4): MountingHole_Pad, MountingHole:MountingHole_3.2mm_M3_Pad_Via, symbol Mechanical:MountingHole_Pad
- Q6: value MJD44 -> BD139; footprint Package_TO_SOT_SMD:TO-252-2 -> Package_TO_SOT_THT:TO-126-3_Vertical; symbol Transistor_BJT:BD249A -> Transistor_BJT:BD139
- Q7: value MJD45 -> BD140; footprint Package_TO_SOT_SMD:TO-252-2 -> Package_TO_SOT_THT:TO-126-3_Vertical; symbol Transistor_BJT:BD250A -> Transistor_BJT:BD140
Connections:
- wire segments 129 -> 132
Changed lines of the file:
@@
 $EndComp
 $Comp
-L Transistor_BJT:BD250A Q7
+L Transistor_BJT:BD140 Q7
 U 1 1 5DA3CB2C
 P 5650 6700
 F 0 "Q7" H 5842 6746 50  0000 L CNN
-F 1 "MJD45" H 5842 6655 50  0000 L CNN
-F 2 "Package_TO_SOT_SMD:TO-252-2" H 5855 6620 50  0001 L CIN
-F 3 "http://www.mospec.com.tw/pdf/power/BD249.pdf" H 5650 6700 50  0001 L CNN
+F 1 "BD140" H 5842 6655 50  0000 L CNN
+F 2 "Package_TO_SOT_THT:TO-126-3_Vertical" H 5855 6620 50  0001 L CIN
+F 3 "http://www.st.com/internet/com/TECHNICAL_RESOURCES/TECHNICAL_LITERATURE/DATASHEET/CD00001225.pdf" H 5650 6700 50  0001 L CNN
 	1    5650 6700
 	1    0    0    -1
 $EndComp
 $Comp
-L Transistor_BJT:BD249A Q6
+L Transistor_BJT:BD139 Q6
 U 1 1 5DA3D22D
 P 5650 5500
 F 0 "Q6" H 5842 5546 50  0000 L CNN
-F 1 "MJD44" H 5842 5455 50  0000 L CNN
-F 2 "Package_TO_SOT_SMD:TO-252-2" H 5900 5425 50  0001 L CIN
-F 3 "http://www.mospec.com.tw/pdf/power/BD249.pdf" H 5650 5500 50  0001 L CNN
+F 1 "BD139" H 5842 5455 50  0000 L CNN
+F 2 "Package_TO_SOT_THT:TO-126-3_Vertical" H 5900 5425 50  0001 L CIN
+F 3 "http://www.st.com/internet/com/TECHNICAL_RESOURCES/TECHNICAL_LITERATURE/DATASHEET/CD00001225.pdf" H 5650 5500 50  0001 L CNN
 	1    5650 5500
 	1    0    0    -1
@@
 F1 "rgb.sch" 50
 $EndSheet
+$Comp
+L Mechanical:MountingHole_Pad H?
+U 1 1 5DBAF035
+P 9900 900
+F 0 "H?" H 10000 903 50  0000 L CNN
+F 1 "MountingHole_Pad" H 10000 858 50  0001 L CNN
+F 2 "MountingHole:MountingHole_3.2mm_M3_Pad_Via" H 9900 900 50  0001 C CNN
+F 3 "~" H 9900 900 50  0001 C CNN
+	1    9900 900
+	1    0    0    -1
+$EndComp
+$Comp
+L Mechanical:MountingHole_Pad H?
+U 1 1 5DBAF035
+P 10200 900
+F 0 "H?" H 10300 903 50  0000 L CNN
+F 1 "MountingHole_Pad" H 10300 858 50  0001 L CNN
+F 2 "MountingHole:MountingHole_3.2mm_M3_Pad_Via" H 10200 900 50  0001 C CNN
+F 3 "~" H 10200 900 50  0001 C CNN
+	1    10200 900
+	1    0    0    -1
+$EndComp
+$Comp
+L Mechanical:MountingHole_Pad H?
+U 1 1 5DBB0FA7
+P 10500 900
+F 0 "H?" H 10600 903 50  0000 L CNN
+F 1 "MountingHole_Pad" H 10600 858 50  0001 L CNN
+F 2 "MountingHole:MountingHole_3.2mm_M3_Pad_Via" H 10500 900 50  0001 C CNN
+F 3 "~" H 10500 900 50  0001 C CNN
+	1    10500 900
+	1    0    0    -1
+$EndComp
+$Comp
+L Mechanical:MountingHole_Pad H?
+U 1 1 5DBB1105
+P 10800 900
+F 0 "H?" H 10900 903 50  0000 L CNN
+F 1 "MountingHole_Pad" H 10900 858 50  0001 L CNN
+F 2 "MountingHole:MountingHole_3.2mm_M3_Pad_Via" H 10800 900 50  0001 C CNN
+F 3 "~" H 10800 900 50  0001 C CNN
+	1    10800 900
+	1    0    0    -1
+$EndComp
+Wire Wire Line
+	9900 1000 10200 1000
+Wire Wire Line
+	10500 1000 10200 1000
+Connection ~ 10200 1000
+Wire Wire Line
+	10500 1000 10800 1000
+Connection ~ 10500 1000
+$Comp
+L power:GND #PWR?
+U 1 1 5DBB13D6
+P 9900 1000
+F 0 "#PWR?" H 9900 750 50  0001 C CNN
+F 1 "GND" H 9905 827 50  0000 C CNN
+F 2 "" H 9900 1000 50  0001 C CNN
+F 3 "" H 9900 1000 50  0001 C CNN
+	1    9900 1000
+	1    0    0    -1
+$EndComp
+Connection ~ 9900 1000
 $EndSCHEMATC

Commit message: asdf
Parts:
- removed H? (x2): MountingHole_Pad, MountingHole:MountingHole_3.2mm_M3_Pad_Via, symbol Mechanical:MountingHole_Pad
- removed J1: Conn_01x02_Male, Connector_Phoenix_MSTB:PhoenixContact_MSTBVA_2,5_2-G_1x02_P5.00mm_Vertical, symbol Connector:Conn_01x02_Male
- added F1, F2: Fuse, Fuse:Fuse_Schurter_UMT250, symbol Device:Fuse
- added H1, H2: MountingHole_Pad, MountingHole:MountingHole_3.2mm_M3_Pad_Via, symbol Mechanical:MountingHole_Pad
- C1, C10, C2, C3, C4, C5, C7, C8, C9: Digikey (none) -> 1276-1099-1-ND
- C11, C14: footprint Capacitor_SMD:C_1210_3225Metric_Pad1.42x2.65mm_HandSolder -> Capacitor_SMD:C_1206_3216Metric_Pad1.42x1.75mm_HandSolder; Digikey (none) -> 1276-3159-1-ND
- C12: Digikey (none) -> 1276-2921-6-ND
- C13: footprint Capacitor_SMD:C_1210_3225Metric_Pad1.42x2.65mm_HandSolder -> Capacitor_SMD:C_1206_3216Metric_Pad1.42x1.75mm_HandSolder; Digikey (none) -> 311-1980-1-ND
- C15: footprint Capacitor_SMD:C_1210_3225Metric_Pad1.42x2.65mm_HandSolder -> Capacitor_SMD:C_1206_3216Metric_Pad1.42x1.75mm_HandSolder; Digikey (none) -> 311-4473-1-ND
- C16: footprint Capacitor_SMD:C_1210_3225Metric_Pad1.42x2.65mm_HandSolder -> Capacitor_SMD:C_1206_3216Metric_Pad1.42x1.75mm_HandSolder; Digikey (none) -> 399-17948-1-ND
- C6: Digikey 495-3231-ND -> 495-3231-ND
- D1: Digikey (none) -> BA157-E3/54GICT-ND
- D2: Digikey (none) -> C3D10170H-ND
- E1: footprint Capacitor_SMD:C_1825_4564Metric_Pad1.88x6.70mm_HandSolder -> Resistor_THT:R_Axial_DIN0309_L9.0mm_D3.2mm_P12.70mm_Horizontal; Digikey F7596TR-ND -> F3681-ND; Voltage 1800V -> 2000V
- J10: footprint Connector_Phoenix_MSTB:PhoenixContact_MSTBVA_2,5_2-G_1x02_P5.00mm_Vertical -> td-deflect:monitor_10_8_2p
- J11: footprint Connector_Phoenix_MSTB:PhoenixContact_MSTBVA_2,5_2-G_1x02_P5.00mm_Vertical -> td-deflect:sony_monitor_2p
- J12: footprint (none) -> td-deflect:sony_monitor_yoke
- J3: Digikey (none) -> 277-1150-ND
- L2: footprint (none) -> td-deflect:LIN-3509
- Q1, Q3: Digikey (none) -> BSC082N10LSGATMA1CT-ND
- Q10, Q11, Q8, Q9: Digikey (none) -> IPD50R380CEAUMA1CT-ND
- Q2: Digikey (none) -> C2M0045170D-ND
- Q4: Digikey (none) -> BCP56-16T1GOSCT-ND
- Q5: Digikey (none) -> BCP53-16T1GOSCT-ND
- Q6: Digikey (none) -> 497-12750-5-ND
- Q7: Digikey (none) -> 497-14760-5-ND
- R4: footprint Resistor_SMD:R_0603_1608Metric_Pad1.05x0.95mm_HandSolder -> Resistor_SMD:R_0805_2012Metric_Pad1.15x1.40mm_HandSolder
- gave numbers to parts that had none: 2
Connections:
- net labels added: S_cap_top, virtual_ground
- net labels removed: +1V5
- wire segments 132 -> 140
- no-connect marks 0 -> 2
Other:
- moved on the sheet: H2
