File: td-deflect/td-deflect.kicad_pcb (KiCad board)
At the start: 2 copper layers, 70 parts, among them J1 Conn_01x02_Male, J2 Conn_01x02_Male, J3 Conn_01x02_Male, J4 Conn_ARM_JTAG_SWD_10, J5 Conn_01x02_Male, Q1 LMG5200, Q2 C2M0045170D, Q3 LMG5200, Q4 LMG5200, Q5 LMG5200, U1 MCP1416, U2 STM32F722RETx, U3 INA193, U4 TPS76933, U5 AMS1117-5.0, X1 SG-8002CA

Commit message: add lots of stuff
Parts:
- removed the C17 at (128.8, 77.8)
- removed C28: 0.1uF, Capacitor_SMD:C_0603_1608Metric_Pad1.05x0.95mm_HandSolder
- removed C32: 4.7uF, Capacitor_SMD:C_1210_3225Metric_Pad1.42x2.65mm_HandSolder
- removed L2: 47uH, Inductor_SMD:L_Bourns_SRP1245A
- removed L3, L4: 10uH, Inductor_SMD:L_Bourns_SRP1245A
- added C43: 0.1uF, Capacitor_SMD:C_0805_2012Metric_Pad1.15x1.40mm_HandSolder, F.Cu at (203.6, 36.7)
- added C44: 0.033uF, Capacitor_SMD:C_0805_2012Metric_Pad1.15x1.40mm_HandSolder, F.Cu at (205.0, 50.5)
- added C45: 22pF, Capacitor_SMD:C_0805_2012Metric_Pad1.15x1.40mm_HandSolder, F.Cu at (200.0, 47.3)
- added D1: BA157, Diode_THT:D_DO-41_SOD81_P10.16mm_Horizontal, F.Cu at (119.0, 23.0)
- added D2: C3D10170H, Package_TO_SOT_THT:TO-247-2_Vertical, F.Cu at (118.0, 106.0)
- added D3: 1N5402, Diode_THT:D_DO-201AD_P15.24mm_Horizontal, F.Cu at (86.0, 10.0)
- added D4: C3D10170H, Package_TO_SOT_THT:TO-247-2_Vertical, F.Cu at (201.0, 107.0)
- added D5: B220, Diode_SMD:D_SMB, F.Cu at (211.6, 37.5)
- added E2: SPARK_GAP, Capacitor_SMD:C_1825_4564Metric_Pad1.88x6.70mm_HandSolder, F.Cu at (200.0, 96.0)
- added J10: Conn_01x02_Male, Connector_Phoenix_MSTB:PhoenixContact_MSTBVA_2,5_2-G_1x02_P5.00mm_Vertical, F.Cu at (160.0, 104.0)
- added J11: Conn_01x02_Male, Connector_Phoenix_MSTB:PhoenixContact_MSTBVA_2,5_2-G_1x02_P5.00mm_Vertical, F.Cu at (61.0, 106.0)
- added J13: Conn_01x02_Male, Connector_Phoenix_MSTB:PhoenixContact_MSTBVA_2,5_2-G_1x02_P5.00mm_Vertical, F.Cu at (219.0, 15.0)
- added J14: Conn_01x02_Male, Connector_Phoenix_MSTB:PhoenixContact_MSTBVA_2,5_2-G_1x02_P5.00mm_Vertical, F.Cu at (218.0, 46.5)
- added J6: Conn_01x06_Male, Connector_PinHeader_2.54mm:PinHeader_1x06_P2.54mm_Vertical, F.Cu at (-7.42, 37.2)
- added J8: Conn_01x02_Male, Connector_Phoenix_MSTB:PhoenixContact_MSTBVA_2,5_2-G_1x02_P5.00mm_Vertical, F.Cu at (220.0, 95.0)
- added J9: Conn_01x02_Male, Connector_Phoenix_MSTB:PhoenixContact_MSTBVA_2,5_2-G_1x02_P5.00mm_Vertical, F.Cu at (195.5, 72.0)
- added Q10: IPD50R380CE, Package_TO_SOT_SMD:TO-252-2, F.Cu at (154.0, 38.0)
- added Q11: IPD50R380CE, Package_TO_SOT_SMD:TO-252-2, F.Cu at (154.0, 47.0)
- added Q12: C2M0045170D, Package_TO_SOT_THT:TO-247-3_Vertical, F.Cu at (220.0, 107.0)
- added Q13: BSC082N10LSG, Package_TO_SOT_SMD:TDSON-8-1, F.Cu at (61.4, 10.0)
- added Q6: MJD44, Package_TO_SOT_SMD:TO-252-2, F.Cu at (83.0, 71.0)
- added Q7: MJD45, Package_TO_SOT_SMD:TO-252-2, F.Cu at (63.0, 71.0)
- added Q8: IPD50R380CE, Package_TO_SOT_SMD:TO-252-2, F.Cu at (154.1, 19.0)
- added Q9: IPD50R380CE, Package_TO_SOT_SMD:TO-252-2, F.Cu at (154.0, 28.5)
- added R10: 10k, Resistor_SMD:R_0805_2012Metric_Pad1.15x1.40mm_HandSolder, F.Cu at (151.0, 99.0)
- added R11: 10k, Resistor_SMD:R_0805_2012Metric_Pad1.15x1.40mm_HandSolder, F.Cu at (80.0, 41.0)
- added R12: 1M, Resistor_THT:R_Axial_DIN0309_L9.0mm_D3.2mm_P15.24mm_Horizontal, F.Cu at (166.6, 76.0)
- added R13: 100, Resistor_SMD:R_0805_2012Metric_Pad1.15x1.40mm_HandSolder, F.Cu at (61.0, 53.0)
- added R14: 10k, Resistor_SMD:R_0805_2012Metric_Pad1.15x1.40mm_HandSolder, F.Cu at (75.0, 79.0)
- added R15: 100, Resistor_SMD:R_0805_2012Metric_Pad1.15x1.40mm_HandSolder, F.Cu at (75.0, 71.0)
- added R16: 100, Resistor_SMD:R_0805_2012Metric_Pad1.15x1.40mm_HandSolder, F.Cu at (71.0, 71.0)
- added R17: 1, Resistor_SMD:R_0805_2012Metric_Pad1.15x1.40mm_HandSolder, F.Cu at (79.0, 79.0)
- added R18: 1, Resistor_SMD:R_0805_2012Metric_Pad1.15x1.40mm_HandSolder, F.Cu at (62.0, 87.0)
- added R19: 1, Resistor_SMD:R_0805_2012Metric_Pad1.15x1.40mm_HandSolder, F.Cu at (174.6, 65.0)
- added R20: 220k, Resistor_SMD:R_0805_2012Metric_Pad1.15x1.40mm_HandSolder, F.Cu at (71.0, 81.0)
- added R21: 1k, Resistor_SMD:R_0805_2012Metric_Pad1.15x1.40mm_HandSolder, F.Cu at (70.0, 87.0)
- added R22: 1, Resistor_SMD:R_0805_2012Metric_Pad1.15x1.40mm_HandSolder, F.Cu at (66.0, 87.0)
- added R23: 100k, Resistor_SMD:R_1206_3216Metric_Pad1.42x1.75mm_HandSolder, F.Cu at (139.0, 19.0)
- added R24: 100k, Resistor_SMD:R_1206_3216Metric_Pad1.42x1.75mm_HandSolder, F.Cu at (139.0, 29.0)
- added R25: 100k, Resistor_SMD:R_1206_3216Metric_Pad1.42x1.75mm_HandSolder, F.Cu at (139.0, 38.0)
- added R26: 100k, Resistor_SMD:R_1206_3216Metric_Pad1.42x1.75mm_HandSolder, F.Cu at (139.0, 46.5)
- added R27: 100k, Resistor_SMD:R_1206_3216Metric_Pad1.42x1.75mm_HandSolder, F.Cu at (139.0, 55.5)
- added R28: 1k, Resistor_SMD:R_1206_3216Metric_Pad1.42x1.75mm_HandSolder, F.Cu at (133.0, 50.5)
- added R29: 1M, Resistor_SMD:R_0805_2012Metric_Pad1.15x1.40mm_HandSolder, F.Cu at (54.0, 6.00)
- added R30: 37.4k, Resistor_SMD:R_0805_2012Metric_Pad1.15x1.40mm_HandSolder, F.Cu at (49.0, 6.00)
- added R31: 49.9k, Resistor_SMD:R_0805_2012Metric_Pad1.15x1.40mm_HandSolder, F.Cu at (47.0, 10.0)
- added R32: 50k, Resistor_SMD:R_0805_2012Metric_Pad1.15x1.40mm_HandSolder, F.Cu at (39.0, 10.0)
- added R33: 10k, Resistor_SMD:R_0805_2012Metric_Pad1.15x1.40mm_HandSolder, F.Cu at (229.0, 90.0)
- added R34: 10k, Resistor_SMD:R_0805_2012Metric_Pad1.15x1.40mm_HandSolder, F.Cu at (233.0, 101.0)
- added R35: 1, Resistor_SMD:R_0805_2012Metric_Pad1.15x1.40mm_HandSolder, F.Cu at (228.0, 107.0)
- added R36: 0.01, Resistor_SMD:R_0603_1608Metric_Pad1.05x0.95mm_HandSolder, F.Cu at (208.0, 99.0)
- added R37: 0.01, Resistor_SMD:R_0805_2012Metric_Pad1.15x1.40mm_HandSolder, F.Cu at (108.0, 100.0)
- added R38: 1M, Resistor_THT:R_Axial_DIN0309_L9.0mm_D3.2mm_P15.24mm_Horizontal, F.Cu at (117.0, 86.0)
- added R39: 70K, Resistor_SMD:R_1206_3216Metric_Pad1.42x1.75mm_HandSolder, F.Cu at (60.5, 16.0)
- added R40: 470, Resistor_SMD:R_0805_2012Metric_Pad1.15x1.40mm_HandSolder, F.Cu at (44.0, 21.0)
- added R41: 100k, Resistor_SMD:R_0805_2012Metric_Pad1.15x1.40mm_HandSolder, F.Cu at (113.0, 95.0)
- added R42: 1k, Resistor_SMD:R_0805_2012Metric_Pad1.15x1.40mm_HandSolder, F.Cu at (108.0, 95.0)
- added R43: 10k, Resistor_SMD:R_0805_2012Metric_Pad1.15x1.40mm_HandSolder, F.Cu at (210.5, 75.0)
- added R44: 39k, Resistor_SMD:R_0805_2012Metric_Pad1.15x1.40mm_HandSolder, F.Cu at (210.5, 70.0)
- added R45: 100k, Resistor_SMD:R_0805_2012Metric_Pad1.15x1.40mm_HandSolder, F.Cu at (202.0, 12.0)
- added R46: 240k, Resistor_SMD:R_0805_2012Metric_Pad1.15x1.40mm_HandSolder, F.Cu at (213.8, 7.80)
- added R47: 249k, Resistor_SMD:R_0805_2012Metric_Pad1.15x1.40mm_HandSolder, F.Cu at (196.6, 42.7)
- added R48: 15.4k, Resistor_SMD:R_0805_2012Metric_Pad1.15x1.40mm_HandSolder, F.Cu at (200.0, 50.5)
- added R49: 147k, Resistor_SMD:R_0805_2012Metric_Pad1.15x1.40mm_HandSolder, F.Cu at (210.1, 47.3)
- added R50: 10.5k, Resistor_SMD:R_0805_2012Metric_Pad1.15x1.40mm_HandSolder, F.Cu at (205.0, 47.3)
- added R7: 10k, Resistor_SMD:R_0805_2012Metric_Pad1.15x1.40mm_HandSolder, F.Cu at (80.0, 44.0)
- added R8: 10k, Resistor_SMD:R_0805_2012Metric_Pad1.15x1.40mm_HandSolder, F.Cu at (80.0, 47.0)
- added R9: 10k, Resistor_SMD:R_0805_2012Metric_Pad1.15x1.40mm_HandSolder, F.Cu at (72.0, 37.0)
- added RV1: 1k, Potentiometer_THT:Potentiometer_Bourns_3339P_Vertical_HandSoldering, F.Cu at (51.0, 21.0)
- added T1: CST1, Transformer_SMD:Transformer_Coilcraft_CST1, F.Cu at (175.0, 73.0)
- added U10: MIC4427, Package_SO:SOIC-8_3.9x4.9mm_P1.27mm, F.Cu at (166.0, 44.0)
- added U11: 24LC08, Package_SO:SOIC-8_3.9x4.9mm_P1.27mm, F.Cu at (-7.92, 83.3)
- added U12: LM1117-3.3, Package_TO_SOT_SMD:TO-252-2, F.Cu at (-7.42, 6.23)
- added U13: MCP1416, Package_TO_SOT_SMD:SOT-23-5, F.Cu at (229.0, 101.0)
- added U14: LT3758AEMSE, Package_SO:MSOP-10-1EP_3x3mm_P0.5mm_EP1.68x1.88mm, F.Cu at (53.0, 10.0)
- added U15: LM1117-ADJ, Package_TO_SOT_SMD:TO-252-2, F.Cu at (220.4, 73.0)
- added U16: LTC7149FE, Package_SO:HTSSOP-28-1EP_4.4x9.7mm_P0.65mm_EP2.85x5.4mm, F.Cu at (204.0, 3.80)
- added U17: TPS54360DDA, Package_SO:TI_SO-PowerPAD-8_ThermalVias, F.Cu at (203.4, 41.9)
- added U6: IRS2005S, Package_SO:SOIC-8_3.9x4.9mm_P1.27mm, F.Cu at (115.2, 30.0)
- added U7: LTC6090, Package_SO:SOIC-8-1EP_3.9x4.9mm_P1.27mm_EP2.29x3mm, F.Cu at (73.0, 51.0)
- added U8: INA181, Package_TO_SOT_SMD:SOT-23-6, F.Cu at (174.6, 60.0)
- added U9: MIC4427, Package_SO:SOIC-8_3.9x4.9mm_P1.27mm, F.Cu at (166.0, 25.0)
- C1, C10, C19, C2, C3, C30, C35, C36, C37, C38, C39, C4, C40, C41, C42, C5, C9: footprint Capacitor_SMD:C_0603_1608Metric_Pad1.05x0.95mm_HandSolder -> Capacitor_SMD:C_0805_2012Metric_Pad1.15x1.40mm_HandSolder
- C11: value 2uF -> 0.033uF
- C12: value 0.1uF -> 0.01uF; footprint Capacitor_SMD:C_0603_1608Metric_Pad1.05x0.95mm_HandSolder -> Capacitor_SMD:C_0805_2012Metric_Pad1.15x1.40mm_HandSolder
- C13: value 0.1uF -> 0.015uF; footprint Capacitor_SMD:C_0603_1608Metric_Pad1.05x0.95mm_HandSolder -> Capacitor_SMD:C_1210_3225Metric_Pad1.42x2.65mm_HandSolder
- C14: value 0.1uF -> 0.033uF; footprint Capacitor_SMD:C_0603_1608Metric_Pad1.05x0.95mm_HandSolder -> Capacitor_SMD:C_1210_3225Metric_Pad1.42x2.65mm_HandSolder
- C15: value 4.7uF -> 0.068uF
- C16: value 4.7uF -> 0.12uF
- C17: renamed from C43; footprint Capacitor_SMD:C_0603_1608Metric_Pad1.05x0.95mm_HandSolder -> Capacitor_SMD:C_0805_2012Metric_Pad1.15x1.40mm_HandSolder
- C18: value 47uF -> 4.7uF; footprint Capacitor_THT:CP_Radial_D10.0mm_P5.00mm -> Capacitor_SMD:C_1210_3225Metric_Pad1.42x2.65mm_HandSolder
- C20: value 0.1uF -> 10nF; footprint Capacitor_SMD:C_0603_1608Metric_Pad1.05x0.95mm_HandSolder -> Capacitor_SMD:C_0805_2012Metric_Pad1.15x1.40mm_HandSolder
- C21: value 0.1uF -> 100pF; footprint Capacitor_SMD:C_0603_1608Metric_Pad1.05x0.95mm_HandSolder -> Capacitor_SMD:C_0805_2012Metric_Pad1.15x1.40mm_HandSolder
- C22, C25: value 0.1uF -> 10uF; footprint Capacitor_SMD:C_0603_1608Metric_Pad1.05x0.95mm_HandSolder -> Capacitor_SMD:C_1210_3225Metric_Pad1.42x2.65mm_HandSolder
- C23: value 2uF -> 4.7uF; footprint Capacitor_SMD:C_1210_3225Metric_Pad1.42x2.65mm_HandSolder -> Capacitor_SMD:C_0805_2012Metric_Pad1.15x1.40mm_HandSolder
- C24: value 2uF -> 0.0073uF
- C26: value 0.1uF -> 4.7uF; footprint Capacitor_SMD:C_0603_1608Metric_Pad1.05x0.95mm_HandSolder -> Capacitor_SMD:C_1210_3225Metric_Pad1.42x2.65mm_HandSolder
- C27: value 0.1uF -> 22uF; footprint Capacitor_SMD:C_0603_1608Metric_Pad1.05x0.95mm_HandSolder -> Capacitor_SMD:C_0805_2012Metric_Pad1.15x1.40mm_HandSolder
- C29: value 0.1uF -> 2.2uF; footprint Capacitor_SMD:C_0603_1608Metric_Pad1.05x0.95mm_HandSolder -> Capacitor_SMD:C_0805_2012Metric_Pad1.15x1.40mm_HandSolder
- C31: value 4.7uF -> 0.01uF; footprint Capacitor_SMD:C_1210_3225Metric_Pad1.42x2.65mm_HandSolder -> Capacitor_SMD:C_0805_2012Metric_Pad1.15x1.40mm_HandSolder
- C33: value 4.7uF -> 2.2uF; footprint Capacitor_SMD:C_1210_3225Metric_Pad1.42x2.65mm_HandSolder -> Capacitor_SMD:C_0805_2012Metric_Pad1.15x1.40mm_HandSolder
- C34: value 4.7uF -> 10uF; footprint Capacitor_SMD:C_1210_3225Metric_Pad1.42x2.65mm_HandSolder -> Capacitor_SMD:C_0805_2012Metric_Pad1.15x1.40mm_HandSolder
- C6: value 0.01uF -> 0.0073uF; footprint Capacitor_SMD:C_1210_3225Metric_Pad1.42x2.65mm_HandSolder -> Capacitor_THT:C_Rect_L18.0mm_W6.0mm_P15.00mm_FKS3_FKP3
- C7, C8: value 4.7uF -> 0.1uF; footprint Capacitor_SMD:C_1210_3225Metric_Pad1.42x2.65mm_HandSolder -> Capacitor_SMD:C_0805_2012Metric_Pad1.15x1.40mm_HandSolder
- J1, J2, J3: footprint Connector_Wire:SolderWirePad_1x02_P7.62mm_Drill2mm -> Connector_Phoenix_MSTB:PhoenixContact_MSTBVA_2,5_2-G_1x02_P5.00mm_Vertical
- J5: value Conn_01x02_Male -> DB15_Female_HighDensity; footprint Connector_Wire:SolderWirePad_1x02_P7.62mm_Drill2mm -> Connector_Dsub:DSUB-15-HD_Female_Horizontal_P2.29x1.98mm_EdgePinOffset3.03mm_Housed_MountingHolesOffset4.94mm
- Q1, Q3: value LMG5200 -> BSC082N10LSG; footprint Package_DFN_QFN:Texas_MOF0009A -> Package_TO_SOT_SMD:TDSON-8-1
- Q4: value LMG5200 -> BCP56; footprint Package_DFN_QFN:Texas_MOF0009A -> Package_TO_SOT_SMD:SOT-223-3_TabPin2
- Q5: value LMG5200 -> BCP53; footprint Package_DFN_QFN:Texas_MOF0009A -> Package_TO_SOT_SMD:SOT-223-3_TabPin2
- R1, R3, R5: value 1M -> 10k; footprint Capacitor_SMD:C_0603_1608Metric_Pad1.05x0.95mm_HandSolder -> Resistor_SMD:R_0805_2012Metric_Pad1.15x1.40mm_HandSolder
- R2: value 2 -> 1; footprint Resistor_SMD:R_MELF_MMB-0207 -> Resistor_SMD:R_0805_2012Metric_Pad1.15x1.40mm_HandSolder
- U5: value AMS1117-5.0 -> TL082; footprint Package_TO_SOT_SMD:SOT-223-3_TabPin2 -> Package_SO:SOIC-8_3.9x4.9mm_P1.27mm
- moved J5 185.8 mm to (-16.0, 91.0), turned to -90 degrees
- moved C17 184.0 mm to (-16.2, 6.25), turned to 90 degrees
- moved C40 158.3 mm to (10.6, 7.23)
- moved C42 158.3 mm to (2.83, 7.23)
- moved U4 158.3 mm to (6.58, 7.36)
- moved C19 145.3 mm to (229.0, 95.0), turned to 0 degrees
- moved C30 143.6 mm to (210.6, 3.60), turned to -90 degrees
- moved C33 136.4 mm to (207.0, 12.0)
- moved C34 134.8 mm to (197.2, 5.00), turned to -90 degrees
- moved C29 133.0 mm to (207.0, 16.0)
- moved C18 126.9 mm to (49.6, 1.40), turned to 180 degrees
- moved C31 126.9 mm to (210.6, 7.80), turned to -90 degrees
- moved C26 124.1 mm to (210.7, 43.1), turned to 90 degrees
- moved C35 118.8 mm to (-0.50, 30.0)
- moved C36 118.8 mm to (4.00, 29.0)
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Connections:
- net Net-(U2-Pad22) renamed HSYNC_UC
- net Net-(U2-Pad23) renamed VSYNC_UC
- C1 pad 1: +5V -> +12V
- C1 pad 2: GND -> -12V
- C10 pad 1: Net-(C10-Pad1) -> +12V
- C10 pad 2: Net-(C10-Pad2) -> GND
- C11 pad 1: /h.return -> Net-(C11-Pad1)
- C12 pad 1: HT -> /v.out
- C12 pad 2: GND -> Net-(C12-Pad2)
- C13 pad 1: HT -> Net-(C11-Pad1)
- C13 pad 2: GND -> Net-(C13-Pad2)
- C14 pad 1: HT -> Net-(C11-Pad1)
- C14 pad 2: GND -> Net-(C14-Pad2)
- C15 pad 1: HT -> Net-(C11-Pad1)
- C15 pad 2: GND -> Net-(C15-Pad2)
- C16 pad 1: HT -> Net-(C11-Pad1)
- C16 pad 2: GND -> Net-(C16-Pad2)
- C17 pad 2: Net-(C43-Pad2) -> Net-(C17-Pad2)
- C18 pad 1: HT -> +48V
- C19 pad 1: +5V -> +12V
- C2 pad 1: Net-(C2-Pad1) -> +12V
- C2 pad 2: Net-(C2-Pad2) -> GND
- C20 pad 1: +5V -> Net-(C20-Pad1)
- C21 pad 2: Net-(C21-Pad2) -> GND
- C22 pad 2: Net-(C22-Pad2) -> GND
- C24 pad 1: Net-(C24-Pad1) -> /power_supply/eht out
- C27 pad 1: HT -> Net-(C27-Pad1)
- C29 pad 1: HT -> Net-(C29-Pad1)
- C3 pad 1: HT -> +12V
- C30 pad 1: HT -> Net-(C30-Pad1)
- C30 pad 2: GND -> Net-(C30-Pad2)
- C31 pad 1: HT -> Net-(C31-Pad1)
- C31 pad 2: GND -> -12V
- C33 pad 1: HT -> Net-(C29-Pad1)
- C34 pad 1: HT -> +48V
- C4 pad 1: HT -> Net-(C4-Pad1)
- C4 pad 2: GND -> /hsupply
- C5 pad 1: HT -> +48V
- C7 pad 1: HT -> -12V
- C8 pad 1: HT -> +3V3
- C9 pad 1: +5V -> +12V
- J1 pad 1: /h.return -> /h.ret
- J3 pad 1: Net-(C24-Pad1) -> /v.ret
- J3 pad 2: Net-(C23-Pad1) -> /v.out
- J5 pad 1: +12V -> /Sheet5C37BEF6/red
- J5 pad 2: GND -> /Sheet5C37BEF6/green
- L1 pad 1: Net-(L1-Pad1) -> /hsupply
- Q1 pad 1: HT -> /hsupply
- Q1 pad 2: Net-(C2-Pad1) -> /hsupply
- Q1 pad 3: Net-(C2-Pad2) -> /hsupply
- Q1 pad 4: B_HI -> Net-(Q13-Pad4)_2
- Q1 pad 5: B_LI -> HT
- Q3 pad 1: HT -> GND
- Q3 pad 2: Net-(C10-Pad1) -> GND
- Q3 pad 3: Net-(C10-Pad2) -> GND
- Q3 pad 4: S_HI -> Net-(Q13-Pad4)
- Q3 pad 5: S_LI -> /hsupply
- Q4 pad 1: HT -> Net-(Q4-Pad1)
- Q4 pad 2: Net-(C21-Pad1) -> +48V
- Q4 pad 3: Net-(C21-Pad2) -> Net-(Q4-Pad3)
- Q5 pad 1: HT -> Net-(Q4-Pad1)
- Q5 pad 2: Net-(C22-Pad1) -> Net-(Q5-Pad2)
- Q5 pad 3: Net-(C22-Pad2) -> -12V
- R1 pad 1: Net-(C23-Pad1) -> +3V3
- R1 pad 2: GND -> Net-(R1-Pad2)
- R3 pad 1: Net-(C24-Pad1) -> Net-(R1-Pad2)
- R5 pad 1: /h.return -> HOT_IN
- U2 pad 21: B_LI -> Net-(U2-Pad21)
- U2 pad 34: S_LI -> Net-(U2-Pad34)
- U2 pad 37: B_HI -> Net-(U2-Pad37)
- U2 pad 41: S_HI -> Net-(U2-Pad41)
- U2 pad 42: Net-(U2-Pad42) -> /Sheet5C37BEF6/tx
- U2 pad 43: Net-(U2-Pad43) -> /Sheet5C37BEF6/rx
- U2 pad 61: Net-(U2-Pad61) -> HOT_IN
- U5 pad 1: Net-(C43-Pad2) -> Net-(R9-Pad2)
- U5 pad 2: +5V -> Net-(R9-Pad2)
- U5 pad 3: +12V -> Net-(R1-Pad2)
Other:
- board text added: "+12V"
- board text added: "-12V"
- board text added: "B+ Supply"
- board text added: "EHT"
- board text added: "Heater"
- board text added: "Horizontal"
- board text added: "Vertical"

Commit message: more stuff
Parts:
- added C28: 22uF, Capacitor_THT:CP_Radial_D8.0mm_P3.50mm, F.Cu at (72.0, 35.0)
- added C32: 100uF, Capacitor_THT:CP_Radial_D8.0mm_P3.50mm, F.Cu at (214.0, 31.0)
- added C46: 100uF, Capacitor_THT:CP_Radial_D8.0mm_P3.50mm, F.Cu at (207.5, 58.0)
- added C47: 0.1uF, Capacitor_SMD:C_0805_2012Metric_Pad1.15x1.40mm_HandSolder, F.Cu at (-7.00, 58.0)
- added C48: 47uF, Capacitor_SMD:C_1206_3216Metric_Pad1.42x1.75mm_HandSolder, F.Cu at (-7.49, 73.0)
- added C49: 47uF, Capacitor_SMD:C_1206_3216Metric_Pad1.42x1.75mm_HandSolder, F.Cu at (-7.49, 83.0)
- added C50: 47uF, Capacitor_SMD:C_1206_3216Metric_Pad1.42x1.75mm_HandSolder, F.Cu at (-7.51, 91.0)
- added C51: 0.1uF, Capacitor_SMD:C_0805_2012Metric_Pad1.15x1.40mm_HandSolder, F.Cu at (-6.95, 22.0)
- added C52: 0.1uF, Capacitor_SMD:C_0805_2012Metric_Pad1.15x1.40mm_HandSolder, F.Cu at (-6.97, 34.0)
- added C53: 2.2uF, Capacitor_SMD:C_0805_2012Metric_Pad1.15x1.40mm_HandSolder, F.Cu at (19.0, 73.0)
- added C54: 0.1uF, Capacitor_SMD:C_0805_2012Metric_Pad1.15x1.40mm_HandSolder, F.Cu at (-6.97, 46.0)
- added C55: 2.2uF, Capacitor_SMD:C_0805_2012Metric_Pad1.15x1.40mm_HandSolder, F.Cu at (19.0, 83.0)
- added C56: 2.2uF, Capacitor_SMD:C_0805_2012Metric_Pad1.15x1.40mm_HandSolder, F.Cu at (19.0, 93.0)
- added C57: 1uF, Capacitor_SMD:C_0805_2012Metric_Pad1.15x1.40mm_HandSolder, F.Cu at (-23.1, 79.2)
- added C58: 0.1uF, Capacitor_SMD:C_0805_2012Metric_Pad1.15x1.40mm_HandSolder, F.Cu at (-23.0, 92.0)
- added H1: MountingHole_Pad, MountingHole:MountingHole_3.2mm_M3_Pad_Via, F.Cu at (-34.0, 106.0)
- added H2: MountingHole_Pad, MountingHole:MountingHole_3.2mm_M3_Pad_Via, F.Cu at (-34.0, 6.00)
- added H3: MountingHole_Pad, MountingHole:MountingHole_3.2mm_M3_Pad_Via, F.Cu at (241.0, 6.00)
- added H4: MountingHole_Pad, MountingHole:MountingHole_3.2mm_M3_Pad_Via, F.Cu at (241.0, 106.0)
- added J7: Conn_01x08_Male, Connector_Phoenix_MC:PhoenixContact_MCV_1,5_8-G-3.5_1x08_P3.50mm_Vertical, F.Cu at (45.0, 97.0)
- added L3: 33uH, Inductor_SMD:L_Bourns_SRR1260, F.Cu at (77.0, 20.0)
- added L4: 7.8uH, Inductor_SMD:L_Bourns_SRR1260, F.Cu at (215.0, 18.0)
- added L5: 100uH, Inductor_SMD:L_Bourns_SRR1260, F.Cu at (214.2, 46.0)
- added Q14: BC847, Package_TO_SOT_SMD:SOT-23, F.Cu at (31.0, 74.0)
- added Q15: BC847, Package_TO_SOT_SMD:SOT-23, F.Cu at (31.0, 80.0)
- added Q16: BC847, Package_TO_SOT_SMD:SOT-23, F.Cu at (31.0, 86.0)
- added R51: 5.5k, Resistor_SMD:R_0805_2012Metric_Pad1.15x1.40mm_HandSolder, F.Cu at (-27.0, 24.0)
- added R52: 2.7k, Resistor_SMD:R_0805_2012Metric_Pad1.15x1.40mm_HandSolder, F.Cu at (-27.0, 19.0)
- added R53: 5.5k, Resistor_SMD:R_0805_2012Metric_Pad1.15x1.40mm_HandSolder, F.Cu at (-27.0, 60.0)
- added R54: 2.7k, Resistor_SMD:R_0805_2012Metric_Pad1.15x1.40mm_HandSolder, F.Cu at (-27.0, 55.0)
- added R55: 1, Resistor_SMD:R_0805_2012Metric_Pad1.15x1.40mm_HandSolder, F.Cu at (-13.0, 73.0)
- added R56: 1, Resistor_SMD:R_0805_2012Metric_Pad1.15x1.40mm_HandSolder, F.Cu at (-13.0, 83.0)
- added R57: 1, Resistor_SMD:R_0805_2012Metric_Pad1.15x1.40mm_HandSolder, F.Cu at (-13.0, 91.0)
- added R58: 5.5k, Resistor_SMD:R_0805_2012Metric_Pad1.15x1.40mm_HandSolder, F.Cu at (-27.0, 36.0)
- added R59: 2.7k, Resistor_SMD:R_0805_2012Metric_Pad1.15x1.40mm_HandSolder, F.Cu at (-27.0, 31.0)
- added R60: 560, Resistor_SMD:R_0805_2012Metric_Pad1.15x1.40mm_HandSolder, F.Cu at (-13.0, 76.0)
- added R61: 5.5k, Resistor_SMD:R_0805_2012Metric_Pad1.15x1.40mm_HandSolder, F.Cu at (-27.0, 48.0)
- added R62: 2.7k, Resistor_SMD:R_0805_2012Metric_Pad1.15x1.40mm_HandSolder, F.Cu at (-27.0, 43.0)
- added R63: 1k, Resistor_SMD:R_0805_2012Metric_Pad1.15x1.40mm_HandSolder, F.Cu at (-7.00, 55.0)
- added R64: 560, Resistor_SMD:R_0805_2012Metric_Pad1.15x1.40mm_HandSolder, F.Cu at (-13.0, 86.0)
- added R65: 220, Resistor_SMD:R_0805_2012Metric_Pad1.15x1.40mm_HandSolder, F.Cu at (-8.00, 76.0)
- added R66: 220, Resistor_SMD:R_0805_2012Metric_Pad1.15x1.40mm_HandSolder, F.Cu at (-8.00, 86.0)
- added R67: 220, Resistor_SMD:R_0805_2012Metric_Pad1.15x1.40mm_HandSolder, F.Cu at (-8.03, 95.0)
- added R68: 560, Resistor_SMD:R_0805_2012Metric_Pad1.15x1.40mm_HandSolder, F.Cu at (-13.0, 94.0)
- added R69: 47k, Resistor_SMD:R_0805_2012Metric_Pad1.15x1.40mm_HandSolder, F.Cu at (19.0, 103.0)
- added R70: 1k, Resistor_SMD:R_0805_2012Metric_Pad1.15x1.40mm_HandSolder, F.Cu at (-7.00, 19.0)
- added R71: 1k, Resistor_SMD:R_0805_2012Metric_Pad1.15x1.40mm_HandSolder, F.Cu at (-6.97, 31.0)
- added R72: 1k, Resistor_SMD:R_0805_2012Metric_Pad1.15x1.40mm_HandSolder, F.Cu at (-6.97, 43.0)
- added R73: 47k, Resistor_SMD:R_0805_2012Metric_Pad1.15x1.40mm_HandSolder, F.Cu at (19.0, 76.0)
- added R74: 47k, Resistor_SMD:R_0805_2012Metric_Pad1.15x1.40mm_HandSolder, F.Cu at (19.0, 86.0)
- added R75: 47k, Resistor_SMD:R_0805_2012Metric_Pad1.15x1.40mm_HandSolder, F.Cu at (19.0, 96.0)
- added R76: 1k, Resistor_SMD:R_0805_2012Metric_Pad1.15x1.40mm_HandSolder, F.Cu at (26.0, 76.0)
- added R77: 1k, Resistor_SMD:R_0805_2012Metric_Pad1.15x1.40mm_HandSolder, F.Cu at (26.0, 82.0)
- added R78: 1k, Resistor_SMD:R_0805_2012Metric_Pad1.15x1.40mm_HandSolder, F.Cu at (26.0, 88.0)
- added R79: 47, Resistor_SMD:R_0805_2012Metric_Pad1.15x1.40mm_HandSolder, F.Cu at (26.0, 73.0)
- added R80: 47, Resistor_SMD:R_0805_2012Metric_Pad1.15x1.40mm_HandSolder, F.Cu at (26.0, 79.0)
- added R81: 47, Resistor_SMD:R_0805_2012Metric_Pad1.15x1.40mm_HandSolder, F.Cu at (26.0, 85.0)
- added R82: 220, Resistor_SMD:R_0805_2012Metric_Pad1.15x1.40mm_HandSolder, F.Cu at (37.0, 67.0)
- added R83: 470, Resistor_SMD:R_0805_2012Metric_Pad1.15x1.40mm_HandSolder, F.Cu at (37.0, 71.0)
- added R84: 470, Resistor_SMD:R_0805_2012Metric_Pad1.15x1.40mm_HandSolder, F.Cu at (37.0, 77.0)
- added R85: 470, Resistor_SMD:R_0805_2012Metric_Pad1.15x1.40mm_HandSolder, F.Cu at (37.0, 83.0)
- added R86: 47, Resistor_SMD:R_0805_2012Metric_Pad1.15x1.40mm_HandSolder, F.Cu at (37.0, 74.0)
- added R87: 47, Resistor_SMD:R_0805_2012Metric_Pad1.15x1.40mm_HandSolder, F.Cu at (37.0, 80.0)
- added R88: 47, Resistor_SMD:R_0805_2012Metric_Pad1.15x1.40mm_HandSolder, F.Cu at (37.0, 86.0)
- added R89: 10k, Resistor_SMD:R_0805_2012Metric_Pad1.15x1.40mm_HandSolder, F.Cu at (-23.1, 83.2)
- added R90: 75, Resistor_SMD:R_0805_2012Metric_Pad1.15x1.40mm_HandSolder, F.Cu at (-26.0, 100.0)
- added R91: 75, Resistor_SMD:R_0805_2012Metric_Pad1.15x1.40mm_HandSolder, F.Cu at (-26.0, 103.0)
- added R92: 75, Resistor_SMD:R_0805_2012Metric_Pad1.15x1.40mm_HandSolder, F.Cu at (-26.0, 106.0)
- added R93: 75, Resistor_SMD:R_0805_2012Metric_Pad1.15x1.40mm_HandSolder, F.Cu at (-26.0, 109.0)
- added RV2: 3.3k, Potentiometer_THT:Potentiometer_Bourns_3386P_Vertical, F.Cu at (-35.0, 24.0)
- added RV3: 3.3k, Potentiometer_THT:Potentiometer_Bourns_3386P_Vertical, F.Cu at (-35.0, 60.0)
- added RV4: 3.3k, Potentiometer_THT:Potentiometer_Bourns_3386P_Vertical, F.Cu at (-35.0, 36.0)
- added RV5: 3.3k, Potentiometer_THT:Potentiometer_Bourns_3386P_Vertical, F.Cu at (-35.0, 48.0)
- added RV6: 3.3k, Potentiometer_THT:Potentiometer_Bourns_3386P_Vertical, F.Cu at (-15.0, 60.0)
- added RV7: 3.3k, Potentiometer_THT:Potentiometer_Bourns_3386P_Vertical, F.Cu at (-15.0, 24.0)
- added RV8: 3.3k, Potentiometer_THT:Potentiometer_Bourns_3386P_Vertical, F.Cu at (-15.0, 36.0)
- added RV9: 3.3k, Potentiometer_THT:Potentiometer_Bourns_3386P_Vertical, F.Cu at (-15.0, 48.0)
- added SW1: SW_DIP_x04, Button_Switch_THT:SW_DIP_SPSTx04_Slide_9.78x12.34mm_W7.62mm_P2.54mm, F.Cu at (-21.0, 101.0)
- added U18: M51387P, td-deflect:DIP-30_600_ELL, F.Cu at (5.00, 86.0)
- added U19: LMH1980, Package_SO:VSSOP-10_3x3mm_P0.5mm, F.Cu at (-23.0, 87.2)
- Q6: value MJD44 -> BD139; footprint Package_TO_SOT_SMD:TO-252-2 -> Package_TO_SOT_THT:TO-126-3_Vertical
- Q7: value MJD45 -> BD140; footprint Package_TO_SOT_SMD:TO-252-2 -> Package_TO_SOT_THT:TO-126-3_Vertical
- moved C26 146.8 mm to (64.0, 38.5), turned to 0 degrees
- moved Q7 36.1 mm to (60.0, 107.0), turned to 0 degrees
- moved Q6 36.0 mm to (84.0, 107.0)
- moved Q4 34.5 mm to (88.0, 94.0), turned to 180 degrees
- moved Q5 34.1 mm to (62.0, 94.0)
- moved R15 33.6 mm to (88.0, 102.0), turned to 180 degrees
- moved J9 33.5 mm to (229.0, 71.0)
- moved R16 30.8 mm to (64.0, 101.0), turned to 0 degrees
- moved C12 30.1 mm to (86.0, 76.0), turned to 0 degrees
- moved R17 27.5 mm to (74.0, 106.0), turned to 90 degrees
- moved R22 22.5 mm to (78.0, 106.0), turned to -90 degrees
- moved C17 21.5 mm to (2.77, 16.3)
- moved C35 21.5 mm to (18.5, 40.0)
- moved C36 21.5 mm to (23.0, 39.0)
- moved C37 21.5 mm to (10.8, 24.5)
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Connections:
- net /Sheet5C37BEF6/vsync renamed /rgb/vsync_vga
- J5 pad 1: /Sheet5C37BEF6/red -> /rgb/red_vga
- J5 pad 13: /Sheet5C37BEF6/hsync -> /rgb/hsync_vga
- J5 pad 2: /Sheet5C37BEF6/green -> /rgb/green_vga
- J5 pad 3: /Sheet5C37BEF6/blue -> /rgb/blue_vga
- Q6 pad 1: Net-(Q4-Pad3) -> Net-(Q6-Pad1)
- Q6 pad 3: Net-(Q6-Pad3) -> Net-(Q4-Pad3)
- Q7 pad 1: Net-(Q5-Pad2) -> -12V
- Q7 pad 3: -12V -> Net-(Q5-Pad2)
- R15 pad 2: Net-(Q6-Pad3) -> Net-(Q6-Pad1)
- R17 pad 1: Net-(Q6-Pad3) -> Net-(Q6-Pad1)

Commit message: asdf
Parts:
- removed J1: Conn_01x02_Male, Connector_Phoenix_MSTB:PhoenixContact_MSTBVA_2,5_2-G_1x02_P5.00mm_Vertical
- added C59: 0.1uF, Capacitor_SMD:C_0805_2012Metric_Pad1.15x1.40mm_HandSolder, F.Cu at (-8.03, 101.0)
- added C60: 220uF, Capacitor_THT:CP_Radial_D8.0mm_P3.50mm, F.Cu at (34.0, 96.0)
- added C61: 0.033uF, Capacitor_SMD:C_1206_3216Metric_Pad1.42x1.75mm_HandSolder, F.Cu at (219.7, 86.6)
- added D6: BAT54S, Package_TO_SOT_SMD:SOT-23, F.Cu at (42.0, 70.5)
- added D7: BAT54S, Package_TO_SOT_SMD:SOT-23, F.Cu at (42.0, 76.0)
- added D8: BAT54S, Package_TO_SOT_SMD:SOT-23, F.Cu at (42.0, 81.5)
- added F1: Fuse, Fuse:Fuse_Schurter_UMT250, F.Cu at (74.0, 99.8)
- added F2: Fuse, Fuse:Fuse_Schurter_UMT250, F.Cu at (141.2, 62.8)
- added J12: Conn_01x06_Male, td-deflect:sony_monitor_yoke, F.Cu at (95.5, 51.0)
- added J15: Conn_01x02_Male, td-deflect:sony_monitor_2p, F.Cu at (219.0, 74.0)
- added J16: Conn_01x06_Male, Connector_JST:JST_EH_B6B-EH-A_1x06_P2.50mm_Vertical, F.Cu at (-3.00, 108.0)
- added J17: Conn_01x06_Male, Connector_JST:JST_XH_B6B-XH-A_1x06_P2.50mm_Vertical, F.Cu at (49.0, 71.0)
- added J18: Conn_01x02_Male, Connector_Phoenix_MSTB:PhoenixContact_MSTBVA_2,5_2-G_1x02_P5.00mm_Vertical, F.Cu at (229.0, 18.0)
- added L2: LTRIM, td-deflect:LIN-3509, F.Cu at (121.8, 58.4)
- added L6: 1mH, Inductor_THT:L_Toroid_Vertical_L31.8mm_W15.9mm_P13.50mm_Bourns_5700, F.Cu at (164.2, 68.5)
- added R94: 33k, Resistor_SMD:R_0805_2012Metric_Pad1.15x1.40mm_HandSolder, F.Cu at (-25.0, 65.0)
- added R95: 220, Resistor_SMD:R_0805_2012Metric_Pad1.15x1.40mm_HandSolder, F.Cu at (-19.0, 65.0)
- added R96: 1, Resistor_SMD:R_0805_2012Metric_Pad1.15x1.40mm_HandSolder, F.Cu at (25.0, 13.0)
- added R97: 1, Resistor_SMD:R_0805_2012Metric_Pad1.15x1.40mm_HandSolder, F.Cu at (212.0, 66.0)
- added REF**: OSHW-Logo_5.7x6mm_SilkScreen, Symbol:OSHW-Logo_5.7x6mm_SilkScreen, F.Cu at (4.50, 8.00)
- added RV10: 10k, Potentiometer_THT:Potentiometer_Bourns_3386P_Vertical, F.Cu at (36.0, 58.0)
- added U20: 74LVC1GU04DRL, Package_TO_SOT_SMD:SOT-553, F.Cu at (-17.8, 93.8)
- C11, C13, C14, C15, C16, C22: footprint Capacitor_SMD:C_1210_3225Metric_Pad1.42x2.65mm_HandSolder -> Capacitor_SMD:C_1206_3216Metric_Pad1.42x1.75mm_HandSolder
- C20: value 10nF -> 0.01uF
- C24: footprint Capacitor_SMD:C_1210_3225Metric_Pad1.42x2.65mm_HandSolder -> Capacitor_THT:C_Rect_L18.0mm_W6.0mm_P15.00mm_FKS3_FKP3
- C25: footprint Capacitor_SMD:C_1210_3225Metric_Pad1.42x2.65mm_HandSolder -> Capacitor_THT:CP_Radial_D8.0mm_P3.50mm
- C26: value 4.7uF -> 0.1uF; footprint Capacitor_SMD:C_1210_3225Metric_Pad1.42x2.65mm_HandSolder -> Capacitor_SMD:C_1206_3216Metric_Pad1.42x1.75mm_HandSolder
- C27: footprint Capacitor_SMD:C_0805_2012Metric_Pad1.15x1.40mm_HandSolder -> Capacitor_SMD:C_1206_3216Metric_Pad1.42x1.75mm_HandSolder
- C34: footprint Capacitor_SMD:C_0805_2012Metric_Pad1.15x1.40mm_HandSolder -> Capacitor_THT:CP_Radial_D8.0mm_P3.50mm
- C40: value 4.7uF -> 22uF; footprint Capacitor_SMD:C_0805_2012Metric_Pad1.15x1.40mm_HandSolder -> Capacitor_SMD:C_1206_3216Metric_Pad1.42x1.75mm_HandSolder
- E1, E2: footprint Capacitor_SMD:C_1825_4564Metric_Pad1.88x6.70mm_HandSolder -> Resistor_THT:R_Axial_DIN0309_L9.0mm_D3.2mm_P12.70mm_Horizontal
- J10: footprint Connector_Phoenix_MSTB:PhoenixContact_MSTBVA_2,5_2-G_1x02_P5.00mm_Vertical -> td-deflect:monitor_10_8_2p
- J11: footprint Connector_Phoenix_MSTB:PhoenixContact_MSTBVA_2,5_2-G_1x02_P5.00mm_Vertical -> td-deflect:sony_monitor_2p
- J7: footprint Connector_Phoenix_MC:PhoenixContact_MCV_1,5_8-G-3.5_1x08_P3.50mm_Vertical -> Connector_JST:JST_PH_B8B-PH-K_1x08_P2.00mm_Vertical
- R32: value 50k -> 49.9k
- R36, R4: footprint Resistor_SMD:R_0603_1608Metric_Pad1.05x0.95mm_HandSolder -> Resistor_SMD:R_1206_3216Metric_Pad1.42x1.75mm_HandSolder
- R41: value 100k -> 1M; footprint Resistor_SMD:R_0805_2012Metric_Pad1.15x1.40mm_HandSolder -> Resistor_THT:R_Axial_DIN0309_L9.0mm_D3.2mm_P15.24mm_Horizontal
- R51, R58, R61: value 5.5k -> 6.8k
- R53: value 5.5k -> 0
- R54: value 2.7k -> 2.2k
- R55, R56, R57: value 1 -> 1.5k
- R6: footprint Capacitor_SMD:C_0603_1608Metric_Pad1.05x0.95mm_HandSolder -> Resistor_SMD:R_0805_2012Metric_Pad1.15x1.40mm_HandSolder
- R63: value 1k -> 0
- RV2, RV4, RV5: value 3.3k -> 2.7k
- RV3: value 3.3k -> 2k
- RV6, RV7, RV8, RV9: value 3.3k -> 1k
- moved C8 150.2 mm to (24.8, 53.9), turned to 180 degrees
- moved U8 149.8 mm to (24.8, 58.5), turned to 0 degrees
- moved R19 149.6 mm to (25.0, 62.5)
- moved U3 113.3 mm to (17.6, 57.0), turned to 0 degrees
- moved R42 102.9 mm to (210.6, 86.6), turned to 90 degrees
- moved R37 82.7 mm to (63.6, 30.2), turned to 0 degrees
- moved R41 80.3 mm to (193.0, 88.0), turned to 0 degrees
- moved R38 76.1 mm to (193.0, 83.0)
- moved T1 74.2 mm to (108.2, 40.8), turned to 180 degrees
- moved J10 66.8 mm to (104.4, 67.0), turned to 90 degrees
- moved R12 32.7 mm to (141.2, 96.6)
- moved J6 26.0 mm to (34.0, 34.0), turned to 0 degrees
- moved C37 25.7 mm to (14.0, 50.0), turned to 180 degrees
- moved C6 22.9 mm to (148.6, 96.6)
- moved C2 22.2 mm to (167.8, 101.8), turned to -90 degrees
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Connections:
- net Net-(C11-Pad1) renamed /S_cap_top
- net Net-(J7-Pad4) renamed /rgb/b_yoke
- net Net-(J7-Pad6) renamed /rgb/g_yoke
- net Net-(J7-Pad8) renamed /rgb/r_yoke
- C12 pad 1: /v.out -> Net-(C12-Pad1)
- C17 pad 2: Net-(C17-Pad2) -> GND
- C40 pad 1: +5V -> Net-(C40-Pad1)
- J2 pad 1: HT -> GND
- J2 pad 2: GND -> HT
- J5 pad 14: /rgb/vsync_vga -> VSYNC_VGA_UC
- J7 pad 1: Net-(J7-Pad1) -> +12V
- J8 pad 1: HT -> Net-(C61-Pad1)
- J9 pad 2: Net-(C27-Pad1) -> Net-(J15-Pad2)
- R14 pad 2: /v.out -> Net-(C12-Pad1)
- R17 pad 2: /v.out -> Net-(C12-Pad1)
- R18 pad 1: /v.out -> Net-(C12-Pad1)
- R43 pad 1: Net-(C27-Pad1) -> Net-(J15-Pad2)
- R9 pad 2: Net-(R9-Pad2) -> /virtual_ground
- RV3 pad 2: Net-(RV3-Pad2) -> Net-(R94-Pad2)
- U12 pad 1: Net-(C17-Pad2) -> GND
- U15 pad 2: Net-(C27-Pad1) -> Net-(J15-Pad2)
- U16 pad 29: (no net) -> -12V
- U18 pad 14: Net-(RV3-Pad2) -> Net-(C59-Pad1)
- U18 pad 15: /rgb/backporch -> Net-(U18-Pad15)
- U19 pad 10: /rgb/oddeven -> ODDEVEN_UC
- U19 pad 6: /rgb/hsync -> HSYNC_UC
- U19 pad 7: /rgb/vsync -> VSYNC_UC
- U2 pad 10: Net-(U2-Pad10) -> S2
- U2 pad 11: Net-(U2-Pad11) -> S3
- U2 pad 14: Net-(U2-Pad14) -> H_CURRENT
- U2 pad 15: Net-(U2-Pad15) -> /Sheet5C37BEF6/hot_current_adc
- U2 pad 16: Net-(U2-Pad16) -> S_VOLTAGE
- U2 pad 17: Net-(U2-Pad17) -> EHT_FLYBACK_VOLTAGE
- U2 pad 20: Net-(U2-Pad20) -> V_DAC
- U2 pad 21: Net-(U2-Pad21) -> EHT_CURRENT
- U2 pad 25: Net-(U2-Pad25) -> VSYNC_VGA_UC
- U2 pad 3: Net-(U2-Pad3) -> uc_blank
- U2 pad 34: Net-(U2-Pad34) -> PIN_LO
- U2 pad 4: Net-(U2-Pad4) -> ODDEVEN_UC
- U2 pad 41: Net-(U2-Pad41) -> PIN_HI
- U2 pad 58: Net-(U2-Pad58) -> EHT_PWM
- U2 pad 8: Net-(U2-Pad8) -> S0
- U2 pad 9: Net-(U2-Pad9) -> S1
- U5 pad 1: Net-(R9-Pad2) -> /virtual_ground
- U5 pad 2: Net-(R9-Pad2) -> /virtual_ground
- U8 pad 5: +1V5 -> /virtual_ground
Routing:
- net +12V: track 0.00 -> 684.2 mm, vias 0 -> 7
- net +48V: track 0.00 -> 371.0 mm, vias 0 -> 4
- net -12V: track 0.00 -> 336.3 mm, vias 0 -> 7
- net EHT_CURRENT: track 0.00 -> 302.2 mm, vias 0 -> 1
- net EHT_FLYBACK_VOLTAGE: track 0.00 -> 267.2 mm, vias 0 -> 1
- net EHT_PWM: track 0.00 -> 260.4 mm, vias 0 -> 2
- net +3V3: track 0.00 -> 257.1 mm, vias 0 -> 8
- net S3: track 0.00 -> 180.6 mm, vias 0 -> 2
- net HT: track 0.00 -> 179.7 mm, vias 0 -> 1
- net S_VOLTAGE: track 0.00 -> 179.3 mm, vias 0 -> 2
- net S2: track 0.00 -> 179.2 mm, vias 0 -> 2
- net HOT_IN: track 0.00 -> 177.5 mm, vias 0 -> 2
- net S1: track 0.00 -> 171.7 mm, vias 0 -> 2
- net S0: track 0.00 -> 170.3 mm, vias 0 -> 2
- net Net-(R19-Pad2): track 0.00 -> 139.6 mm, vias 0 -> 4
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- added copper zone on B.Cu, net GND
- added copper zone on F.Cu, net GND
Other:
- board outline added: 275 x 110 mm
- net class 1700V: clearance 3 -> 2.5
- net class 200V added: clearance 0.4, trace_width 0.25, via_dia 0.8, via_drill 0.4
- net class 80V removed
- net class Default: clearance 0.2 -> 0.16; trace_width 0.25 -> 0.16; via_dia 0.8 -> 0.6; via_drill 0.4 -> 0.3
- rule pad_to_mask_clearance: 0.051 -> 0
- rule trace_clearance: 0.2 -> 0.16
- rule trace_min: 0.2 -> 0.16
- rule via_min_size: 0.4 -> 0.508
- board text added: "+48V"
- board text added: "All"
- board text added: "B"
- board text added: "Bias"
- board text added: "G"
- board text added: "Gain"
- board text added: "High Voltage"
- board text added: "Neck"
- board text added: "R"
- board text added: "RGB"
- board text added: "Serial"
- board text added: "b+ adj"
- board text added: "sub contrast"
- board text added: "td-deflect v0.1 http://github.com/tdaede/td-rgb cc-by-sa 4.0"

Commit message: asdf
Parts:
- C18: value 4.7uF -> 22uF; footprint Capacitor_SMD:C_1210_3225Metric_Pad1.42x2.65mm_HandSolder -> Capacitor_THT:CP_Radial_D8.0mm_P3.50mm
- R36, R4: footprint Resistor_SMD:R_1206_3216Metric_Pad1.42x1.75mm_HandSolder -> Resistor_SMD:R_0805_2012Metric_Pad1.15x1.40mm_HandSolder
- RV1: footprint Potentiometer_THT:Potentiometer_Bourns_3339P_Vertical_HandSoldering -> Potentiometer_THT:Potentiometer_Bourns_3386P_Vertical
- T1: value CST1 -> CST1-125LC
- U4: value TPS76933 -> TPS70933
- moved C28 115.7 mm to (189.5, 39.3), turned to 180 degrees
- moved C25 54.9 mm to (99.8, 26.1), turned to -90 degrees
- moved RV1 5.10 mm to (55.0, 29.9), turned to 180 degrees
- moved C18 2.73 mm to (54.2, 12.8)
- moved R16 0.50 mm to (63.5, 101.0)
Routing:
- net HT: track 179.7 -> 158.8 mm
- net Net-(R40-Pad1): track 4.17 -> 10.1 mm
- net +48V: track 371.0 -> 375.6 mm, vias 4 -> 5
- net Net-(R19-Pad2): track 139.6 -> 141.7 mm
- net PIN_LO: track 110.4 -> 112.3 mm
- net PIN_HI: track 108.1 -> 110.1 mm
- net Net-(Q5-Pad2): track 24.7 -> 25.3 mm
- net GND: vias 110 -> 116

Commit message: asdf
Routing:
- net HT: track 158.8 -> 159.3 mm, vias 1 -> 2
- net GND: vias 116 -> 119
