File: td-deflect/td-deflect.kicad_pcb (KiCad board)
At the start: 2 copper layers, 275 x 110 mm, 247 parts, among them J10 Conn_01x02_Male, J11 Conn_01x02_Male, J12 Conn_01x06_Male, J13 Conn_01x02_Male, J14 Conn_01x02_Male, J15 Conn_01x02_Male, J16 Conn_01x06_Male, J17 Conn_01x06_Male, J18 Conn_01x02_Male, J2 Conn_01x02_Male, J3 Conn_01x02_Male, J4 Conn_ARM_JTAG_SWD_10, J5 DB15_Female_HighDensity, J6 Conn_01x06_Male, J7 Conn_01x08_Male, J8 Conn_01x02_Male, J9 Conn_01x02_Male, Q1 BSC082N10LSG, Q10 IPD50R380CE, Q11 IPD50R380CE, Q12 C2M0045170D, Q13 BSC082N10LSG, Q14 BC847, Q15 BC847, Q16 BC847, Q2 C2M0045170D, Q3 BSC082N10LSG, Q4 BCP56, Q5 BCP53, Q6 BD139, Q7 BD140, Q8 IPD50R380CE, Q9 IPD50R380CE, SW1 SW_DIP_x04, T1 CST1-125LC, U1 MCP1416, U10 MIC4427, U11 24LC08, U12 LM1117-3.3, U13 MCP1416, U14 LT3758AEMSE, U15 LM1117-ADJ, U16 LTC7149FE, U17 TPS54360DDA, U18 M51387P, U19 LMH1980, U2 STM32F722RETx, U20 74LVC1GU04DRL, U3 INA193, U4 TPS70933, U5 TL082, U6 IRS2005S, U7 LTC6090, U8 INA181, U9 MIC4427, X1 SG-8002CA

Commit message: convert deflect pcb to newer nightly
Other:
- net class 1700V removed
- net class 200V removed
- net class Default removed

Commit message: small bugfix
Parts:
- removed C19, C43, C47, C51, C52, C54: 0.1uF, Capacitor_SMD:C_0805_2012Metric_Pad1.15x1.40mm_HandSolder
- removed C24: 0.0073uF, Capacitor_THT:C_Rect_L18.0mm_W6.0mm_P15.00mm_FKS3_FKP3
- removed C27: 22uF, Capacitor_SMD:C_1206_3216Metric_Pad1.42x1.75mm_HandSolder
- removed C28: 22uF, Capacitor_THT:CP_Radial_D8.0mm_P3.50mm
- removed C29, C53, C55, C56: 2.2uF, Capacitor_SMD:C_0805_2012Metric_Pad1.15x1.40mm_HandSolder
- removed C31: 0.01uF, Capacitor_SMD:C_0805_2012Metric_Pad1.15x1.40mm_HandSolder
- removed C44: 0.033uF, Capacitor_SMD:C_0805_2012Metric_Pad1.15x1.40mm_HandSolder
- removed C45: 22pF, Capacitor_SMD:C_0805_2012Metric_Pad1.15x1.40mm_HandSolder
- removed C48, C49, C50: 47uF, Capacitor_SMD:C_1206_3216Metric_Pad1.42x1.75mm_HandSolder
- removed C60: 220uF, Capacitor_THT:CP_Radial_D8.0mm_P3.50mm
- removed C61: 0.033uF, Capacitor_SMD:C_1206_3216Metric_Pad1.42x1.75mm_HandSolder
- removed D2: C3D10170H, Package_TO_SOT_THT:TO-247-2_Vertical
- removed E1, E2: SPARK_GAP, Resistor_THT:R_Axial_DIN0309_L9.0mm_D3.2mm_P12.70mm_Horizontal
- removed J3: Conn_01x02_Male, Connector_Phoenix_MSTB:PhoenixContact_MSTBVA_2,5_2-G_1x02_P5.00mm_Vertical
- removed L4: 7.8uH, Inductor_SMD:L_Bourns_SRR1260
- removed R12, R41: 1M, Resistor_THT:R_Axial_DIN0309_L9.0mm_D3.2mm_P15.24mm_Horizontal
- removed R33, R34, R43: 10k, Resistor_SMD:R_0805_2012Metric_Pad1.15x1.40mm_HandSolder
- removed R35, R97: 1, Resistor_SMD:R_0805_2012Metric_Pad1.15x1.40mm_HandSolder
- removed R36: 0.01, Resistor_SMD:R_0805_2012Metric_Pad1.15x1.40mm_HandSolder
- removed R42, R70, R71, R72, R76, R77, R78: 1k, Resistor_SMD:R_0805_2012Metric_Pad1.15x1.40mm_HandSolder
- removed R45: 100k, Resistor_SMD:R_0805_2012Metric_Pad1.15x1.40mm_HandSolder
- removed R46: 240k, Resistor_SMD:R_0805_2012Metric_Pad1.15x1.40mm_HandSolder
- removed R47: 249k, Resistor_SMD:R_0805_2012Metric_Pad1.15x1.40mm_HandSolder
- removed R48: 15.4k, Resistor_SMD:R_0805_2012Metric_Pad1.15x1.40mm_HandSolder
- removed R49: 147k, Resistor_SMD:R_0805_2012Metric_Pad1.15x1.40mm_HandSolder
- removed R50: 10.5k, Resistor_SMD:R_0805_2012Metric_Pad1.15x1.40mm_HandSolder
- removed R51, R58, R61: 6.8k, Resistor_SMD:R_0805_2012Metric_Pad1.15x1.40mm_HandSolder
- removed R52, R59, R62: 2.7k, Resistor_SMD:R_0805_2012Metric_Pad1.15x1.40mm_HandSolder
- removed R53, R63: 0, Resistor_SMD:R_0805_2012Metric_Pad1.15x1.40mm_HandSolder
- removed R54: 2.2k, Resistor_SMD:R_0805_2012Metric_Pad1.15x1.40mm_HandSolder
- removed R55, R56, R57: 1.5k, Resistor_SMD:R_0805_2012Metric_Pad1.15x1.40mm_HandSolder
- removed R60, R64, R68: 560, Resistor_SMD:R_0805_2012Metric_Pad1.15x1.40mm_HandSolder
- removed R65, R67, R95: 220, Resistor_SMD:R_0805_2012Metric_Pad1.15x1.40mm_HandSolder
- removed R73, R74, R75: 47k, Resistor_SMD:R_0805_2012Metric_Pad1.15x1.40mm_HandSolder
- removed R79, R80, R81, R86, R87, R88: 47, Resistor_SMD:R_0805_2012Metric_Pad1.15x1.40mm_HandSolder
- removed R83, R84, R85: 470, Resistor_SMD:R_0805_2012Metric_Pad1.15x1.40mm_HandSolder
- removed R94: 33k, Resistor_SMD:R_0805_2012Metric_Pad1.15x1.40mm_HandSolder
- removed REF**: OSHW-Logo_5.7x6mm_SilkScreen, Symbol:OSHW-Logo_5.7x6mm_SilkScreen
- removed RV2, RV4, RV5: 2.7k, Potentiometer_THT:Potentiometer_Bourns_3386P_Vertical
- removed RV3: 2k, Potentiometer_THT:Potentiometer_Bourns_3386P_Vertical
- removed RV6, RV7, RV8, RV9: 1k, Potentiometer_THT:Potentiometer_Bourns_3386P_Vertical
- removed T1: CST1-125LC, Transformer_SMD:Transformer_Coilcraft_CST1
- added C64: 10uF, Capacitor_THT:CP_Radial_D8.0mm_P3.50mm, F.Cu at (18.1, -55.9)
- added C69: 10uF 100V, Capacitor_SMD:CP_Elec_8x11.9, F.Cu at (-63.5, -18.0)
- added C70: 10uF, Capacitor_THT:CP_Radial_D8.0mm_P3.50mm, F.Cu at (18.1, -46.4)
- added C74: 100uF, Capacitor_THT:CP_Radial_D8.0mm_P3.50mm, F.Cu at (18.1, -36.8)
- added C75: 100uF, Capacitor_THT:CP_Radial_D8.0mm_P3.50mm, F.Cu at (18.1, -27.3)
- added C89: 0.47uF, Capacitor_THT:C_Rect_L18.0mm_W8.0mm_P15.00mm_FKS3_FKP3, F.Cu at (64.4, -30.4)
- added D10: WNSC2D04650DJ, Package_TO_SOT_SMD:TO-252-2_TabPin1, F.Cu at (32.5, -56.4)
- added D12: 1N4148W, Diode_SMD:D_SOD-123, F.Cu at (43.9, -76.2)
- added D13: 1N4148W, Diode_SMD:D_SOD-123, F.Cu at (43.9, -72.8)
- added D14: 1N4148W, Diode_SMD:D_SOD-123, F.Cu at (43.9, -69.5)
- added D15: B220, Diode_SMD:D_SMB, F.Cu at (37.2, -38.3)
- added D16: B220, Diode_SMD:D_SMB, F.Cu at (37.2, -32.7)
- added D18: ES1G-13-F, Diode_SMD:D_SMA, F.Cu at (55.9, -45.0)
- added D19: ES1G-13-F, Diode_SMD:D_SMA, F.Cu at (55.9, -40.4)
- added D20: ES1G-13-F, Diode_SMD:D_SMA, F.Cu at (78.7, -15.3)
- added L7: 680uH, td-deflect:Murata_6000B, F.Cu at (112.0, 29.2)
- added L8: 680uH, td-deflect:Murata_6000B, F.Cu at (79.0, 29.2)
- added L9: 680uH, td-deflect:Murata_6000B, F.Cu at (79.0, 60.2)
- added Q17: BSZ42DN25NS3GATMA1, Package_TO_SOT_SMD:TDSON-8-1, F.Cu at (86.4, -45.0)
- added Q18: G3R450MT17J, Package_TO_SOT_SMD:TO-263-7_TabPin8, F.Cu at (72.8, -54.5)
- added Q19: BSZ42DN25NS3GATMA1, Package_TO_SOT_SMD:TDSON-8-1, F.Cu at (37.1, -26.6)
- added Q20: BSZ42DN25NS3GATMA1, Package_TO_SOT_SMD:TDSON-8-1, F.Cu at (56.0, -57.3)
- added Q21: BSZ42DN25NS3GATMA1, Package_TO_SOT_SMD:TDSON-8-1, F.Cu at (56.0, -50.6)
- added Q22: IPD50R380CE, Package_TO_SOT_SMD:TO-252-2, F.Cu at (81.5, -21.6)
- added R110: 1k, Resistor_THT:R_Radial_Power_L11.0mm_W7.0mm_P5.00mm, F.Cu at (65.9, -21.4)
- added RV11: 10k, Potentiometer_THT:Potentiometer_Bourns_3386P_Vertical, F.Cu at (85.3, -52.6)
- added RV12: 1k, Potentiometer_THT:Potentiometer_Bourns_3386P_Vertical, F.Cu at (125.5, -40.5)
- added TP1: TestPoint, TestPoint:TestPoint_Keystone_5010-5014_Multipurpose, F.Cu at (17.4, -75.3)
- added TP10: TestPoint, TestPoint:TestPoint_Keystone_5010-5014_Multipurpose, F.Cu at (79.8, -45.8)
- added TP11: TestPoint, TestPoint:TestPoint_Keystone_5010-5014_Multipurpose, F.Cu at (79.8, -40.8)
- added TP2: TestPoint, TestPoint:TestPoint_Keystone_5010-5014_Multipurpose, F.Cu at (17.4, -70.3)
- added TP3: TestPoint, TestPoint:TestPoint_Keystone_5010-5014_Multipurpose, F.Cu at (17.4, -65.2)
- added TP4: TestPoint, TestPoint:TestPoint_Keystone_5010-5014_Multipurpose, F.Cu at (64.6, -45.8)
- added TP5: TestPoint, TestPoint:TestPoint_Keystone_5010-5014_Multipurpose, F.Cu at (64.6, -40.8)
- added TP6: TestPoint, TestPoint:TestPoint_Keystone_5010-5014_Multipurpose, F.Cu at (69.7, -45.8)
- added TP7: TestPoint, TestPoint:TestPoint_Keystone_5010-5014_Multipurpose, F.Cu at (69.7, -40.8)
- added TP8: TestPoint, TestPoint:TestPoint_Keystone_5010-5014_Multipurpose, F.Cu at (74.7, -45.8)
- added TP9: TestPoint, TestPoint:TestPoint_Keystone_5010-5014_Multipurpose, F.Cu at (74.7, -40.8)
- added U21: MCP1416, Package_TO_SOT_SMD:SOT-23-5, F.Cu at (84.9, -39.4)
- added U22: LT3758AEMSE, Package_SO:MSOP-10-1EP_3x3mm_P0.5mm_EP1.68x1.88mm, F.Cu at (141.6, -44.5)
- added U23: TPS70933, Package_TO_SOT_SMD:SOT-23-5, F.Cu at (46.0, -30.7)
- added U24: INA181, Package_TO_SOT_SMD:SOT-23-6, F.Cu at (46.0, -26.2)
- added U25: FM24C64B, Package_SO:SOIC-8_3.9x4.9mm_P1.27mm, F.Cu at (52.8, -29.7)
- added U26: MCP4728, Package_SO:MSOP-10_3x3mm_P0.5mm, F.Cu at (9.20, 69.0)
- added U27: MCP4728, Package_SO:MSOP-10_3x3mm_P0.5mm, F.Cu at (9.00, 63.0)
- added U28: TL082, Package_SO:SOIC-8_3.9x4.9mm_P1.27mm, F.Cu at (24.1, -74.6)
- added U29: MCP6001U, Package_SO:SOIC-8_3.9x4.9mm_P1.27mm, F.Cu at (93.0, -31.9)
- added U30: TL082, Package_SO:SOIC-8_3.9x4.9mm_P1.27mm, F.Cu at (24.1, -68.2)
- added U31: ASSR-1218, Package_SO:SO-4_4.4x4.3mm_P2.54mm, F.Cu at (51.2, -74.9)
- added U32: BD9G341AEFJ, Package_SO:SOIC-8-1EP_3.9x4.9mm_P1.27mm_EP2.41x3.3mm_ThermalVias, F.Cu at (28.8, -37.8)
- added U33: BD9G341AEFJ, Package_SO:SOIC-8-1EP_3.9x4.9mm_P1.27mm_EP2.41x3.3mm_ThermalVias, F.Cu at (28.8, -31.4)
- added U34: IRS2005S, Package_SO:SOIC-8_3.9x4.9mm_P1.27mm, F.Cu at (47.6, -57.5)
- added U35: IRS2005S, Package_SO:SOIC-8_3.9x4.9mm_P1.27mm, F.Cu at (47.6, -51.0)
- added U36: MAX9919F, Package_SO:SOIC-8-1EP_3.9x4.9mm_P1.27mm_EP2.41x3.3mm, F.Cu at (47.6, -44.6)
- added U37: MAX9919F, Package_SO:SOIC-8-1EP_3.9x4.9mm_P1.27mm_EP2.41x3.3mm, F.Cu at (47.6, -38.1)
- added U38: MCP1416, Package_TO_SOT_SMD:SOT-23-5, F.Cu at (84.2, -33.0)
- C11: value 0.033uF -> 0.056uF; footprint Capacitor_SMD:C_1206_3216Metric_Pad1.42x1.75mm_HandSolder -> Capacitor_THT:C_Rect_L18.0mm_W5.0mm_P15.00mm_FKS3_FKP3
- C13: value 0.015uF -> 0.056uF; footprint Capacitor_SMD:C_1206_3216Metric_Pad1.42x1.75mm_HandSolder -> Capacitor_THT:C_Rect_L18.0mm_W5.0mm_P15.00mm_FKS3_FKP3
- C14: value 0.033uF -> 0.12uF; footprint Capacitor_SMD:C_1206_3216Metric_Pad1.42x1.75mm_HandSolder -> Capacitor_THT:C_Rect_L18.0mm_W8.0mm_P15.00mm_FKS3_FKP3
- C15: value 0.068uF -> 0.22uF; footprint Capacitor_SMD:C_1206_3216Metric_Pad1.42x1.75mm_HandSolder -> Capacitor_THT:C_Rect_L18.0mm_W6.0mm_P15.00mm_FKS3_FKP3
- C16: value 0.12uF -> 0.47uF; footprint Capacitor_SMD:C_1206_3216Metric_Pad1.42x1.75mm_HandSolder -> Capacitor_THT:C_Rect_L18.0mm_W8.0mm_P15.00mm_FKS3_FKP3
- C30: value 0.1uF -> 47pF 2000V NP0; footprint Capacitor_SMD:C_0805_2012Metric_Pad1.15x1.40mm_HandSolder -> Capacitor_SMD:C_1206_3216Metric
- C32: value 100uF -> 1000pf; footprint Capacitor_THT:CP_Radial_D8.0mm_P3.50mm -> Capacitor_THT:C_Rect_L18.0mm_W6.0mm_P15.00mm_FKS3_FKP3
- C33: value 2.2uF -> 22uF; footprint Capacitor_SMD:C_0805_2012Metric_Pad1.15x1.40mm_HandSolder -> Capacitor_THT:CP_Radial_D8.0mm_P3.50mm
- C35: value 4.7uF -> 0.01uF
- C59: value 0.1uF -> C
- D1: value BA157 -> ES1G-13-F; footprint Diode_THT:D_DO-41_SOD81_P10.16mm_Horizontal -> Diode_SMD:D_SMA
- D3: value 1N5402 -> WNSC2D04650DJ; footprint Diode_THT:D_DO-201AD_P15.24mm_Horizontal -> Package_TO_SOT_SMD:TO-252-2_TabPin1
- D4: value C3D10170H -> ES1G-13-F; footprint Package_TO_SOT_THT:TO-247-2_Vertical -> Diode_SMD:D_SMA
- D6, D7, D8: value BAT54S -> 1N4148W; footprint Package_TO_SOT_SMD:SOT-23 -> Diode_SMD:D_SOD-123
- J12: value Conn_01x06_Male -> Conn_01x02_Male; footprint td-deflect:sony_monitor_yoke -> td-deflect:monitor_10_8_2p
- J15: footprint td-deflect:sony_monitor_2p -> td-deflect:monitor_10_8_2p
- J8: footprint Connector_Phoenix_MSTB:PhoenixContact_MSTBVA_2,5_2-G_1x02_P5.00mm_Vertical -> td-deflect:sony_monitor_2p
- L1: value 1mH -> 680uH; footprint Inductor_THT:L_Toroid_Vertical_L31.8mm_W15.9mm_P13.50mm_Bourns_5700 -> td-deflect:Murata_6000B
- L5: value 100uH -> 47uH; footprint Inductor_SMD:L_Bourns_SRR1260 -> Inductor_SMD:L_Bourns_SRF1260
- L6: value 1mH -> 33uH; footprint Inductor_THT:L_Toroid_Vertical_L31.8mm_W15.9mm_P13.50mm_Bourns_5700 -> Inductor_SMD:L_Bourns_SRR1260
- Q1, Q13, Q3: value BSC082N10LSG -> BSZ42DN25NS3GATMA1
- Q12: value C2M0045170D -> BSZ42DN25NS3GATMA1; footprint Package_TO_SOT_THT:TO-247-3_Vertical -> Package_TO_SOT_SMD:TDSON-8-1
- Q14: value BC847 -> BCP56; footprint Package_TO_SOT_SMD:SOT-23 -> Package_TO_SOT_SMD:SOT-223-3_TabPin2
- Q15, Q16: value BC847 -> BSZ42DN25NS3GATMA1; footprint Package_TO_SOT_SMD:SOT-23 -> Package_TO_SOT_SMD:TDSON-8-1
- Q2: value C2M0045170D -> G3R450MT17J; footprint Package_TO_SOT_THT:TO-247-3_Vertical -> Package_TO_SOT_SMD:TO-263-7_TabPin8
- R13: value 100 -> 1k
- R14: value 10k -> 1k
- R22: footprint Resistor_SMD:R_0805_2012Metric_Pad1.15x1.40mm_HandSolder -> Resistor_SMD:R_1210_3225Metric
- R30: value 37.4k -> 100k
- R38: value 1M -> 3k; footprint Resistor_THT:R_Axial_DIN0309_L9.0mm_D3.2mm_P15.24mm_Horizontal -> Resistor_SMD:R_2512_6332Metric
- R44: value 39k -> 1M 3000V; footprint Resistor_SMD:R_0805_2012Metric_Pad1.15x1.40mm_HandSolder -> Resistor_SMD:R_2512_6332Metric
- R66: value 220 -> 1M 3000V; footprint Resistor_SMD:R_0805_2012Metric_Pad1.15x1.40mm_HandSolder -> Resistor_SMD:R_2512_6332Metric
- R69: value 47k -> 10k; footprint Resistor_SMD:R_0805_2012Metric_Pad1.15x1.40mm_HandSolder -> Resistor_SMD:R_1210_3225Metric
- R82: value 220 -> 1
- SW1: footprint Button_Switch_THT:SW_DIP_SPSTx04_Slide_9.78x12.34mm_W7.62mm_P2.54mm -> Button_Switch_SMD:SW_DIP_SPSTx04_Slide_Omron_A6S-410x_W8.9mm_P2.54mm
- U12: value LM1117-3.3 -> LM1117-5.0
- U13: value MCP1416 -> LM2903; footprint Package_TO_SOT_SMD:SOT-23-5 -> Package_SO:SOIC-8_3.9x4.9mm_P1.27mm
- U15: value LM1117-ADJ -> 74HC00; footprint Package_TO_SOT_SMD:TO-252-2 -> Package_SO:SOIC-14_3.9x8.7mm_P1.27mm
- U16: value LTC7149FE -> IRS2005S; footprint Package_SO:HTSSOP-28-1EP_4.4x9.7mm_P0.65mm_EP2.85x5.4mm -> Package_SO:SOIC-8_3.9x4.9mm_P1.27mm
- U17: value TPS54360DDA -> LM2903; footprint Package_SO:TI_SO-PowerPAD-8_ThermalVias -> Package_SO:SOIC-8_3.9x4.9mm_P1.27mm
- U18: value M51387P -> LM1205; footprint td-deflect:DIP-30_600_ELL -> Package_DIP:DIP-28_W15.24mm
- U2: value STM32F722RETx -> STM32G474RETx
- U20: value 74LVC1GU04DRL -> 74LVC1GU04DRLR
- U3: value INA193 -> INA181; footprint Package_TO_SOT_SMD:SOT-23-5 -> Package_TO_SOT_SMD:SOT-23-6
- U7: value LTC6090 -> 74HC00; footprint Package_SO:SOIC-8-1EP_3.9x4.9mm_P1.27mm_EP2.29x3mm -> Package_SO:SOIC-14_3.9x8.7mm_P1.27mm
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Connections:
- net /Sheet5C37BEF6/16mhz renamed /uc/16mhz
- net /Sheet5C37BEF6/nrst renamed /uc/nrst
- net Net-(U2-Pad2) renamed V_EN
- net Net-(U2-Pad33) renamed BPLUS_VOLTAGE
- net Net-(U2-Pad44) renamed V_CURRENT_CLASSD
- C11 pad 2: GND -> Net-(Q10-S)
- C30 pad 1: Net-(C30-Pad1) -> /flyback/eht out
- C32 pad 1: GND -> /flyback/eht out
- C32 pad 2: -12V -> GND
- C33 pad 1: Net-(C29-Pad1) -> +48V
- C59 pad 1: Net-(C59-Pad1) -> HT
- D4 pad 1: /power_supply/eht out -> Net-(D4-K)
- D4 pad 2: GND -> +12V
- D5 pad 1: Net-(C43-Pad2) -> Net-(D5-K)
- D6 pad 1: GND -> Net-(D6-K)
- D6 pad 2: Net-(C60-Pad1) -> +48V
- D7 pad 1: GND -> Net-(D7-K)
- D7 pad 2: Net-(C60-Pad1) -> +12V
- D8 pad 1: GND -> Net-(D6-K)
- D8 pad 2: Net-(C60-Pad1) -> Net-(D7-K)
- F1 pad 1: /v.out -> Net-(F1-Pad1)
- J11 pad 2: /v.ret -> V_CURRENT
- J12 pad 1: /h.out -> Net-(J12-Pin_1)
- J12 pad 2: /h.out -> GND
- J15 pad 1: GND -> Net-(J12-Pin_1)
- J15 pad 2: Net-(J15-Pad2) -> GND
- J4 pad 2: /Sheet5C37BEF6/tms -> /uc/tms
- J4 pad 4: /Sheet5C37BEF6/tck -> /uc/tck
- J4 pad 6: /Sheet5C37BEF6/tdo -> /uc/tdo
- J4 pad 7: Net-(J4-Pad7) -> unconnected-(J4-KEY-Pad7)
- J4 pad 8: /Sheet5C37BEF6/tdi -> unconnected-(J4-NC/TDI-Pad8)
- J5 pad 11: Net-(J5-Pad11) -> unconnected-(J5-Pad11)
- J5 pad 4: Net-(J5-Pad4) -> unconnected-(J5-Pad4)
- J6 pad 2: Net-(J6-Pad2) -> unconnected-(J6-Pin_2-Pad2)
- J6 pad 3: Net-(J6-Pad3) -> unconnected-(J6-Pin_3-Pad3)
- J6 pad 4: /Sheet5C37BEF6/rx -> /uc/rx
- J6 pad 5: /Sheet5C37BEF6/tx -> /uc/tx
- J6 pad 6: Net-(J6-Pad6) -> unconnected-(J6-Pin_6-Pad6)
- J7 pad 2: Net-(J7-Pad2) -> unconnected-(J7-Pin_2-Pad2)
- J8 pad 2: /power_supply/eht out -> Net-(J8-Pin_2)
- J9 pad 2: Net-(J15-Pad2) -> +6V
- L1 pad 2: /h.out -> Net-(L1-Pad2)
- L2 pad 1: Net-(L2-Pad1) -> /h.ret
- L5 pad 1: Net-(C43-Pad2) -> GND
- L5 pad 2: +12V -> Net-(D5-K)
- L6 pad 1: HT -> +48V
- L6 pad 2: /power_supply/eht out -> Net-(D10-A)
- Q1 pad 4: Net-(Q1-Pad4) -> Net-(Q1-G)
- Q10 pad 3: GND -> Net-(Q10-S)
- Q11 pad 3: GND -> Net-(Q10-S)
- Q12 pad 1: Net-(Q12-Pad1) -> Net-(Q17-D)
- Q12 pad 2: /power_supply/eht out -> Net-(Q17-D)
- Q12 pad 3: EHT_CURRENT -> Net-(Q17-D)
- Q14 pad 2: GND -> Net-(D13-K)
- Q15 pad 1: Net-(Q15-Pad1) -> Net-(Q16-D)
- Q15 pad 2: GND -> Net-(Q16-D)
- Q15 pad 3: Net-(Q15-Pad3) -> Net-(Q16-D)
- Q16 pad 1: Net-(Q16-Pad1) -> GND
- Q16 pad 3: Net-(Q16-Pad3) -> GND
- Q2 pad 2: /h.out -> HOT_CURRENT
- Q3 pad 4: Net-(Q3-Pad4) -> Net-(Q3-G)
- Q4 pad 1: Net-(Q4-Pad1) -> Net-(D12-A)
- Q4 pad 2: +48V -> Net-(Q7-B)
- Q4 pad 3: Net-(Q4-Pad3) -> Net-(D14-A)
- Q5 pad 1: Net-(Q4-Pad1) -> Net-(D13-K)
- Q5 pad 2: Net-(Q5-Pad2) -> Net-(Q6-B)
- Q5 pad 3: -12V -> Net-(Q5-E)
- Q6 pad 1: Net-(Q6-Pad1) -> -12V
- Q6 pad 2: +48V -> Net-(Q5-E)
- Q6 pad 3: Net-(Q4-Pad3) -> Net-(Q6-B)
- Q7 pad 1: -12V -> +48V
- Q7 pad 2: Net-(Q7-Pad2) -> Net-(D14-A)
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Routing:
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Other:
- board size 275 x 110 mm -> 270 x 110 mm
- board text removed: "All"
- board text removed: "B"
- board text removed: "Bias"
- board text removed: "G"
- board text removed: "Gain"
- board text removed: "R"

Commit message: more layout work
Parts:
- removed C20, C35: 0.01uF, Capacitor_SMD:C_0805_2012Metric_Pad1.15x1.40mm_HandSolder
- removed C21: 100pF, Capacitor_SMD:C_0805_2012Metric_Pad1.15x1.40mm_HandSolder
- removed C22: 10uF, Capacitor_SMD:C_1206_3216Metric_Pad1.42x1.75mm_HandSolder
- removed C23: 4.7uF, Capacitor_SMD:C_0805_2012Metric_Pad1.15x1.40mm_HandSolder
- removed C25, C34, C64, C70: 10uF, Capacitor_THT:CP_Radial_D8.0mm_P3.50mm
- removed C26: 0.1uF, Capacitor_SMD:C_1206_3216Metric_Pad1.42x1.75mm_HandSolder
- removed C30: 47pF 2000V NP0, Capacitor_SMD:C_1206_3216Metric
- removed C32: 1000pf, Capacitor_THT:C_Rect_L18.0mm_W6.0mm_P15.00mm_FKS3_FKP3
- removed C33: 22uF, Capacitor_THT:CP_Radial_D8.0mm_P3.50mm
- removed C40: 22uF, Capacitor_SMD:C_1206_3216Metric_Pad1.42x1.75mm_HandSolder
- removed C46, C74, C75: 100uF, Capacitor_THT:CP_Radial_D8.0mm_P3.50mm
- removed C57: 1uF, Capacitor_SMD:C_0805_2012Metric_Pad1.15x1.40mm_HandSolder
- removed C58: 0.1uF, Capacitor_SMD:C_0805_2012Metric_Pad1.15x1.40mm_HandSolder
- removed D10, D3: WNSC2D04650DJ, Package_TO_SOT_SMD:TO-252-2_TabPin1
- removed D15, D16, D5: B220, Diode_SMD:D_SMB
- removed D4: ES1G-13-F, Diode_SMD:D_SMA
- removed J15: Conn_01x02_Male, td-deflect:monitor_10_8_2p
- removed L3, L6: 33uH, Inductor_SMD:L_Bourns_SRR1260
- removed L5: 47uH, Inductor_SMD:L_Bourns_SRF1260
- removed Q12, Q13, Q17, Q19: BSZ42DN25NS3GATMA1, Package_TO_SOT_SMD:TDSON-8-1
- removed Q18: G3R450MT17J, Package_TO_SOT_SMD:TO-263-7_TabPin8
- removed R19, R96: 1, Resistor_SMD:R_0805_2012Metric_Pad1.15x1.40mm_HandSolder
- removed R32: 49.9k, Resistor_SMD:R_0805_2012Metric_Pad1.15x1.40mm_HandSolder
- removed R37: 0.01, Resistor_SMD:R_0805_2012Metric_Pad1.15x1.40mm_HandSolder
- removed R38: 3k, Resistor_SMD:R_2512_6332Metric
- removed R39: 70K, Resistor_SMD:R_1206_3216Metric_Pad1.42x1.75mm_HandSolder
- removed R40: 470, Resistor_SMD:R_0805_2012Metric_Pad1.15x1.40mm_HandSolder
- removed R44: 1M 3000V, Resistor_SMD:R_2512_6332Metric
- removed R89: 10k, Resistor_SMD:R_0805_2012Metric_Pad1.15x1.40mm_HandSolder
- removed R90, R91, R92, R93: 75, Resistor_SMD:R_0805_2012Metric_Pad1.15x1.40mm_HandSolder
- removed RV1, RV12: 1k, Potentiometer_THT:Potentiometer_Bourns_3386P_Vertical
- removed RV10, RV11: 10k, Potentiometer_THT:Potentiometer_Bourns_3386P_Vertical
- removed TP10, TP11, TP4, TP5, TP6, TP7, TP8, TP9: TestPoint, TestPoint:TestPoint_Keystone_5010-5014_Multipurpose
- removed U12: LM1117-5.0, Package_TO_SOT_SMD:TO-252-2
- removed U13, U17: LM2903, Package_SO:SOIC-8_3.9x4.9mm_P1.27mm
- removed U14, U22: LT3758AEMSE, Package_SO:MSOP-10-1EP_3x3mm_P0.5mm_EP1.68x1.88mm
- removed U15: 74HC00, Package_SO:SOIC-14_3.9x8.7mm_P1.27mm
- removed U16: IRS2005S, Package_SO:SOIC-8_3.9x4.9mm_P1.27mm
- removed U18: LM1205, Package_DIP:DIP-28_W15.24mm
- removed U19: LMH1980, Package_SO:VSSOP-10_3x3mm_P0.5mm
- removed U20: 74LVC1GU04DRLR, Package_TO_SOT_SMD:SOT-553
- removed U21: MCP1416, Package_TO_SOT_SMD:SOT-23-5
- removed U26, U27: MCP4728, Package_SO:MSOP-10_3x3mm_P0.5mm
- removed U29: MCP6001U, Package_SO:SOIC-8_3.9x4.9mm_P1.27mm
- removed U30: TL082, Package_SO:SOIC-8_3.9x4.9mm_P1.27mm
- removed U32, U33: BD9G341AEFJ, Package_SO:SOIC-8-1EP_3.9x4.9mm_P1.27mm_EP2.41x3.3mm_ThermalVias
- removed U36, U37: MAX9919F, Package_SO:SOIC-8-1EP_3.9x4.9mm_P1.27mm_EP2.41x3.3mm
- added C19: 0.1uF, Capacitor_SMD:C_0805_2012Metric_Pad1.18x1.45mm_HandSolder, F.Cu at (-2.31, 86.0)
- added C60: 0.1uF, Capacitor_SMD:C_0805_2012Metric_Pad1.18x1.45mm_HandSolder, F.Cu at (22.0, 64.2)
- added C66: 4.7uF, Capacitor_SMD:C_0805_2012Metric_Pad1.18x1.45mm_HandSolder, F.Cu at (-29.1, 91.1)
- added C76: 1uF 50V, Capacitor_SMD:C_0805_2012Metric_Pad1.18x1.45mm_HandSolder, F.Cu at (80.0, 75.1)
- added C77: 1uF 50V, Capacitor_SMD:C_0805_2012Metric_Pad1.18x1.45mm_HandSolder, F.Cu at (94.0, 75.1)
- added C78: 0.1uF, Capacitor_SMD:C_0805_2012Metric_Pad1.18x1.45mm_HandSolder, F.Cu at (92.0, 56.9)
- added C79: 0.1uF, Capacitor_SMD:C_0805_2012Metric_Pad1.18x1.45mm_HandSolder, F.Cu at (78.8, 57.1)
- added C80: 0.1uF, Capacitor_SMD:C_0805_2012Metric_Pad1.18x1.45mm_HandSolder, F.Cu at (95.2, 63.2)
- added C81: 0.1uF, Capacitor_SMD:C_0805_2012Metric_Pad1.18x1.45mm_HandSolder, F.Cu at (79.5, 62.9)
- added C82: 15uF, Capacitor_SMD:C_0805_2012Metric_Pad1.18x1.45mm_HandSolder, F.Cu at (93.0, 93.0)
- added C83: 15uF, Capacitor_SMD:C_0805_2012Metric_Pad1.18x1.45mm_HandSolder, F.Cu at (76.0, 93.0)
- added C84: 10uF, Capacitor_SMD:C_0805_2012Metric_Pad1.18x1.45mm_HandSolder, F.Cu at (88.0, 93.0)
- added C85: 10uF, Capacitor_SMD:C_0805_2012Metric_Pad1.18x1.45mm_HandSolder, F.Cu at (71.0, 93.0)
- added C86: 0.1uF, Capacitor_SMD:C_0805_2012Metric_Pad1.18x1.45mm_HandSolder, F.Cu at (66.0, 64.0)
- added C87: 0.1uF, Capacitor_SMD:C_0805_2012Metric_Pad1.18x1.45mm_HandSolder, F.Cu at (66.0, 73.0)
- added C88: 0.1uF, Capacitor_SMD:C_0805_2012Metric_Pad1.18x1.45mm_HandSolder, F.Cu at (106.5, 53.5)
- added D17: D_Zener, Diode_SMD:D_0805_2012Metric_Pad1.15x1.40mm_HandSolder, F.Cu at (23.0, 41.0)
- added F3: 1A, Fuse:Fuse_Schurter_UMT250, F.Cu at (19.8, 36.0)
- added H10: MountingHole, MountingHole:MountingHole_3.2mm_M3, F.Cu at (-11.0, 26.0)
- added H11: MountingHole, MountingHole:MountingHole_3.2mm_M3, F.Cu at (41.0, 26.0)
- added H12: MountingHole, MountingHole:MountingHole_3.2mm_M3, F.Cu at (103.0, 6.00)
- added H13: MountingHole, MountingHole:MountingHole_3.2mm_M3, F.Cu at (103.0, 26.0)
- added H14: MountingHole, MountingHole:MountingHole_3.2mm_M3, F.Cu at (103.0, 46.0)
- added H5: MountingHole, MountingHole:MountingHole_3.2mm_M3, F.Cu at (41.0, 6.00)
- added H6: MountingHole, MountingHole:MountingHole_3.2mm_M3, F.Cu at (-11.0, 6.00)
- added H7: MountingHole, MountingHole:MountingHole_3.2mm_M3, F.Cu at (51.0, 6.00)
- added H8: MountingHole, MountingHole:MountingHole_3.2mm_M3, F.Cu at (51.0, 26.0)
- added H9: MountingHole, MountingHole:MountingHole_3.2mm_M3, F.Cu at (51.0, 46.0)
- added HS1: Heatsink_Pad, td-deflect:c220-050-2ae, F.Cu at (60.9, 94.5)
- added J1: Conn_01x05_Pin, Connector_JST:JST_XH_B5B-XH-A_1x05_P2.50mm_Vertical, F.Cu at (-5.00, 100.0)
- added J19: Conn_01x08_Socket, Connector_PinSocket_2.54mm:PinSocket_1x08_P2.54mm_Vertical, F.Cu at (87.5, 6.00)
- added J20: Conn_01x08_Socket, Connector_PinSocket_2.54mm:PinSocket_1x08_P2.54mm_Vertical, F.Cu at (87.5, 26.0)
- added J21: Conn_01x08_Socket, Connector_PinSocket_2.54mm:PinSocket_1x08_P2.54mm_Vertical, F.Cu at (87.5, 46.0)
- added J3: Conn_01x04_Male, Connector_JST:JST_XH_B4B-XH-A_1x04_P2.50mm_Vertical, F.Cu at (35.0, 35.0)
- added JP1: Jumper_2_Open, Connector_PinHeader_2.54mm:PinHeader_1x02_P2.54mm_Vertical, F.Cu at (87.5, 15.0)
- added JP2: Jumper_2_Open, Connector_PinHeader_2.54mm:PinHeader_1x02_P2.54mm_Vertical, F.Cu at (88.0, 35.0)
- added L11: 100uF, Inductor_SMD:L_Bourns_SRR1260, F.Cu at (89.0, 84.0)
- added L12: 100uF, Inductor_SMD:L_Bourns_SRR1260, F.Cu at (75.0, 84.0)
- added R107: 0.01, Resistor_SMD:R_0805_2012Metric_Pad1.20x1.40mm_HandSolder, F.Cu at (76.0, 96.0)
- added R108: 10k, Resistor_SMD:R_0805_2012Metric_Pad1.20x1.40mm_HandSolder, F.Cu at (106.5, 57.5)
- added R109: 1, Resistor_SMD:R_0805_2012Metric_Pad1.20x1.40mm_HandSolder, F.Cu at (112.0, 48.0)
- added R112: 10k, Resistor_SMD:R_0805_2012Metric_Pad1.20x1.40mm_HandSolder, F.Cu at (-13.0, 33.0)
- added R12: 10k, Resistor_SMD:R_0805_2012Metric, F.Cu at (-31.0, 47.1)
- added R56: R, Resistor_SMD:R_0805_2012Metric_Pad1.20x1.40mm_HandSolder, F.Cu at (-13.0, 44.0)
- added R57: R, Resistor_SMD:R_0805_2012Metric_Pad1.20x1.40mm_HandSolder, F.Cu at (-13.0, 42.0)
- added R64: 1, Resistor_SMD:R_0805_2012Metric_Pad1.20x1.40mm_HandSolder, F.Cu at (121.5, 8.00)
- added R65: 1, Resistor_SMD:R_0805_2012Metric_Pad1.20x1.40mm_HandSolder, F.Cu at (121.5, 15.0)
- added R67: 1k, Resistor_SMD:R_0805_2012Metric_Pad1.20x1.40mm_HandSolder, F.Cu at (112.5, 89.5)
- added R68: 10, Resistor_SMD:R_0805_2012Metric_Pad1.20x1.40mm_HandSolder, F.Cu at (28.5, 64.0)
- added R70: 100, Resistor_SMD:R_0805_2012Metric_Pad1.20x1.40mm_HandSolder, F.Cu at (28.5, 68.5)
- added R71: 1k, Resistor_SMD:R_0805_2012Metric_Pad1.20x1.40mm_HandSolder, F.Cu at (22.0, 68.5)
- added R72: 0.01, Resistor_SMD:R_0805_2012Metric_Pad1.20x1.40mm_HandSolder, F.Cu at (152.6, 85.3)
- added R73: 220k, Resistor_SMD:R_0805_2012Metric_Pad1.20x1.40mm_HandSolder, F.Cu at (87.0, 3.00)
- added R74: 1k, Resistor_SMD:R_0805_2012Metric_Pad1.20x1.40mm_HandSolder, F.Cu at (83.0, 3.00)
- added R80: 1, Resistor_SMD:R_0805_2012Metric_Pad1.20x1.40mm_HandSolder, F.Cu at (92.0, 63.9)
- added R81: 1, Resistor_SMD:R_0805_2012Metric_Pad1.20x1.40mm_HandSolder, F.Cu at (85.0, 63.9)
- added R83: 1, Resistor_SMD:R_0805_2012Metric_Pad1.20x1.40mm_HandSolder, F.Cu at (71.0, 63.9)
- added R84: 0.01, Resistor_SMD:R_0805_2012Metric_Pad1.20x1.40mm_HandSolder, F.Cu at (86.0, 75.1)
- added R85: 5.1, Resistor_SMD:R_0805_2012Metric_Pad1.20x1.40mm_HandSolder, F.Cu at (93.0, 96.0)
- added R94: 5.1, Resistor_SMD:R_0805_2012Metric_Pad1.20x1.40mm_HandSolder, F.Cu at (71.0, 96.0)
- added R95: 330, Resistor_SMD:R_0805_2012Metric_Pad1.20x1.40mm_HandSolder, F.Cu at (80.5, 93.0)
- C1, C10, C12, C2, C3, C36, C37, C38, C39, C4, C41, C42, C5, C7, C8, C9: footprint Capacitor_SMD:C_0805_2012Metric_Pad1.15x1.40mm_HandSolder -> Capacitor_SMD:C_0805_2012Metric_Pad1.18x1.45mm_HandSolder
- C17: value 4.7uF -> 0.1uF; footprint Capacitor_SMD:C_0805_2012Metric_Pad1.15x1.40mm_HandSolder -> Capacitor_SMD:C_0805_2012Metric_Pad1.18x1.45mm_HandSolder
- C18: value 22uF -> 0.1uF; footprint Capacitor_THT:CP_Radial_D8.0mm_P3.50mm -> Capacitor_SMD:C_0805_2012Metric_Pad1.18x1.45mm_HandSolder
- C59: value C -> 0.1uF; footprint Capacitor_SMD:C_0805_2012Metric_Pad1.15x1.40mm_HandSolder -> Capacitor_SMD:C_0805_2012Metric_Pad1.18x1.45mm_HandSolder
- D1: value ES1G-13-F -> DNP; footprint Diode_SMD:D_SMA -> Diode_SMD:D_SOD-123
- D18, D19: value ES1G-13-F -> 1N4148W-TP; footprint Diode_SMD:D_SMA -> Diode_SMD:D_SOD-123
- J13, J14: value Conn_01x02_Male -> Conn_01x12_Socket; footprint Connector_Phoenix_MSTB:PhoenixContact_MSTBVA_2,5_2-G_1x02_P5.00mm_Vertical -> Connector_PinSocket_2.54mm:PinSocket_1x12_P2.54mm_Vertical
- J16: value Conn_01x06_Male -> Conn_02x10_Odd_Even; footprint Connector_JST:JST_EH_B6B-EH-A_1x06_P2.50mm_Vertical -> Connector_IDC:IDC-Header_2x10_P2.54mm_Vertical
- J17: value Conn_01x06_Male -> Barrel_Jack; footprint Connector_JST:JST_XH_B6B-XH-A_1x06_P2.50mm_Vertical -> Connector_BarrelJack:BarrelJack_CLIFF_FC681465S_SMT_Horizontal
- J2: value Conn_01x02_Male -> USB_C_Receptacle_USB2.0; footprint Connector_Phoenix_MSTB:PhoenixContact_MSTBVA_2,5_2-G_1x02_P5.00mm_Vertical -> Connector_USB:USB_C_Receptacle_XKB_U262-16XN-4BVC11
- J5: value DB15_Female_HighDensity -> Conn_01x07_Male; footprint Connector_Dsub:DSUB-15-HD_Female_Horizontal_P2.29x1.98mm_EdgePinOffset3.03mm_Housed_MountingHolesOffset4.94mm -> Connector_JST:JST_XH_B7B-XH-A_1x07_P2.50mm_Vertical
- J7: value Conn_01x08_Male -> Conn_02x10_Odd_Even; footprint Connector_JST:JST_PH_B8B-PH-K_1x08_P2.00mm_Vertical -> Connector_IDC:IDC-Header_2x10_P2.54mm_Vertical
- J9: value Conn_01x02_Male -> Conn_01x14; footprint Connector_Phoenix_MSTB:PhoenixContact_MSTBVA_2,5_2-G_1x02_P5.00mm_Vertical -> Connector_JST:JST_XH_B14B-XH-A_1x14_P2.50mm_Vertical
- Q1, Q15, Q16, Q20, Q21, Q3: value BSZ42DN25NS3GATMA1 -> BSC600N25NS3GATMA1CT-ND
- Q2: footprint Package_TO_SOT_SMD:TO-263-7_TabPin8 -> td-hv:TO-263-7_TabPin8_GeneSiC
- Q6: value BD139 -> 2SC4382
- Q7: value BD140 -> 2SA1668
- R1, R10, R11, R15, R16, R17, R18, R2, R20, R21, R3, R4, R5, R7, R8, R82, R9: footprint Resistor_SMD:R_0805_2012Metric_Pad1.15x1.40mm_HandSolder -> Resistor_SMD:R_0805_2012Metric_Pad1.20x1.40mm_HandSolder
- R13, R14: value 1k -> 5.1k; footprint Resistor_SMD:R_0805_2012Metric_Pad1.15x1.40mm_HandSolder -> Resistor_SMD:R_0805_2012Metric
- R23, R24, R25, R26, R27, R28: footprint Resistor_SMD:R_1206_3216Metric_Pad1.42x1.75mm_HandSolder -> Resistor_SMD:R_1206_3216Metric_Pad1.30x1.75mm_HandSolder
- R29: value 1M -> 1k; footprint Resistor_SMD:R_0805_2012Metric_Pad1.15x1.40mm_HandSolder -> Resistor_SMD:R_0805_2012Metric_Pad1.20x1.40mm_HandSolder
- R30: value 100k -> 220k; footprint Resistor_SMD:R_0805_2012Metric_Pad1.15x1.40mm_HandSolder -> Resistor_SMD:R_0805_2012Metric_Pad1.20x1.40mm_HandSolder
- R31: value 49.9k -> 1k; footprint Resistor_SMD:R_0805_2012Metric_Pad1.15x1.40mm_HandSolder -> Resistor_SMD:R_0805_2012Metric_Pad1.20x1.40mm_HandSolder
- R6: value 10k -> 220k; footprint Resistor_SMD:R_0805_2012Metric_Pad1.15x1.40mm_HandSolder -> Resistor_SMD:R_0805_2012Metric_Pad1.20x1.40mm_HandSolder
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Connections:
- C17 pad 1: +12V -> +3.3VA
- C18 pad 1: +48V -> +3.3V
- C36 pad 1: +3V3 -> +3.3V
- C37 pad 1: +3V3 -> +3.3V
- C38 pad 1: +3V3 -> +3.3V
- C39 pad 1: +3V3 -> +3.3V
- C41 pad 1: +3V3 -> +3.3V
- C42 pad 1: +3V3 -> +3.3V
- C59 pad 1: HT -> B+H
- C8 pad 1: +3V3 -> +3.3VA
- D20 pad 2: HT -> B+H
- J13 pad 1: GND -> -12V
- J14 pad 1: GND -> unconnected-(J14-Pin_1-Pad1)
- J14 pad 2: +12V -> unconnected-(J14-Pin_2-Pad2)
- J16 pad 1: /rgb/red_vga -> +3.3V
- J16 pad 2: /rgb/green_vga -> +3.3V
- J16 pad 3: /rgb/blue_vga -> /uc/pd0
- J16 pad 4: GND -> /uc/pd1
- J16 pad 5: /rgb/hsync_vga -> /uc/pd2
- J16 pad 6: VSYNC_VGA_UC -> /uc/pd3
- J17 pad 1: +12V -> +48V
- J17 pad 2: /rgb/r_yoke -> GND
- J17 pad 3: /rgb/g_yoke -> unconnected-(J17-Pad3)
- J4 pad 1: +3V3 -> +3.3V
- J5 pad 1: /rgb/red_vga -> GND
- J5 pad 2: /rgb/green_vga -> +12V
- J5 pad 3: /rgb/blue_vga -> VGA_VSYNC
- J5 pad 4: unconnected-(J5-Pad4) -> SEP_HSYNC
- J5 pad 5: GND -> SEP_OE
- J5 pad 6: GND -> SEP_VSYNC
- J5 pad 7: GND -> LM1205_BLANK
- J7 pad 1: +12V -> +3.3V
- J7 pad 2: unconnected-(J7-Pin_2-Pad2) -> +3.3V
- J7 pad 3: GND -> /uc/pe0
- J7 pad 4: /rgb/b_yoke -> /uc/pe1
- J7 pad 5: GND -> /uc/pe2
- J7 pad 6: /rgb/g_yoke -> /uc/pe3
- J7 pad 7: GND -> /uc/pe4
- J7 pad 8: /rgb/r_yoke -> /uc/pe5
- J9 pad 1: GND -> +12V
- J9 pad 2: +6V -> GND
- Q1 pad 5: HT -> B+H
- R1 pad 1: +3V3 -> +3.3VA
- R13 pad 1: +3.3V -> Net-(J2-CC1)
- R13 pad 2: Net-(D2-A) -> GND
- R14 pad 1: +3.3V -> Net-(J2-CC2)
- R14 pad 2: Net-(R14-Pad2) -> GND
- R29 pad 1: +48V -> BPLUS_F_VOLTAGE
- R29 pad 2: BPLUS_EN -> GND
- R30 pad 1: BPLUS_EN -> B+C
- R30 pad 2: GND -> BPLUS_C_VOLTAGE
- R31 pad 1: Net-(U14-RT) -> BPLUS_C_VOLTAGE
- R6 pad 1: +3V3 -> B+F
- R6 pad 2: /uc/nrst -> BPLUS_F_VOLTAGE
- SW1 pad 1: Net-(R90-Pad1) -> +3.3V
- SW1 pad 2: Net-(R91-Pad1) -> BOOT0
- SW1 pad 3: Net-(R92-Pad1) -> (no net)
- SW1 pad 4: Net-(R93-Pad1) -> (no net)
- SW1 pad 5: GND -> (no net)
- SW1 pad 6: GND -> (no net)
- U11 pad 1: GND -> Net-(U11-IN-)
- U11 pad 4: GND -> unconnected-(U11-NC-Pad4)
- U11 pad 5: Net-(U11-SDA) -> V_CURRENT_CLASSD_AFTER
- U11 pad 6: Net-(U11-SCL) -> +3.3VA
- U11 pad 7: GND -> +3.3VA
- U11 pad 8: Net-(U11-VCC) -> Net-(J8-Pin_2)
- U2 pad 1: unconnected-(U2-VBAT-Pad1) -> /uc/pe2
- U2 pad 10: S2 -> unconnected-(U2-PF9-Pad10)
- U2 pad 11: S3 -> unconnected-(U2-PF10-Pad11)
- U2 pad 12: H_CURRENT -> /uc/16mhz
- U2 pad 13: /uc/hot_current_adc -> unconnected-(U2-PF1-Pad13)
- U2 pad 14: S_VOLTAGE -> /uc/nrst
- U2 pad 15: GND -> V_CURRENT_CLASSD
- U2 pad 16: +3V3 -> S1
- U2 pad 17: EHT_VOLTAGE_DIVIDER -> S2
- U2 pad 18: V_DAC -> S3
- U2 pad 19: BEAM_CURRENT -> unconnected-(U2-PF2-Pad19)
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Routing:
- removed copper zone on B.Cu, net GND
- removed copper zone on F.Cu, net GND
Other:
- board size 270 x 110 mm -> 260 x 104 mm
- board text added: "td-deflect v0.2 http://github.com/tdaede/td-rgb CERN-OHL-W 2023"
- board text removed: "+12V"
- board text removed: "+48V"
- board text removed: "-12V"
- board text removed: "B+ Supply"
- board text removed: "EHT"
- board text removed: "Heater"
- board text removed: "High Voltage"
- board text removed: "Horizontal"
- board text removed: "Neck"
- board text removed: "RGB"
- board text removed: "Serial"
- board text removed: "Vertical"
- board text removed: "b+ adj"
- board text removed: "sub contrast"
- board text removed: "td-deflect v0.1 http://github.com/tdaede/td-rgb cc-by-sa 4.0"

Commit message: more layout
Parts:
- removed J7: Conn_02x10_Odd_Even, Connector_IDC:IDC-Header_2x10_P2.54mm_Vertical
- added C20: 4.7uF, Capacitor_SMD:C_0805_2012Metric_Pad1.18x1.45mm_HandSolder, F.Cu at (-29.0, 95.0)
- added F4: Polyfuse, Fuse:Fuse_0805_2012Metric, F.Cu at (-10.1, 32.0)
- added J15: Conn_01x04_Pin, Connector_JST:JST_XH_B4B-XH-A_1x04_P2.50mm_Vertical, F.Cu at (-9.00, 36.5)
- added J22: Conn_02x05_Odd_Even, Connector_IDC:IDC-Header_2x05_P2.54mm_Vertical, F.Cu at (-20.9, 77.0)
- added J23: Conn_02x05_Odd_Even, Connector_IDC:IDC-Header_2x05_P2.54mm_Vertical, F.Cu at (1.54, 77.0)
- added TH1: Polyfuse, Fuse:Fuse_0805_2012Metric, F.Cu at (-20.6, 95.0)
- added U12: AP2204K-3.3, Package_TO_SOT_SMD:SOT-23-5, F.Cu at (-25.1, 95.0)
- added U13: TSOP43xx, OptoDevice:Vishay_MOLD-3Pin, F.Cu at (-34.7, 85.5)
- U23: value TPS70933 -> AP2204K-5.0
- U4: value TPS70933 -> AP2204K-3.3
- moved R25 16.6 mm to (175.0, 89.5), turned to -90 degrees
- moved R22 13.9 mm to (48.5, 74.5), turned to 0 degrees
- moved R26 12.4 mm to (165.0, 89.5), turned to -90 degrees
- moved D13 11.5 mm to (43.0, 85.8)
- moved R24 11.4 mm to (185.0, 89.5), turned to -90 degrees
- moved Q11 11.0 mm to (160.0, 89.4)
- moved R23 10.4 mm to (195.0, 89.5), turned to -90 degrees
- moved Q10 8.03 mm to (170.0, 89.5)
- moved C507 7.43 mm to (85.5, 93.0), turned to 180 degrees
- moved J6 6.40 mm to (-35.0, 70.2), turned to 180 degrees
- moved X1 5.92 mm to (-33.5, 50.1)
- moved R506 3.36 mm to (94.5, 93.0)
- moved R12 3.01 mm to (-28.0, 46.9)
- moved D6 2.53 mm to (19.4, 72.0)
- moved U28 2.53 mm to (24.5, 58.9)
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- renumbered C76 to C501, C77 to C502, C78 to C503, C79 to C504, C80 to C505, C81 to C506, C82 to C507, C83 to C508, C84 to C509, C85 to C510, C86 to C511, C87 to C512, D18 to D501, D19 to D502, J8 to J501, L11 to L501, L12 to L502, Q15 to Q501, Q16 to Q502, Q20 to Q503, Q21 to Q504, R80 to R501, R81 to R502, R82 to R503, R83 to R504, R84 to R505, R85 to R506, R94 to R507, R95 to R508, R107 to R509, U34 to U501, U35 to U502, U7 to U503, U11 to U504
Connections:
- C66 pad 1: +3.3VA -> +5V
- J5 pad 2: +12V -> /rgb/+12v_sync
- U2 pad 1: /uc/pe2 -> /uc/beeper
- U2 pad 19: unconnected-(U2-PF2-Pad19) -> /uc/ir
- U2 pad 2: /uc/pe3 -> /uc/sd_det
- U2 pad 3: /uc/pe4 -> /uc/sd_cs
- U2 pad 38: /uc/pe7 -> LM1205_BLANK
- U2 pad 39: /uc/pe8 -> /uc/btn_en1
- U2 pad 4: /uc/pe5 -> /uc/btn_enc
- U2 pad 40: /uc/pe9 -> /uc/btn_en2
- U2 pad 41: /uc/pe10 -> /uc/lcd_a0
- U2 pad 42: /uc/pe11 -> /uc/lcd_cs
- U2 pad 43: /uc/pe12 -> /uc/lcd_sck
- U2 pad 44: /uc/pe13 -> /uc/lcd_si
- U2 pad 45: /uc/pe14 -> /uc/lcd_so
- U2 pad 46: /uc/pe15 -> unconnected-(U2-PE15-Pad46)
- U2 pad 5: /uc/pe6 -> /uc/lcd_rst
- U2 pad 79: BIAS_LOAD -> /uc/tx2
- U2 pad 80: LM1205_BLANK -> /uc/rx2
- U2 pad 81: SEP_OE -> /uc/ws2811
- U2 pad 97: /uc/pe0 -> SEP_OE
- U2 pad 98: /uc/pe1 -> BIAS_LOAD
- U23 pad 5: +3.3VA -> +5V
Routing:
- net +12V: track 0.00 -> 440.0 mm, vias 0 -> 8
- net Net-(Q10-S): track 0.00 -> 277.1 mm, vias 0 -> 6
- net S0: track 0.00 -> 270.4 mm, vias 0 -> 2
- net S1: track 0.00 -> 269.1 mm, vias 0 -> 2
- net S3: track 0.00 -> 247.6 mm, vias 0 -> 2
- net S2: track 0.00 -> 245.4 mm, vias 0 -> 2
- net S_VOLTAGE: track 0.00 -> 224.2 mm, vias 0 -> 2
- net +3.3VA: track 0.00 -> 198.8 mm, vias 0 -> 7
- net +48V: track 0.00 -> 198.5 mm
- net +3.3V: track 0.00 -> 197.3 mm, vias 0 -> 7
- net PIN_LO: track 0.00 -> 176.5 mm, vias 0 -> 2
- net HOT_CURRENT: track 0.00 -> 173.5 mm, vias 0 -> 4
- net PIN_HI: track 0.00 -> 168.3 mm, vias 0 -> 2
- net -12V: track 0.00 -> 160.1 mm, vias 0 -> 6
- net B+F: track 0.00 -> 115.0 mm
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
Commit message: more stuff
Parts:
- added C21: 0.1uF, Capacitor_SMD:C_0805_2012Metric_Pad1.18x1.45mm_HandSolder, F.Cu at (-20.8, 68.2)
- J16: value Conn_02x10_Odd_Even -> Conn_02x6_Odd_Even; footprint Connector_IDC:IDC-Header_2x10_P2.54mm_Vertical -> Connector_IDC:IDC-Header_2x06_P2.54mm_Vertical
- moved J15 22.4 mm to (-18.2, 16.1)
- moved F4 18.9 mm to (-13.2, 13.4), turned to 0 degrees
- moved J16 4.02 mm to (3.20, 66.6)
- moved R14 3.38 mm to (-28.0, 38.2)
Connections:
- J16 pad 10: /uc/pd7 -> /uc/pd15
- J16 pad 11: /uc/pd8 -> GND
- J16 pad 12: /uc/pd9 -> GND
- J16 pad 3: /uc/pd0 -> /uc/pd8
- J16 pad 4: /uc/pd1 -> /uc/pd9
- J16 pad 5: /uc/pd2 -> /uc/pd10
- J16 pad 6: /uc/pd3 -> /uc/pd11
- J16 pad 7: /uc/pd4 -> /uc/pd12
- J16 pad 8: /uc/pd5 -> /uc/pd13
- J16 pad 9: /uc/pd6 -> /uc/pd14
Routing:
- net +48V: track 198.5 -> 428.4 mm, vias 0 -> 6
- net BPLUS_H_VOLTAGE: track 2.00 -> 165.4 mm, vias 0 -> 2
- net +12V: track 440.0 -> 594.2 mm, vias 8 -> 12
- net DEGAUSS: track 5.55 -> 154.0 mm
- net V_CURRENT_CLASSD_AFTER: track 0.00 -> 141.4 mm, vias 0 -> 4
- net HOT_IN: track 3.33 -> 139.8 mm
- net V_CURRENT_CLASSD: track 0.00 -> 129.0 mm, vias 0 -> 4
- net V_DAC: track 0.00 -> 123.5 mm, vias 0 -> 4
- net V_HI_1: track 0.00 -> 116.8 mm, vias 0 -> 2
- net V_LO_1: track 0.00 -> 115.7 mm, vias 0 -> 2
- net BPLUS_EN: track 40.0 -> 153.2 mm, vias 0 -> 2
- net V_HI_2: track 0.00 -> 103.9 mm, vias 0 -> 2
- net V_LO_2: track 0.00 -> 102.6 mm, vias 0 -> 2
- net BIAS_LOAD: track 0.00 -> 97.6 mm, vias 0 -> 2
- net V_EN: track 0.00 -> 82.4 mm, vias 0 -> 2
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- added copper zone on B.Cu, net GND
- added copper zone on F.Cu, net GND
Other:
- board size 260 x 104 mm -> 240 x 104 mm

Commit message: update pcb
Parts:
- C59: value 0.1uF -> 0.1uF 250V
- D17: value D_Zener -> 6.3V; footprint Diode_SMD:D_0805_2012Metric_Pad1.15x1.40mm_HandSolder -> Diode_SMD:D_SMA
- J17: footprint Connector_BarrelJack:BarrelJack_CLIFF_FC681465S_SMT_Horizontal -> Connector_BarrelJack:BarrelJack_Wuerth_6941xx301002
- L501, L502: value 100uF -> 100uH
- Q14, Q4, Q5: footprint Package_TO_SOT_SMD:SOT-223-3_TabPin2 -> Package_TO_SOT_SMD:SOT-223
- R110: footprint Resistor_THT:R_Radial_Power_L11.0mm_W7.0mm_P5.00mm -> Resistor_THT:R_Radial_Power_L13.0mm_W9.0mm_P5.00mm
- R56, R57: value R -> 2.2k; footprint Resistor_SMD:R_0805_2012Metric_Pad1.20x1.40mm_HandSolder -> Resistor_SMD:R_0805_2012Metric
- U23: value AP2204K-5.0 -> AP2205-5.0
- moved J17 6.08 mm to (-25.0, 18.0), turned to -90 degrees
- moved D17 1.60 mm to (21.8, 40.0)
- moved Q10 1.04 mm to (170.0, 88.5)
- moved Q8 1.04 mm to (190.0, 88.5)
- moved Q11 1.04 mm to (160.0, 88.4)
- moved Q9 1.04 mm to (180.0, 88.4)
- moved F3 0.50 mm to (19.8, 35.5)
- moved R17 0.20 mm to (40.0, 86.5)
- moved R18 0.20 mm to (37.0, 86.5)
- moved J16 0.20 mm to (3.00, 66.6)
Connections:
- net Net-(F2-Pad2) renamed /s_fuse
- net Net-(L1-Pad2) renamed /h_coil_1
- net Net-(L7-Pad2) renamed /h_coil_2
- net Net-(L8-Pad2) renamed /h_coil_3
Routing:
- net HOT_CURRENT: track 173.5 -> 177.1 mm
- net +48V: track 428.4 -> 426.2 mm
- net B+F: track 117.5 -> 119.5 mm
- net HEATER_EN: track 51.1 -> 52.1 mm
- net +12V: track 594.2 -> 595.1 mm
- net V_CURRENT_CLASSD: track 129.0 -> 128.1 mm
- net EHT_VOLTAGE_DIVIDER: track 60.8 -> 61.6 mm
- net virtual_ground: track 117.1 -> 116.6 mm
- net PIN_HI: track 168.5 -> 167.9 mm
- net Net-(C12-Pad1): track 50.1 -> 50.6 mm
- net +3.3V: track 219.9 -> 219.4 mm
- net VGA_VSYNC: vias 2 -> 1
- net GND: vias 91 -> 104
Other:
- board text added: "+/-12V"
- board text added: "24-48V"
- board text added: "B+ Cathode"
- board text added: "B+ Flyback"
- board text added: "B+ Horizontal"
- board text added: "BOOT0"
- board text added: "Degauss"
- board text added: "EXP1"
- board text added: "EXP2"
- board text added: "Flyback"
- board text added: "GPIO"
- board text added: "Heater"
- board text added: "High Voltage"
- board text added: "Horizontal"
- board text added: "I2C"
- board text added: "IR"
- board text added: "Neck Power"
- board text added: "Remote"
- board text added: "S-Capacitors"
- board text added: "Serial"
- board text added: "Sync"
- board text added: "USB"
- board text added: "Vertical (Class AB)"
- board text added: "Vertical (Class D)"
- board text added: "v.lin"
