File: td-deflect/td-deflect.kicad_pcb (KiCad board)
At the start: 2 copper layers, 240 x 104 mm, 206 parts, among them J1 Conn_01x05_Pin, J10 Conn_01x02_Male, J11 Conn_01x02_Male, J12 Conn_01x02_Male, J13 Conn_01x12_Socket, J14 Conn_01x12_Socket, J15 Conn_01x04_Pin, J16 Conn_02x6_Odd_Even, J17 Barrel_Jack, J18 Conn_01x02_Male, J19 Conn_01x08_Socket, J2 USB_C_Receptacle_USB2.0, J20 Conn_01x08_Socket, J21 Conn_01x08_Socket, J22 Conn_02x05_Odd_Even, J23 Conn_02x05_Odd_Even, J3 Conn_01x04_Male, J4 Conn_ARM_JTAG_SWD_10, J5 Conn_01x07_Male, J501 Conn_01x02_Male, J6 Conn_01x06_Male, J9 Conn_01x14, Q1 BSC600N25NS3GATMA1CT-ND, Q10 IPD50R380CE, Q11 IPD50R380CE, Q14 BCP56, Q2 G3R450MT17J, Q22 IPD50R380CE, Q3 BSC600N25NS3GATMA1CT-ND, Q4 BCP56, Q5 BCP53, Q501 BSC600N25NS3GATMA1CT-ND, Q502 BSC600N25NS3GATMA1CT-ND, Q503 BSC600N25NS3GATMA1CT-ND, Q504 BSC600N25NS3GATMA1CT-ND, Q6 2SC4382, Q7 2SA1668, Q8 IPD50R380CE, Q9 IPD50R380CE, SW1 SW_SPST, U1 MCP1416, U10 MIC4427, U12 AP2204K-3.3, U13 TSOP43xx, U2 STM32G474VETx, U23 AP2205-5.0, U24 INA181, U25 FM24C64B, U28 TL082, U3 INA181, U31 ASSR-1218, U38 MCP1416, U4 AP2204K-3.3, U5 TL082, U501 IRS2005S, U502 IRS2005S, U503 AD8417, U504 AD8417, U6 IRS2005S, U8 INA181, U9 MIC4427, X1 SG-8002CA

Commit message: shrink board a lot
Parts:
- removed C1, C18, C39, C5, C60, C7, C88: 0.1uF, Capacitor_SMD:C_0805_2012Metric_Pad1.18x1.45mm_HandSolder
- removed C12: 0.01uF, Capacitor_SMD:C_0805_2012Metric_Pad1.18x1.45mm_HandSolder
- removed C66: 4.7uF, Capacitor_SMD:C_0805_2012Metric_Pad1.18x1.45mm_HandSolder
- removed C69: 10uF 100V, Capacitor_SMD:CP_Elec_8x11.9
- removed C89: 0.47uF, Capacitor_THT:C_Rect_L18.0mm_W8.0mm_P15.00mm_FKS3_FKP3
- removed D12, D13, D14, D6, D7, D8: 1N4148W, Diode_SMD:D_SOD-123
- removed D20: ES1G-13-F, Diode_SMD:D_SMA
- removed F1, F2: Fuse, Fuse:Fuse_Schurter_UMT250
- removed HS1: Heatsink_Pad, td-deflect:c220-050-2ae
- removed J11: Conn_01x02_Male, td-deflect:sony_monitor_2p
- removed J12: Conn_01x02_Male, td-deflect:monitor_10_8_2p
- removed J22, J23: Conn_02x05_Odd_Even, Connector_IDC:IDC-Header_2x05_P2.54mm_Vertical
- removed L1, L7, L8, L9: 680uH, td-deflect:Murata_6000B
- removed L2: LTRIM, td-deflect:LIN-3509
- removed Q14, Q4: BCP56, Package_TO_SOT_SMD:SOT-223
- removed Q22: IPD50R380CE, Package_TO_SOT_SMD:TO-252-2
- removed Q5: BCP53, Package_TO_SOT_SMD:SOT-223
- removed Q6: 2SC4382, Package_TO_SOT_THT:TO-126-3_Vertical
- removed Q7: 2SA1668, Package_TO_SOT_THT:TO-126-3_Vertical
- removed R1, R108, R11, R3, R7, R8, R9: 10k, Resistor_SMD:R_0805_2012Metric_Pad1.20x1.40mm_HandSolder
- removed R109, R17, R18: 1, Resistor_SMD:R_0805_2012Metric_Pad1.20x1.40mm_HandSolder
- removed R110: 1k, Resistor_THT:R_Radial_Power_L13.0mm_W9.0mm_P5.00mm
- removed R15, R16, R70: 100, Resistor_SMD:R_0805_2012Metric_Pad1.20x1.40mm_HandSolder
- removed R20: 220k, Resistor_SMD:R_0805_2012Metric_Pad1.20x1.40mm_HandSolder
- removed R21, R71: 1k, Resistor_SMD:R_0805_2012Metric_Pad1.20x1.40mm_HandSolder
- removed R22: 1, Resistor_SMD:R_1210_3225Metric
- removed R68: 10, Resistor_SMD:R_0805_2012Metric_Pad1.20x1.40mm_HandSolder
- removed R69: 10k, Resistor_SMD:R_1210_3225Metric
- removed TH1: Polyfuse, Fuse:Fuse_0805_2012Metric
- removed TP3: TestPoint, TestPoint:TestPoint_Keystone_5015_Micro-Minature
- removed U12: AP2204K-3.3, Package_TO_SOT_SMD:SOT-23-5
- removed U13: TSOP43xx, OptoDevice:Vishay_MOLD-3Pin
- removed U23: AP2205-5.0, Package_TO_SOT_SMD:SOT-23-5
- removed U28: TL082, Package_SO:SOIC-8_3.9x4.9mm_P1.27mm
- removed U31: ASSR-1218, Package_SO:SO-4_4.4x4.3mm_P2.54mm
- removed U38: MCP1416, Package_TO_SOT_SMD:SOT-23-5
- added J7: Conn_01x02_Pin, td-deflect:monitor_10_8_2p, F.Cu at (126.8, 44.0)
- U4: value AP2204K-3.3 -> R-78B3.3-2.0; footprint Package_TO_SOT_SMD:SOT-23-5 -> Converter_DCDC:Converter_DCDC_RECOM_R-78B-2.0_THT
- U5: value TL082 -> R-78B3.3-2.0; footprint Package_SO:SOIC-8_3.9x4.9mm_P1.27mm -> Converter_DCDC:Converter_DCDC_RECOM_R-78B-2.0_THT
- moved C10 120.5 mm to (67.6, 91.9), turned to 180 degrees
- moved R23 118.9 mm to (76.4, 98.9), turned to 180 degrees
- moved U9 117.5 mm to (66.6, 87.5), turned to 0 degrees
- moved Q8 112.7 mm to (77.4, 94.0), turned to 0 degrees
- moved R24 108.6 mm to (76.4, 88.9), turned to 180 degrees
- moved C9 105.4 mm to (67.6, 74.2), turned to 180 degrees
- moved U10 103.7 mm to (66.7, 70.2), turned to 0 degrees
- moved Q9 102.6 mm to (77.5, 83.9), turned to 0 degrees
- moved R25 99.2 mm to (76.3, 78.9), turned to 180 degrees
- moved R28 97.8 mm to (67.1, 61.5), turned to 0 degrees
- moved R27 95.7 mm to (67.1, 57.5), turned to 180 degrees
- moved Q10 93.7 mm to (77.4, 73.9), turned to 0 degrees
- moved C13 92.2 mm to (99.9, 92.2), turned to 180 degrees
- moved R26 91.0 mm to (76.3, 68.9), turned to 180 degrees
- moved Q11 86.0 mm to (77.5, 63.9), turned to 0 degrees
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Connections:
- J10 pad 2: /h.ret -> /S_cap_top
- J2 pad A4: unconnected-(J2-VBUS-PadA4) -> unconnected-(J2-VBUS-PadA4)_2
- J2 pad A9: unconnected-(J2-VBUS-PadA4) -> unconnected-(J2-VBUS-PadA4)_3
- J2 pad B4: unconnected-(J2-VBUS-PadA4) -> unconnected-(J2-VBUS-PadA4)_1
- J5 pad 2: /rgb/+12v_sync -> +12V
- U2 pad 1: /uc/beeper -> unconnected-(U2-PE2-Pad1)
- U2 pad 2: /uc/sd_det -> unconnected-(U2-PE3-Pad2)
- U2 pad 26: V_DAC -> unconnected-(U2-PA4-Pad26)
- U2 pad 3: /uc/sd_cs -> unconnected-(U2-PE4-Pad3)
- U2 pad 39: /uc/btn_en1 -> unconnected-(U2-PE8-Pad39)
- U2 pad 4: /uc/btn_enc -> unconnected-(U2-PE5-Pad4)
- U2 pad 40: /uc/btn_en2 -> unconnected-(U2-PE9-Pad40)
- U2 pad 41: /uc/lcd_a0 -> unconnected-(U2-PE10-Pad41)
- U2 pad 42: /uc/lcd_cs -> unconnected-(U2-PE11-Pad42)
- U2 pad 43: /uc/lcd_sck -> unconnected-(U2-PE12-Pad43)
- U2 pad 44: /uc/lcd_si -> unconnected-(U2-PE13-Pad44)
- U2 pad 45: /uc/lcd_so -> unconnected-(U2-PE14-Pad45)
- U2 pad 5: /uc/lcd_rst -> unconnected-(U2-PE6-Pad5)
- U4 pad 3: +12V -> +3.3V
- U5 pad 1: virtual_ground -> +12V
- U5 pad 2: virtual_ground -> GND
- U5 pad 3: Net-(U5A-+) -> +3.3VA
Routing:
- net +12V: track 595.1 -> 51.4 mm, vias 12 -> 0
- net S1: track 276.0 -> 2.76 mm, vias 2 -> 0
- net S0: track 269.4 -> 2.31 mm, vias 2 -> 0
- net S3: track 246.4 -> 1.94 mm, vias 2 -> 0
- net S2: track 244.3 -> 1.49 mm, vias 2 -> 0
- net +48V: track 426.2 -> 195.0 mm, vias 6 -> 1
- net +3.3VA: track 234.4 -> 8.95 mm, vias 9 -> 2
- net S_VOLTAGE: track 225.7 -> 7.24 mm, vias 2 -> 0
- net +3.3V: track 219.4 -> 20.4 mm, vias 12 -> 1
- net Net-(Q10-S): track 268.4 -> 84.6 mm, vias 6 -> 4
- net HOT_CURRENT: track 177.1 -> 10.9 mm, vias 4 -> 0
- net BPLUS_H_VOLTAGE: track 165.7 -> 2.00 mm, vias 2 -> 0
- net DEGAUSS: track 154.0 -> 0.00 mm
- net -12V: track 160.1 -> 6.32 mm, vias 6 -> 0
- net PIN_LO: track 176.4 -> 29.7 mm, vias 2 -> 1
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- removed copper zone on B.Cu, net GND
- removed copper zone on F.Cu, net GND
Other:
- board size 240 x 104 mm -> 174 x 104 mm
- board text added: "td-deflect v0.3 http://github.com/tdaede/td-rgb CERN-OHL-W 2025"
- board text removed: "EXP1"
- board text removed: "EXP2"
- board text removed: "Sync"
- board text removed: "Vertical (Class AB)"
- board text removed: "td-deflect v0.2 http://github.com/tdaede/td-rgb CERN-OHL-W 2023"
- board text removed: "v.lin"

Commit message: stuff
Parts:
- removed F4: Polyfuse, Fuse:Fuse_0805_2012Metric
- removed H5, H6, H7, H8: MountingHole, MountingHole:MountingHole_3.2mm_M3
- removed J13, J14: Conn_01x12_Socket, Connector_PinSocket_2.54mm:PinSocket_1x12_P2.54mm_Vertical
- added C1: C, Capacitor_SMD:C_1210_3225Metric, F.Cu at (-1.50, 34.1)
- added C12: 22pF, Capacitor_SMD:C_0805_2012Metric, F.Cu at (6.40, 22.5)
- added C18: 0.1uF, Capacitor_SMD:C_0805_2012Metric_Pad1.18x1.45mm_HandSolder, F.Cu at (-25.0, 78.0)
- added C22: 22uF, Capacitor_SMD:C_0805_2012Metric, F.Cu at (23.5, 34.0)
- added C34: C, Capacitor_SMD:C_1210_3225Metric, F.Cu at (-1.15, 16.5)
- added C39: 0.1uF, Capacitor_SMD:C_0805_2012Metric_Pad1.18x1.45mm_HandSolder, F.Cu at (-9.00, 84.0)
- added C43: 0.1uF, Capacitor_SMD:C_0805_2012Metric, F.Cu at (5.55, 30.6)
- added C44: 0.033uF, Capacitor_SMD:C_0805_2012Metric, F.Cu at (6.50, 40.5)
- added C45: 22pF, Capacitor_SMD:C_0805_2012Metric, F.Cu at (3.05, 38.5)
- added C46: 22uF, Capacitor_SMD:C_0805_2012Metric, F.Cu at (23.4, 16.1)
- added C5: 0.033uF, Capacitor_SMD:C_0805_2012Metric, F.Cu at (2.85, 20.5)
- added C7: 0.1uF, Capacitor_SMD:C_0805_2012Metric, F.Cu at (5.55, 12.5)
- added D2: B220, Diode_SMD:D_SMB, F.Cu at (4.65, 27.1)
- added D5: B220, Diode_SMD:D_SMB, F.Cu at (4.65, 9.00)
- added L1: 47uH, Inductor_SMD:L_Bourns_SRR1260, F.Cu at (15.5, 31.1)
- added L5: 47uH, Inductor_SMD:L_Bourns_SRR1260, F.Cu at (15.5, 13.0)
- added R1: 20k, Resistor_SMD:R_0805_2012Metric, F.Cu at (1.44, 12.5)
- added R3: 15.4k, Resistor_SMD:R_0805_2012Metric, F.Cu at (6.35, 20.5)
- added R47: 20k, Resistor_SMD:R_0805_2012Metric, F.Cu at (0.41, 30.5)
- added R48: 15.4k, Resistor_SMD:R_0805_2012Metric, F.Cu at (6.50, 38.5)
- added R49: 11k, Resistor_SMD:R_0805_2012Metric, F.Cu at (23.4, 11.5)
- added R50: 1k, Resistor_SMD:R_0805_2012Metric, F.Cu at (23.4, 8.00)
- added R7: 11k, Resistor_SMD:R_0805_2012Metric, F.Cu at (23.5, 29.6)
- added R8: 1k, Resistor_SMD:R_0805_2012Metric, F.Cu at (23.5, 26.1)
- added U32: BD9G341AEFJ, Package_SO:SOIC-8-1EP_3.9x4.9mm_P1.27mm_EP2.41x3.3mm_ThermalVias, F.Cu at (4.53, 34.5)
- added U7: BD9G341AEFJ, Package_SO:SOIC-8-1EP_3.9x4.9mm_P1.27mm_EP2.41x3.3mm_ThermalVias, F.Cu at (4.60, 16.7)
- moved H10 65.1 mm to (51.0, 6.00)
- moved C42 45.0 mm to (-18.0, 40.0), turned to 0 degrees
- moved C20 44.5 mm to (-6.04, 40.0), turned to 0 degrees
- moved F3 14.3 mm to (32.2, 28.5)
- moved U5 10.9 mm to (-6.79, 29.5), turned to -90 degrees
- moved U4 10.6 mm to (-18.8, 29.5), turned to -90 degrees
- moved H11 10.0 mm to (51.0, 26.0)
- moved D17 8.28 mm to (29.0, 36.0), turned to -90 degrees
Routing:
- net +48V: track 195.0 -> 176.7 mm, vias 1 -> 0
- net +6V: track 13.3 -> 0.00 mm
- net /power_supply/heater: track 23.0 -> 13.8 mm
- net PIN_LO: track 29.7 -> 22.3 mm, vias 1 -> 0
- net -12V: track 6.32 -> 0.00 mm
- net PIN_HI: track 29.4 -> 23.6 mm, vias 1 -> 0
- net /uc/power_serial2: track 5.18 -> 0.00 mm
- net SEP_HSYNC: track 21.6 -> 16.7 mm
- net +3.3V: track 20.4 -> 16.7 mm, vias 1 -> 0
- net +12V: track 51.4 -> 48.9 mm
- net GND: vias 46 -> 39
Other:
- board text removed: "Heater"

Commit message: finish board
Parts:
- added C23: 0.1uF, Capacitor_SMD:C_0805_2012Metric_Pad1.18x1.45mm_HandSolder, F.Cu at (-13.5, 94.0)
- added C24: 0.1uF, Capacitor_SMD:C_0805_2012Metric_Pad1.18x1.45mm_HandSolder, F.Cu at (-11.0, 94.0)
- added C25: 0.1uF, Capacitor_SMD:C_0805_2012Metric_Pad1.18x1.45mm_HandSolder, F.Cu at (-8.53, 94.0)
- added C26: 0.1uF, Capacitor_SMD:C_0805_2012Metric_Pad1.18x1.45mm_HandSolder, F.Cu at (-6.03, 94.0)
- added C27: 0.1uF, Capacitor_SMD:C_0805_2012Metric, F.Cu at (10.9, 71.0)
- added F1: Polyfuse, Fuse:Fuse_0805_2012Metric, F.Cu at (-16.0, 94.1)
- added F4: Polyfuse, Fuse:Fuse_0805_2012Metric, F.Cu at (-27.7, 74.2)
- added J11: Conn_01x06_Pin, Connector_JST:JST_XH_B6B-XH-A_1x06_P2.50mm_Vertical, F.Cu at (-16.0, 99.5)
- added J8: Conn_01x03_Pin, Connector_JST:JST_XH_B3B-XH-A_1x03_P2.50mm_Vertical, F.Cu at (-18.0, 18.5)
- added R11: 1k, Resistor_SMD:R_0805_2012Metric, F.Cu at (5.41, 74.0)
- added R9: 1k, Resistor_SMD:R_0805_2012Metric, F.Cu at (9.00, 74.0)
- C507, C508: footprint Capacitor_SMD:C_0805_2012Metric_Pad1.18x1.45mm_HandSolder -> Capacitor_SMD:C_Elec_6.3x7.7
- C509, C510: footprint Capacitor_SMD:C_0805_2012Metric_Pad1.18x1.45mm_HandSolder -> Capacitor_SMD:C_Elec_6.3x5.8
- TP1, TP2: footprint TestPoint:TestPoint_Keystone_5015_Micro-Minature -> TestPoint:TestPoint_Keystone_5015_Micro_Mini
- moved TP2 104.3 mm to (106.8, 66.5)
- moved C12 18.3 mm to (7.05, 40.8)
- moved C5 18.3 mm to (3.50, 38.8)
- moved R3 18.3 mm to (7.00, 38.8)
- moved C43 18.1 mm to (6.55, 12.5)
- moved C7 18.0 mm to (6.55, 30.5)
- moved R1 18.0 mm to (1.00, 30.5)
- moved R47 18.0 mm to (0.59, 12.5)
- moved U32 17.8 mm to (4.53, 16.7)
- moved U7 17.8 mm to (4.80, 34.5)
- moved C44 17.5 mm to (7.00, 23.0)
- moved C45 17.5 mm to (3.55, 21.0)
- moved R48 17.5 mm to (7.00, 21.0), turned to 0 degrees
- moved R508 13.8 mm to (52.0, 101.0), turned to 0 degrees
- moved C509 7.35 mm to (55.0, 93.0)
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Connections:
- C43 pad 2: /power_supply/SW -> /power_supply/SW_48V
- C7 pad 2: /power_supply/SW -> /power_supply/SW_12V
- D2 pad 1: /power_supply/SW -> /power_supply/SW_12V
- D5 pad 1: /power_supply/SW -> /power_supply/SW_48V
- J2 pad A4: unconnected-(J2-VBUS-PadA4)_2 -> VBUS
- J2 pad A9: unconnected-(J2-VBUS-PadA4)_3 -> VBUS
- J2 pad B4: unconnected-(J2-VBUS-PadA4)_1 -> VBUS
- J2 pad B9: unconnected-(J2-VBUS-PadA4) -> VBUS
- L1 pad 1: /power_supply/SW -> /power_supply/SW_12V
- L5 pad 1: /power_supply/SW -> /power_supply/SW_48V
- U2 pad 19: /uc/ir -> unconnected-(U2-PF2-Pad19)
- U2 pad 39: unconnected-(U2-PE8-Pad39) -> /uc/hsize_pot
- U2 pad 40: unconnected-(U2-PE9-Pad40) -> /uc/hpos_pot
- U2 pad 41: unconnected-(U2-PE10-Pad41) -> /uc/vsize_pot
- U2 pad 42: unconnected-(U2-PE11-Pad42) -> /uc/vpos_pot
- U2 pad 81: /uc/ws2811 -> unconnected-(U2-PC12-Pad81)
- U2 pad 82: /uc/pd0 -> unconnected-(U2-PD0-Pad82)
- U2 pad 83: /uc/pd1 -> unconnected-(U2-PD1-Pad83)
- U2 pad 84: /uc/pd2 -> unconnected-(U2-PD2-Pad84)
- U2 pad 85: /uc/pd3 -> unconnected-(U2-PD3-Pad85)
- U2 pad 86: /uc/pd4 -> unconnected-(U2-PD4-Pad86)
- U2 pad 87: /uc/pd5 -> unconnected-(U2-PD5-Pad87)
- U2 pad 88: /uc/pd6 -> unconnected-(U2-PD6-Pad88)
- U2 pad 89: /uc/pd7 -> unconnected-(U2-PD7-Pad89)
- U32 pad 1: /power_supply/SW -> /power_supply/SW_48V
- U7 pad 1: /power_supply/SW -> /power_supply/SW_12V
Routing:
- net +3.3VA: track 8.95 -> 181.1 mm, vias 2 -> 7
- net BPLUS_H_VOLTAGE: track 2.00 -> 156.6 mm, vias 0 -> 2
- net S2: track 1.49 -> 143.4 mm, vias 0 -> 2
- net S3: track 1.94 -> 142.2 mm, vias 0 -> 2
- net HOT_CURRENT: track 10.9 -> 151.0 mm, vias 0 -> 2
- net PIN_LO: track 22.3 -> 157.9 mm, vias 0 -> 2
- net S0: track 2.31 -> 137.6 mm, vias 0 -> 2
- net HOT_IN: track 0.00 -> 132.7 mm
- net PIN_HI: track 23.6 -> 149.3 mm, vias 0 -> 2
- net S1: track 2.76 -> 127.2 mm, vias 0 -> 2
- net BPLUS_EN: track 40.0 -> 151.1 mm, vias 0 -> 5
- net S_VOLTAGE: track 7.24 -> 108.5 mm, vias 0 -> 2
- net +48V: track 176.7 -> 269.4 mm, vias 0 -> 5
- net +12V: track 48.9 -> 134.6 mm, vias 0 -> 8
- net Net-(Q10-S): track 84.6 -> 169.5 mm, vias 4 -> 6
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- added copper zone on In2.Cu, net +12V
- added copper zone on In2.Cu, net +3.3V
- added copper zone on B.Cu, net GND
- added copper zone on F.Cu, net GND
- added copper zone on In1.Cu, net GND
Other:
- copper layers 2 -> 4
- board text removed: "IR"

Commit message: Update td-deflect to 0.3
Parts:
- added R15: 20k, Resistor_SMD:R_0805_2012Metric_Pad1.20x1.40mm_HandSolder, F.Cu at (-15.0, 14.0)
- added R16: 1k, Resistor_SMD:R_0805_2012Metric_Pad1.20x1.40mm_HandSolder, F.Cu at (-20.0, 14.0)
- C20, C42, C59: footprint Capacitor_SMD:C_0805_2012Metric_Pad1.18x1.45mm_HandSolder -> Capacitor_SMD:C_1206_3216Metric
- F4: footprint Fuse:Fuse_0805_2012Metric -> Fuse:Fuse_1206_3216Metric
- moved C59 0.25 mm to (114.8, 12.5)
Connections:
- U2 pad 26: unconnected-(U2-PA4-Pad26) -> INPUT_VOLTAGE
Routing:
- net INPUT_VOLTAGE: track 0.00 -> 84.6 mm, vias 0 -> 4
- net +48V: track 269.4 -> 274.2 mm
- net /h.out: track 52.2 -> 53.7 mm
- net +12V: track 134.6 -> 136.0 mm
- net GND: track 60.3 -> 61.4 mm, vias 74 -> 97
- net +3.3V: track 44.4 -> 45.4 mm
- net B+F: track 87.6 -> 87.0 mm
- net DEGAUSS: track 58.2 -> 58.7 mm
Other:
- board text added: "+12v"
- board text added: "+3.3v"
- board text added: "+in"
- board text added: "+out"
- board text added: "Analog Geometry Remote"
- board text added: "Hpos"
- board text added: "Hsize"
- board text added: "Inductor Board"
- board text added: "RGB / Sync"
- board text added: "Retrace Capacitor"
- board text added: "Vpos"
- board text added: "Vsize"
- board text added: "b+c"
- board text added: "b+f"
- board text added: "beam_current"
- board text added: "bias_load"
- board text added: "blank"
- board text added: "degauss"
- board text added: "eht_flyback_current"
- board text added: "eht_flyback_voltage"
- board text added: "eht_pwm"
- board text added: "eht_tertiary_winding"
- board text added: "eht_voltage_divider"
- board text added: "en"
- board text added: "gain_load"
- board text added: "gnd"
- board text added: "h"
- board text added: "heater"
- board text added: "hv_Hi"
- board text added: "hv_lo"
- board text added: "hv_protect"
- board text added: "rx"
- board text added: "scl"
- board text added: "sda"
- board text added: "sep_hsync"
- board text added: "sep_oe"
- board text added: "sep_vsync"
- board text added: "td-deflect v0.3 http://github.com/tdaede/td-crt CERN-OHL-W 2025"
- board text added: "tx"
- board text added: "vga_vsync"
- board text removed: "td-deflect v0.3 http://github.com/tdaede/td-rgb CERN-OHL-W 2025"
