File: td-deflect/rgb.kicad_sch (KiCad schematic)
At the start: 83 parts, among them J16 Conn_01x06_Male, J17 Conn_01x06_Male, J5 DB15_Female_HighDensity, J7 Conn_01x08_Male, Q14 BC847, Q15 BC847, Q16 BC847, SW1 SW_DIP_x04, U11 24LC08, U18 M51387P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

Commit message: add todos to schematic
Other:
- note added: "todo: replace this chip entirely lol"
Changed lines of the file:
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@@
     (stroke (width 0) (type solid) (color 0 0 0 0))
+  )
+  (text "todo: replace this chip entirely lol" (at 83.82 124.46 0)
+    (effects (font (size 1.27 1.27)) (justify left bottom))
   )
   (label "red_vga" (at 25.4 83.82 180)
