File: td-180v/td-180v.kicad_pcb (KiCad board)
At the start: 2 copper layers, 73 x 28 mm, 21 parts, among them J18 Conn_01x02_Male, J2 Conn_01x02_Male, Q1 IPD50R3K0CE, U14 LT3758AEMSE

Commit message: 180v fixes
Parts:
- removed J18, J2: Conn_01x02_Male, Connector_Phoenix_MSTB:PhoenixContact_MSTBVA_2,5_2-G_1x02_P5.00mm_Vertical
- added H1: MountingHole, MountingHole:MountingHole_3.2mm_M3, F.Cu at (214.0, 130.0)
- added H2: MountingHole, MountingHole:MountingHole_3.2mm_M3, F.Cu at (130.0, 130.0)
- added J1: Conn_01x05_Male, Connector_JST:JST_XH_S5B-XH-A_1x05_P2.50mm_Horizontal, F.Cu at (207.0, 121.0)
- added J3: Conn_01x05_Male, Connector_JST:JST_XH_B5B-XH-A_1x05_P2.50mm_Vertical, B.Cu at (197.0, 121.0)
- D1: value BAS21 -> C3D02060E; footprint Package_TO_SOT_SMD:SOT-23 -> Package_TO_SOT_SMD:TO-252-2_TabPin1
- moved C25 17.1 mm to (196.0, 111.0)
- moved D1 10.6 mm to (168.6, 128.0)
Connections:
- D1 pad 1: Net-(D1-Pad1) -> HT
- L3 pad 2: Net-(D1-Pad1) -> Net-(D1-Pad2)
- Q1 pad 2: Net-(D1-Pad1) -> Net-(D1-Pad2)
Other:
- board size 73 x 28 mm -> 92 x 30 mm

Commit message: more fixes
Parts:
- added C1: 22uF, Capacitor_THT:CP_Radial_D8.0mm_P3.50mm, F.Cu at (203.0, 129.0)
- added JP1: SolderJumper_2_Open, Jumper:SolderJumper-2_P1.3mm_Open_Pad1.0x1.5mm, F.Cu at (202.0, 118.0)
- added JP2: SolderJumper_2_Bridged, Jumper:SolderJumper-2_P1.3mm_Bridged_Pad1.0x1.5mm, F.Cu at (202.0, 113.0)
- added JP3: SolderJumper_2_Bridged, Jumper:SolderJumper-2_P1.3mm_Bridged_Pad1.0x1.5mm, F.Cu at (202.0, 121.0)
- added R1: R, Resistor_SMD:R_0805_2012Metric_Pad1.20x1.40mm_HandSolder, F.Cu at (183.0, 127.0)
- added R2: R, Resistor_SMD:R_0805_2012Metric_Pad1.20x1.40mm_HandSolder, F.Cu at (183.0, 130.0)
- added U1: AMS1117CD, Package_TO_SOT_SMD:TO-252-3_TabPin2, F.Cu at (191.7, 129.2)
- moved R30 17.7 mm to (164.0, 106.0), turned to 0 degrees
- moved D1 3.21 mm to (168.4, 124.8)
- moved RV1 0.80 mm to (138.5, 112.8)
- moved R29 0.15 mm to (164.0, 108.0)
Connections:
- C18 pad 1: +48V -> +12V
- C25 pad 1: HT -> /180v_out
- C26 pad 1: HT -> /180v_out
- D1 pad 1: HT -> /180v_out
- J1 pad 2: Net-(J1-Pad2) -> +12V
- J1 pad 4: /heater -> /heater_in
- J3 pad 1: Net-(J3-Pad1) -> /180v_out
- J3 pad 3: Net-(J3-Pad3) -> GND
- J3 pad 4: Net-(J3-Pad4) -> /heater_out
- J3 pad 5: Net-(J3-Pad5) -> /g1
- L3 pad 1: +48V -> Net-(JP1-Pad2)
- R29 pad 1: +48V -> +12V
- R39 pad 1: HT -> /180v_out
- U14 pad 10: +48V -> +12V
Routing:
- net +12V: track 0.00 -> 101.6 mm
- net Net-(R39-Pad2): track 0.00 -> 56.7 mm
- net /180v_out: track 0.00 -> 54.4 mm, vias 0 -> 1
- net /heater_out: track 0.00 -> 48.3 mm, vias 0 -> 1
- net Net-(JP1-Pad2): track 0.00 -> 33.6 mm
- net /g1: track 0.00 -> 27.1 mm, vias 0 -> 1
- net Net-(D1-Pad2): track 0.00 -> 21.7 mm
- net Net-(RV1-Pad2): track 0.00 -> 14.8 mm
- net Net-(R29-Pad2): track 0.00 -> 14.5 mm
- net Net-(R40-Pad1): track 0.00 -> 8.63 mm
- net Net-(Q1-Pad3): track 0.00 -> 8.47 mm
- net Net-(R1-Pad1): track 0.00 -> 7.35 mm
- net Net-(C21-Pad1): track 0.00 -> 5.59 mm
- net Net-(C22-Pad1): track 0.00 -> 5.12 mm
- net /heater_in: track 0.00 -> 4.56 mm
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- added copper zone on B.Cu, net GND
- added copper zone on F.Cu, net GND
Other:
- board text added: "td-180v v1.0 2021 CC0 https://github.com/tdaede/td-crt"
