File: td-180v/td-180v.sch (KiCad schematic (older format))
At the start: 21 parts, among them J18 Conn_01x02_Male, J2 Conn_01x02_Male, Q1 IPD50R3K0CE, U14 LT3758AEMSE

Commit message: 180v fixes
Parts:
- removed D1: BAS21, Package_TO_SOT_SMD:SOT-23, symbol Diode:BAS21
- removed J18, J2: Conn_01x02_Male, Connector_Phoenix_MSTB:PhoenixContact_MSTBVA_2,5_2-G_1x02_P5.00mm_Vertical, symbol Connector:Conn_01x02_Male
- added D1: C3D02060E, Package_TO_SOT_SMD:TO-252-2_TabPin1, symbol Diode:C3D02060E
- added H1, H2: MountingHole, MountingHole:MountingHole_3.2mm_M3, symbol Mechanical:MountingHole
- added J1: Conn_01x05_Male, Connector_JST:JST_XH_S5B-XH-A_1x05_P2.50mm_Horizontal, symbol Connector:Conn_01x05_Male
- added J3: Conn_01x05_Male, Connector_JST:JST_XH_B5B-XH-A_1x05_P2.50mm_Vertical, symbol Connector:Conn_01x05_Male
Connections:
- net labels added: 160v_in, g1, heater
- no-connect marks 0 -> 1
Changed lines of the file:
@@
 Comment4 ""
 $EndDescr
-$Comp
-L Connector:Conn_01x02_Male J18
-U 1 1 5DC2E1D1
-P 8000 1225
-F 0 "J18" H 8108 1406 50  0000 C CNN
-F 1 "Conn_01x02_Male" H 8108 1315 50  0000 C CNN
-F 2 "Connector_Phoenix_MSTB:PhoenixContact_MSTBVA_2,5_2-G_1x02_P5.00mm_Vertical" H 8000 1225 50  0001 C CNN
-F 3 "277-1150-ND " H 8000 1225 50  0001 C CNN
-F 4 "277-1150-ND " H 8000 1225 50  0001 C CNN "Digikey"
-	1    8000 1225
-	-1   0    0    1
-$EndComp
-$Comp
-L power:GND #PWR0119
-U 1 1 5DC2E1F0
-P 7800 1225
-F 0 "#PWR0119" H 7800 975 50  0001 C CNN
-F 1 "GND" H 7805 1052 50  0000 C CNN
-F 2 "" H 7800 1225 50  0001 C CNN
-F 3 "" H 7800 1225 50  0001 C CNN
-	1    7800 1225
-	1    0    0    -1
-$EndComp
-$Comp
-L power:+48V #PWR0181
-U 1 1 5DC2E736
-P 7450 1125
-F 0 "#PWR0181" H 7450 975 50  0001 C CNN
-F 1 "+48V" H 7465 1298 50  0000 C CNN
-F 2 "" H 7450 1125 50  0001 C CNN
-F 3 "" H 7450 1125 50  0001 C CNN
-	1    7450 1125
-	1    0    0    -1
-$EndComp
-$Comp
-L power:PWR_FLAG #FLG0104
-U 1 1 5DC2EB43
-P 7800 1125
-F 0 "#FLG0104" H 7800 1200 50  0001 C CNN
-F 1 "PWR_FLAG" H 7800 1298 50  0000 C CNN
-F 2 "" H 7800 1125 50  0001 C CNN
-F 3 "~" H 7800 1125 50  0001 C CNN
-	1    7800 1125
-	1    0    0    -1
-$EndComp
-Connection ~ 7800 1125
-Wire Wire Line
-	7450 1125 7800 1125
-$Comp
-L power:GND #PWR0102
-U 1 1 5C3770B4
-P 6200 1300
-F 0 "#PWR0102" H 6200 1050 50  0001 C CNN
-F 1 "GND" H 6205 1127 50  0000 C CNN
-F 2 "" H 6200 1300 50  0001 C CNN
-F 3 "" H 6200 1300 50  0001 C CNN
-	1    6200 1300
-	1    0    0    -1
-$EndComp
-$Comp
-L power:HT #PWR0101
-U 1 1 5C3769B2
-P 6200 1200
-F 0 "#PWR0101" H 6200 1320 50  0001 C CNN
-F 1 "HT" H 6220 1343 50  0000 C CNN
-F 2 "" H 6200 1200 50  0001 C CNN
-F 3 "" H 6200 1200 50  0001 C CNN
-	1    6200 1200
-	1    0    0    -1
-$EndComp
-$Comp
-L Connector:Conn_01x02_Male J2
-U 1 1 5C375524
-P 6400 1300
-F 0 "J2" H 6508 1481 50  0000 C CNN
-F 1 "Conn_01x02_Male" H 6508 1390 50  0000 C CNN
-F 2 "Connector_Phoenix_MSTB:PhoenixContact_MSTBVA_2,5_2-G_1x02_P5.00mm_Vertical" H 6400 1300 50  0001 C CNN
-F 3 "277-1150-ND " H 6400 1300 50  0001 C CNN
-F 4 "277-1150-ND " H 6400 1300 50  0001 C CNN "Digikey"
-	1    6400 1300
-	-1   0    0    1
-$EndComp
 Connection ~ 4100 1650
 $Comp
@@
 	1    4000 1450
 	1    0    0    -1
-$EndComp
-$Comp
-L Diode:BAS21 D1
-U 1 1 60CCF117
-P 4400 1150
-F 0 "D1" H 4400 933 50  0000 C CNN
-F 1 "BAS21" H 4400 1024 50  0000 C CNN
-F 2 "Package_TO_SOT_SMD:SOT-23" H 4400 975 50  0001 C CNN
-F 3 "https://www.diodes.com/assets/Datasheets/Ds12004.pdf" H 4400 1150 50  0001 C CNN
-	1    4400 1150
-	-1   0    0    1
 $EndComp
 $Comp
@@
 	0    -1   -1   0
 $EndComp
-Entry Wire Line
-	4250 1600 4350 1700
+$Comp
+L Diode:C3D02060E D1
+U 1 1 60E13622
+P 4400 1150
+F 0 "D1" H 4400 933 50  0000 C CNN
+F 1 "C3D02060E" H 4400 1024 50  0000 C CNN
+F 2 "Package_TO_SOT_SMD:TO-252-2_TabPin1" H 4400 975 50  0001 C CNN
+F 3 "https://www.wolfspeed.com/media/downloads/116/C3D02060E.pdf" H 4400 1150 50  0001 C CNN
+	1    4400 1150
+	-1   0    0    1
+$EndComp
+$Comp
+L Mechanical:MountingHole H1
+U 1 1 60E164B2
+P 5500 3050
+F 0 "H1" H 5600 3096 50  0000 L CNN
+F 1 "MountingHole" H 5600 3005 50  0000 L CNN
+F 2 "MountingHole:MountingHole_3.2mm_M3" H 5500 3050 50  0001 C CNN
+F 3 "~" H 5500 3050 50  0001 C CNN
+	1    5500 3050
+	1    0    0    -1
+$EndComp
+$Comp
+L Mechanical:MountingHole H2
+U 1 1 60E16BE7
+P 6300 3000
+F 0 "H2" H 6400 3046 50  0000 L CNN
+F 1 "MountingHole" H 6400 2955 50  0000 L CNN
+F 2 "MountingHole:MountingHole_3.2mm_M3" H 6300 3000 50  0001 C CNN
+F 3 "~" H 6300 3000 50  0001 C CNN
+	1    6300 3000
+	1    0    0    -1
+$EndComp
+$Comp
+L Connector:Conn_01x05_Male J1
+U 1 1 60E1A185
+P 2650 3150
+F 0 "J1" H 2758 3531 50  0000 C CNN
+F 1 "Conn_01x05_Male" H 2758 3440 50  0000 C CNN
+F 2 "Connector_JST:JST_XH_S5B-XH-A_1x05_P2.50mm_Horizontal" H 2650 3150 50  0001 C CNN
+F 3 "~" H 2650 3150 50  0001 C CNN
+	1    2650 3150
+	1    0    0    -1
+$EndComp
+Text Label 2850 2950 0    50   ~ 0
+160v_in
+NoConn ~ 2850 3050
+$Comp
+L power:GND #PWR0103
+U 1 1 60E1BD74
+P 3250 3150
+F 0 "#PWR0103" H 3250 2900 50  0001 C CNN
+F 1 "GND" H 3255 2977 50  0000 C CNN
+F 2 "" H 3250 3150 50  0001 C CNN
+F 3 "" H 3250 3150 50  0001 C CNN
+	1    3250 3150
+	1    0    0    -1
+$EndComp
+Wire Wire Line
+	3250 3150 2850 3150
+Text Label 2850 3350 0    50   ~ 0
+g1
+Text Label 2850 3250 0    50   ~ 0
+heater
+$Comp
+L Connector:Conn_01x05_Male J3
+U 1 1 60E1DC4D
+P 4000 3150
+F 0 "J3" H 4108 3531 50  0000 C CNN
+F 1 "Conn_01x05_Male" H 4108 3440 50  0000 C CNN
+F 2 "Connector_JST:JST_XH_B5B-XH-A_1x05_P2.50mm_Vertical" H 4000 3150 50  0001 C CNN
+F 3 "~" H 4000 3150 50  0001 C CNN
+	1    4000 3150
+	1    0    0    -1
+$EndComp
 $EndSCHEMATC

Commit message: more fixes
Parts:
- added C1: 22uF, Capacitor_THT:CP_Radial_D8.0mm_P3.50mm, symbol Device:C
- added JP1: SolderJumper_2_Open, Jumper:SolderJumper-2_P1.3mm_Open_Pad1.0x1.5mm, symbol Jumper:SolderJumper_2_Open
- added JP2, JP3: SolderJumper_2_Bridged, Jumper:SolderJumper-2_P1.3mm_Bridged_Pad1.0x1.5mm, symbol Jumper:SolderJumper_2_Bridged
- added R1, R2: R, Resistor_SMD:R_0805_2012Metric_Pad1.20x1.40mm_HandSolder, symbol Device:R
- added U1: AMS1117CD, Package_TO_SOT_SMD:TO-252-3_TabPin2, symbol Regulator_Linear:AMS1117CD
Connections:
- net labels added: +12V, 180v_out, heater_in, heater_out
- net labels removed: +48V, HT, heater
- wire segments 53 -> 64
Other:
- moved on the sheet: C18, C20, C21, C22, C23, C25, C26, D1, H1, H2, J1, J3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

Commit message: add td-hv
Parts:
- C26: Digikey 1276-3084-1-ND -> 732-12118-1-ND
- D1: Digikey (none) -> C3D02060E-ND
- J1: Digikey (none) -> 455-2242-ND
- U1: Digikey (none) -> NCP1117DT33T5GOSCT-ND
Changed lines of the file:
@@
 F 3 "~" H 7000 3050 50  0001 C CNN
 F 4 "200V" H 7000 3050 50  0001 C CNN "Voltage"
-F 5 "1276-3084-1-ND " H 7000 3050 50  0001 C CNN "Digikey"
+F 5 "732-12118-1-ND" H 7000 3050 50  0001 C CNN "Digikey"
 	1    7000 3050
 	1    0    0    -1
@@
 F 2 "Package_TO_SOT_SMD:TO-252-2_TabPin1" H 5750 2225 50  0001 C CNN
 F 3 "https://www.wolfspeed.com/media/downloads/116/C3D02060E.pdf" H 5750 2400 50  0001 C CNN
+F 4 "C3D02060E-ND" H 5750 2400 50  0001 C CNN "Digikey"
 	1    5750 2400
 	-1   0    0    1
@@
 F 2 "Connector_JST:JST_XH_S5B-XH-A_1x05_P2.50mm_Horizontal" H 4000 4400 50  0001 C CNN
 F 3 "~" H 4000 4400 50  0001 C CNN
+F 4 "455-2242-ND" H 4000 4400 50  0001 C CNN "Digikey"
 	1    4000 4400
 	1    0    0    -1
@@
 F 2 "Package_TO_SOT_SMD:TO-252-3_TabPin2" H 2600 5350 50  0001 C CNN
 F 3 "http://www.advanced-monolithic.com/pdf/ds1117.pdf" H 2700 4900 50  0001 C CNN
+F 4 "NCP1117DT33T5GOSCT-ND" H 2600 5150 50  0001 C CNN "Digikey"
 	1    2600 5150
 	1    0    0    -1
