File: td-hv/td-hv.sch (KiCad schematic (older format))
At the start: 26 parts, among them J1 Conn_01x06_Male, Q1 IMBF170R450M1XTMA1, U1 UCC3801, U2 TL081, U3 LM2903

Commit message: footprints
Parts:
- C1, C2, C3, C5, C6: footprint (none) -> Capacitor_SMD:C_0805_2012Metric
- C4: footprint (none) -> Capacitor_SMD:C_Elec_4x5.4
- D2, D3: footprint (none) -> LED_SMD:LED_0805_2012Metric_Castellated
- F1: footprint (none) -> Fuse:Fuseholder_Littelfuse_Nano2_157x
- J1: footprint (none) -> Connector_JST:JST_XH_B6B-XH-AM_1x06_P2.50mm_Vertical
- L1: footprint (none) -> td-hv:053X0528-001
- R1, R2, R3, R4, R5, R6, R7, R8: footprint (none) -> Resistor_SMD:R_0805_2012Metric
- RV1, RV2: footprint (none) -> Potentiometer_SMD:Potentiometer_Bourns_3314G_Vertical
- U1, U3: footprint (none) -> Package_SO:SOIC-8_3.9x4.9mm_P1.27mm
- U2: footprint (none) -> Package_TO_SOT_SMD:SOT-23-6
Changed lines of the file:
@@
 F 0 "L1" H 5750 3645 50  0000 C CNN
 F 1 "053X0528-001" H 5750 3554 50  0000 C CNN
-F 2 "" V 5750 3350 50  0001 C CNN
+F 2 "td-hv:053X0528-001" V 5750 3350 50  0001 C CNN
 F 3 "~" V 5750 3350 50  0001 C CNN
 	1    5750 3300
@@
 F 0 "R4" H 4570 4146 50  0000 L CNN
 F 1 "R" H 4570 4055 50  0000 L CNN
-F 2 "" V 4430 4100 50  0001 C CNN
+F 2 "Resistor_SMD:R_0805_2012Metric" V 4430 4100 50  0001 C CNN
 F 3 "~" H 4500 4100 50  0001 C CNN
 	1    4500 4100
@@
 F 0 "C5" H 5065 2946 50  0000 L CNN
 F 1 "C" H 5065 2855 50  0000 L CNN
-F 2 "" H 4988 2750 50  0001 C CNN
+F 2 "Capacitor_SMD:C_0805_2012Metric" H 4988 2750 50  0001 C CNN
 F 3 "~" H 4950 2900 50  0001 C CNN
 	1    4950 2900
@@
 F 0 "C4" H 4718 2946 50  0000 L CNN
 F 1 "CP" H 4718 2855 50  0000 L CNN
-F 2 "" H 4638 2750 50  0001 C CNN
+F 2 "Capacitor_SMD:C_Elec_4x5.4" H 4638 2750 50  0001 C CNN
 F 3 "~" H 4600 2900 50  0001 C CNN
 	1    4600 2900
@@
 F 0 "F1" V 4453 1550 50  0000 C CNN
 F 1 "Fuse" V 4544 1550 50  0000 C CNN
-F 2 "" V 4580 1550 50  0001 C CNN
+F 2 "Fuse:Fuseholder_Littelfuse_Nano2_157x" V 4580 1550 50  0001 C CNN
 F 3 "~" H 4650 1550 50  0001 C CNN
 	1    4650 1550
@@
 F 0 "U1" H 3150 4331 50  0000 C CNN
 F 1 "UCC3801" H 3150 4240 50  0000 C CNN
-F 2 "" H 3150 3750 50  0001 C CNN
+F 2 "Package_SO:SOIC-8_3.9x4.9mm_P1.27mm" H 3150 3750 50  0001 C CNN
 F 3 "http://www.ti.com/lit/ds/symlink/ucc3800.pdf" H 3150 3750 50  0001 C CNN
 	1    3150 3750
@@
 F 0 "R3" V 3693 3550 50  0000 C CNN
 F 1 "R" V 3784 3550 50  0000 C CNN
-F 2 "" V 3830 3550 50  0001 C CNN
+F 2 "Resistor_SMD:R_0805_2012Metric" V 3830 3550 50  0001 C CNN
 F 3 "~" H 3900 3550 50  0001 C CNN
 	1    3900 3550
@@
 F 0 "R5" H 6020 4346 50  0000 L CNN
 F 1 "R" H 6020 4255 50  0000 L CNN
-F 2 "" V 5880 4300 50  0001 C CNN
+F 2 "Resistor_SMD:R_0805_2012Metric" V 5880 4300 50  0001 C CNN
 F 3 "~" H 5950 4300 50  0001 C CNN
 	1    5950 4300
@@
 F 0 "R1" H 2220 3546 50  0000 L CNN
 F 1 "R" H 2220 3455 50  0000 L CNN
-F 2 "" V 2080 3500 50  0001 C CNN
+F 2 "Resistor_SMD:R_0805_2012Metric" V 2080 3500 50  0001 C CNN
 F 3 "~" H 2150 3500 50  0001 C CNN
 	1    2150 3500
@@
 F 0 "C1" H 1965 3546 50  0000 L CNN
 F 1 "C" H 1965 3455 50  0000 L CNN
-F 2 "" H 1888 3350 50  0001 C CNN
+F 2 "Capacitor_SMD:C_0805_2012Metric" H 1888 3350 50  0001 C CNN
 F 3 "~" H 1850 3500 50  0001 C CNN
 	1    1850 3500
@@
 F 0 "C2" H 2165 4046 50  0000 L CNN
 F 1 "C" H 2165 3955 50  0000 L CNN
-F 2 "" H 2088 3850 50  0001 C CNN
+F 2 "Capacitor_SMD:C_0805_2012Metric" H 2088 3850 50  0001 C CNN
 F 3 "~" H 2050 4000 50  0001 C CNN
 	1    2050 4000
@@
 F 0 "R2" H 2370 4146 50  0000 L CNN
 F 1 "R" H 2370 4055 50  0000 L CNN
-F 2 "" V 2230 4100 50  0001 C CNN
+F 2 "Resistor_SMD:R_0805_2012Metric" V 2230 4100 50  0001 C CNN
 F 3 "~" H 2300 4100 50  0001 C CNN
 	1    2300 4100
@@
 F 0 "C3" H 2665 4146 50  0000 L CNN
 F 1 "C" H 2665 4055 50  0000 L CNN
-F 2 "" H 2588 3950 50  0001 C CNN
+F 2 "Capacitor_SMD:C_0805_2012Metric" H 2588 3950 50  0001 C CNN
 F 3 "~" H 2550 4100 50  0001 C CNN
 	1    2550 4100
@@
 F 0 "U3" H 7900 4767 50  0000 C CNN
 F 1 "LM2903" H 7900 4676 50  0000 C CNN
-F 2 "" H 7900 4400 50  0001 C CNN
+F 2 "Package_SO:SOIC-8_3.9x4.9mm_P1.27mm" H 7900 4400 50  0001 C CNN
 F 3 "http://www.ti.com/lit/ds/symlink/lm393.pdf" H 7900 4400 50  0001 C CNN
 	1    7900 4400
@@
 F 0 "RV1" H 6630 4546 50  0000 R CNN
 F 1 "R_POT_TRIM" H 6630 4455 50  0000 R CNN
-F 2 "" H 6700 4500 50  0001 C CNN
+F 2 "Potentiometer_SMD:Potentiometer_Bourns_3314G_Vertical" H 6700 4500 50  0001 C CNN
 F 3 "~" H 6700 4500 50  0001 C CNN
 	1    6700 4500
@@
 F 0 "C6" H 6265 4496 50  0000 L CNN
 F 1 "C" H 6265 4405 50  0000 L CNN
-F 2 "" H 6188 4300 50  0001 C CNN
+F 2 "Capacitor_SMD:C_0805_2012Metric" H 6188 4300 50  0001 C CNN
 F 3 "~" H 6150 4450 50  0001 C CNN
 	1    6150 4450
@@
 F 0 "RV2" H 8430 3646 50  0000 R CNN
 F 1 "R_POT_TRIM" H 8430 3555 50  0000 R CNN
-F 2 "" H 8500 3600 50  0001 C CNN
+F 2 "Potentiometer_SMD:Potentiometer_Bourns_3314G_Vertical" H 8500 3600 50  0001 C CNN
 F 3 "~" H 8500 3600 50  0001 C CNN
 	1    8500 3600
@@
 F 0 "U2" H 7994 3496 50  0000 L CNN
 F 1 "TL081" H 7994 3405 50  0000 L CNN
-F 2 "" H 7700 3500 50  0001 C CNN
+F 2 "Package_TO_SOT_SMD:SOT-23-6" H 7700 3500 50  0001 C CNN
 F 3 "http://www.ti.com/lit/ds/symlink/tl081.pdf" H 7800 3600 50  0001 C CNN
 	1    7650 3450
@@
 F 0 "U3" H 7900 5567 50  0000 C CNN
 F 1 "LM2903" H 7900 5476 50  0000 C CNN
-F 2 "" H 7900 5200 50  0001 C CNN
+F 2 "Package_SO:SOIC-8_3.9x4.9mm_P1.27mm" H 7900 5200 50  0001 C CNN
 F 3 "http://www.ti.com/lit/ds/symlink/lm393.pdf" H 7900 5200 50  0001 C CNN
 	2    7900 5200
@@
 F 0 "D3" V 8839 4932 50  0000 R CNN
 F 1 "LED" V 8748 4932 50  0000 R CNN
-F 2 "" H 8800 5050 50  0001 C CNN
+F 2 "LED_SMD:LED_0805_2012Metric_Castellated" H 8800 5050 50  0001 C CNN
 F 3 "~" H 8800 5050 50  0001 C CNN
 	1    8800 5050
@@
 F 0 "R8" H 8870 4746 50  0000 L CNN
 F 1 "R" H 8870 4655 50  0000 L CNN
-F 2 "" V 8730 4700 50  0001 C CNN
+F 2 "Resistor_SMD:R_0805_2012Metric" V 8730 4700 50  0001 C CNN
 F 3 "~" H 8800 4700 50  0001 C CNN
 	1    8800 4700
@@
 F 0 "R7" H 7070 4946 50  0000 L CNN
 F 1 "R" H 7070 4855 50  0000 L CNN
-F 2 "" V 6930 4900 50  0001 C CNN
+F 2 "Resistor_SMD:R_0805_2012Metric" V 6930 4900 50  0001 C CNN
 F 3 "~" H 7000 4900 50  0001 C CNN
 	1    7000 4900
@@
 F 0 "D2" V 7039 5182 50  0000 R CNN
 F 1 "LED" V 6948 5182 50  0000 R CNN
-F 2 "" H 7000 5300 50  0001 C CNN
+F 2 "LED_SMD:LED_0805_2012Metric_Castellated" H 7000 5300 50  0001 C CNN
 F 3 "~" H 7000 5300 50  0001 C CNN
 	1    7000 5300
@@
 F 0 "R6" H 6120 3546 50  0000 L CNN
 F 1 "R" H 6120 3455 50  0000 L CNN
-F 2 "" V 5980 3500 50  0001 C CNN
+F 2 "Resistor_SMD:R_0805_2012Metric" V 5980 3500 50  0001 C CNN
 F 3 "~" H 6050 3500 50  0001 C CNN
 	1    6050 3500
@@
 F 0 "J1" H 3158 1931 50  0000 C CNN
 F 1 "Conn_01x06_Male" H 3158 1840 50  0000 C CNN
-F 2 "" H 3050 1550 50  0001 C CNN
+F 2 "Connector_JST:JST_XH_B6B-XH-AM_1x06_P2.50mm_Vertical" H 3050 1550 50  0001 C CNN
 F 3 "~" H 3050 1550 50  0001 C CNN
 	1    3050 1550
@@
 F 0 "U3" H 9658 4746 50  0000 L CNN
 F 1 "LM2903" H 9658 4655 50  0000 L CNN
-F 2 "" H 9700 4700 50  0001 C CNN
+F 2 "Package_SO:SOIC-8_3.9x4.9mm_P1.27mm" H 9700 4700 50  0001 C CNN
 F 3 "http://www.ti.com/lit/ds/symlink/lm393.pdf" H 9700 4700 50  0001 C CNN
 	3    9700 4700

Commit message: add digikey pns
Parts:
- added C?: 470pF 2000V NP0, Capacitor_SMD:C_1812_4532Metric, symbol Device:C
- added R?: 20k, Resistor_SMD:R_0805_2012Metric, symbol Device:R
- added R?: 100k, Resistor_SMD:R_1210_3225Metric, symbol Device:R
- added R?: 100k, Resistor_SMD:R_0805_2012Metric, symbol Device:R
- added R?: 100, Resistor_SMD:R_0805_2012Metric, symbol Device:R
- C1: value C -> 10000pF; Digikey (none) -> 732-12139-1-ND
- C2, C6: value C -> 0.1uF; Digikey (none) -> 478-10836-1-ND
- C3: value C -> 22000pF; Digikey (none) -> 478-08053C223KAT2ACT-ND
- C4: value CP -> 12uF 250V; Digikey (none) -> 493-6735-1-ND
- C5: value C -> 0.1uF 200V; Digikey (none) -> 732-12081-1-ND
- D1: Digikey (none) -> BAV99RWT1GOSCT-ND
- D2: Digikey (none) -> 732-4986-1-ND
- D3: Digikey (none) -> 732-4984-1-ND
- F1: Digikey (none) -> F1889-ND
- J1: Digikey (none) -> 455-2238-ND
- Q1: Digikey (none) -> 448-IMBF170R450M1XTMA1CT-ND
- R1, R2, R7, R8: value R -> 10k; Digikey (none) -> 311-10.0KCRCT-ND
- R3, R4: value R -> 1; Digikey (none) -> YAG3705CT-ND
- R5: value R -> 100k; Digikey (none) -> YAG3688CT-ND
- R6: value R -> 100; Digikey (none) -> 311-100CRCT-ND
- RV1, RV2: value R_POT_TRIM -> 1k; Digikey (none) -> 3314G-1-102E
- U1: value UCC3801 -> UCC2801; Digikey (none) -> 296-27157-1-ND
- U2: footprint Package_TO_SOT_SMD:SOT-23-6 -> Package_SO:SOIC-8_3.9x4.9mm_P1.27mm; Digikey (none) -> 296-7204-5-ND
- U3: Digikey (none) -> LM2903EDR2GOSCT-ND
Connections:
- wire segments 75 -> 83
Other:
- note added: "Note: SiC MOSFET with 12V gate drive"
- moved on the sheet: C1, C2, C6, D1, D2, D3, R7, R8, RV1, U3A, U3B, U3C

Commit message: pcb
Parts:
- added C8, C9: 0.1uF, Capacitor_SMD:C_0805_2012Metric, symbol Device:C
- added E1: SPARK_GAP, Resistor_SMD:R_1218_3246Metric_Pad1.22x4.75mm_HandSolder, symbol Device:SPARK_GAP
- added H1, H2, H3, H4: MountingHole_Pad, MountingHole:MountingHole_3.2mm_M3_Pad_Via, symbol Mechanical:MountingHole_Pad
- added R13: 1k, Resistor_SMD:R_0805_2012Metric, symbol Device:R
- C4: footprint Capacitor_SMD:C_Elec_4x5.4 -> Capacitor_SMD:C_Elec_8x10.2
- F1: footprint Fuse:Fuseholder_Littelfuse_Nano2_157x -> Fuse:Fuse_Schurter_UMT250
- gave numbers to parts that had none: 5
Connections:
- net labels added: VBUS, snubber_node, sw
- net labels removed: HT
- wire segments 83 -> 85

Commit message: some td-hv layout
Parts:
- added C10: 0.1uF, Capacitor_SMD:C_0805_2012Metric, symbol Device:C
- added D4: BAS21, Package_TO_SOT_SMD:SOT-23, symbol Diode:BAS21
- added D5: SMAJ400ALFCT-ND, Diode_SMD:D_SMA, symbol Device:D_Zener
- added R14: 50, Resistor_SMD:R_1206_3216Metric, symbol Device:R
- added unit 3 of U2
- J1: value Conn_01x06_Male -> Conn_01x07_Male; footprint Connector_JST:JST_XH_B6B-XH-AM_1x06_P2.50mm_Vertical -> Connector_JST:JST_XH_B7B-XH-AM_1x07_P2.50mm_Vertical; symbol Connector:Conn_01x06_Male -> Connector:Conn_01x07_Male
- R10, R4: footprint Resistor_SMD:R_0805_2012Metric -> Resistor_SMD:R_1206_3216Metric
- R11: value 100k -> 120; Digikey YAG3688CT-ND -> (none)
- R12: value 100 -> 50; Digikey 311-100CRCT-ND -> (none)
- U2: value TL081 -> TLC272; symbol Amplifier_Operational:TL081 -> Amplifier_Operational:TLC272
Connections:
- net labels added: sync_in, vbus_in
- wire segments 85 -> 92
- no-connect marks 6 -> 4
Other:
- moved on the sheet: C4, C5, C6, C8, C9, D1, D2, D3, L1, R2, R5, R6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
