File: td-hv/td-hv.sch (KiCad schematic (older format))
At the start: 43 parts, among them J1 Conn_01x07_Male, Q1 IMBF170R450M1XTMA1, U1 UCC2801, U2 TLC272, U3 LM2903

Commit message: pn updates for hv
Parts:
- D2: value LED -> ‎150080GS75000‎; Digikey 732-4986-1-ND -> ‎732-4983-1-ND‎; Manufacturer (none) -> Würth Elektronik
Changed lines of the file:
@@
 P 8350 5650
 F 0 "D2" V 8389 5532 50  0000 R CNN
-F 1 "LED" V 8298 5532 50  0000 R CNN
+F 1 "‎150080GS75000‎" V 8298 5532 50  0000 R CNN
 F 2 "LED_SMD:LED_0805_2012Metric_Castellated" H 8350 5650 50  0001 C CNN
 F 3 "~" H 8350 5650 50  0001 C CNN
-F 4 "732-4986-1-ND" V 8350 5650 50  0001 C CNN "Digikey"
+F 4 " ‎732-4983-1-ND‎ " V 8350 5650 50  0001 C CNN "Digikey"
+F 5 " Würth Elektronik" V 8350 5650 50  0001 C CNN "Manufacturer"
 	1    8350 5650
 	0    -1   -1   0

Commit message: td-hv bugfixes
Parts:
- C3: value 22000pF -> 560pF; Digikey 478-08053C223KAT2ACT-ND -> 399-1134-1-ND
- C5: footprint Capacitor_SMD:C_0805_2012Metric -> Capacitor_SMD:C_1206_3216Metric
- C7: value 470pF 2000V NP0 -> 47pF 2000V NP0; footprint Capacitor_SMD:C_1812_4532Metric -> Capacitor_SMD:C_1206_3216Metric; Digikey 399-17981-1-ND -> 1276-3272-1-ND‎
- R10: value 20k -> 3k; footprint Resistor_SMD:R_1206_3216Metric -> Resistor_SMD:R_2512_6332Metric; Digikey 311-20.0KCRCT-ND -> 13-RC2512JK-073KLCT-ND‎
- R2: value 10k -> 100k; Digikey 311-10.0KCRCT-ND -> YAG3688CT-ND
- R4: value 1 -> 4.7; Digikey YAG3705CT-ND -> RNCP1206FTD4R70
Connections:
- net eht_current: now also L1.8
- net ucc3801_ref: no longer U3.5 (+)
- net at L1.7: now also RV2.1
- net at RV1.2, U3.2 (-): now also U3.5 (+)
Other:
- moved on the sheet: R5, R6, RV2
Changed lines of the file:
@@
 $EndDescr
-$Comp
-L td-hv:053X0528-001 L1
-U 1 1 60FCCF60
-P 6550 3300
-F 0 "L1" H 6550 3645 50  0000 C CNN
-F 1 "053X0528-001" H 6550 3554 50  0000 C CNN
-F 2 "td-hv:053X0528-001" V 6550 3350 50  0001 C CNN
-F 3 "~" V 6550 3350 50  0001 C CNN
-	1    6550 3300
-	1    0    0    -1
-$EndComp
 $Comp
 L Transistor_FET:C2M1000170J Q1
@@
 Wire Wire Line
 	4500 3350 4750 3350
-$Comp
-L Device:R R4
-U 1 1 60FD3507
-P 4500 4100
-F 0 "R4" H 4570 4146 50  0000 L CNN
-F 1 "1" H 4570 4055 50  0000 L CNN
-F 2 "Resistor_SMD:R_1206_3216Metric" V 4430 4100 50  0001 C CNN
-F 3 "~" H 4500 4100 50  0001 C CNN
-F 4 "YAG3705CT-ND" H 4500 4100 50  0001 C CNN "Digikey"
-	1    4500 4100
-	1    0    0    -1
-$EndComp
 Wire Wire Line
 	4500 3950 4500 3850
@@
 F 0 "C5" H 5865 2396 50  0000 L CNN
 F 1 "0.1uF 200V" H 5865 2305 50  0000 L CNN
-F 2 "Capacitor_SMD:C_0805_2012Metric" H 5788 2200 50  0001 C CNN
+F 2 "Capacitor_SMD:C_1206_3216Metric" H 5788 2200 50  0001 C CNN
 F 3 "~" H 5750 2350 50  0001 C CNN
 F 4 "732-12081-1-ND" H 5750 2350 50  0001 C CNN "Digikey"
@@
 L Device:R R5
 U 1 1 60FEDC18
-P 6750 4650
-F 0 "R5" H 6820 4696 50  0000 L CNN
-F 1 "100k" H 6820 4605 50  0000 L CNN
-F 2 "Resistor_SMD:R_0805_2012Metric" V 6680 4650 50  0001 C CNN
-F 3 "~" H 6750 4650 50  0001 C CNN
-F 4 "YAG3688CT-ND" H 6750 4650 50  0001 C CNN "Digikey"
-	1    6750 4650
+P 6950 4650
+F 0 "R5" H 7020 4696 50  0000 L CNN
+F 1 "100k" H 7020 4605 50  0000 L CNN
+F 2 "Resistor_SMD:R_0805_2012Metric" V 6880 4650 50  0001 C CNN
+F 3 "~" H 6950 4650 50  0001 C CNN
+F 4 "YAG3688CT-ND" H 6950 4650 50  0001 C CNN "Digikey"
+	1    6950 4650
 	1    0    0    -1
 $EndComp
@@
 P 2150 3950
 F 0 "R2" H 2220 3996 50  0000 L CNN
-F 1 "10k" H 2220 3905 50  0000 L CNN
+F 1 "100k" H 2220 3905 50  0000 L CNN
 F 2 "Resistor_SMD:R_0805_2012Metric" V 2080 3950 50  0001 C CNN
 F 3 "~" H 2150 3950 50  0001 C CNN
-F 4 "311-10.0KCRCT-ND" H 2150 3950 50  0001 C CNN "Digikey"
+F 4 "YAG3688CT-ND" H 2150 3950 50  0001 C CNN "Digikey"
 	1    2150 3950
 	0    1    1    0
@@
 P 2550 4100
 F 0 "C3" H 2665 4146 50  0000 L CNN
-F 1 "22000pF" H 2665 4055 50  0000 L CNN
+F 1 "560pF" H 2665 4055 50  0000 L CNN
 F 2 "Capacitor_SMD:C_0805_2012Metric" H 2588 3950 50  0001 C CNN
 F 3 "~" H 2550 4100 50  0001 C CNN
-F 4 "478-08053C223KAT2ACT-ND" H 2550 4100 50  0001 C CNN "Digikey"
+F 4 "399-1134-1-ND" H 2550 4100 50  0001 C CNN "Digikey"
 	1    2550 4100
 	1    0    0    -1
@@
 Connection ~ 8050 5050
 Wire Wire Line
-	8950 4850 8200 4850
+	8950 4850 8800 4850
 Text Label 2150 3850 0    50   ~ 0
 ucc3801_ref
 Text Label 8450 4650 0    50   ~ 0
 ucc3801_ref
-Wire Wire Line
-	8950 4650 8800 4650
 Text Label 2250 3350 0    50   ~ 0
 comp
@@
 Wire Wire Line
 	8950 5450 8800 5450
-Wire Wire Line
-	8800 5450 8800 4650
-Connection ~ 8800 4650
-Wire Wire Line
-	8800 4650 8700 4650
 Wire Wire Line
 	8700 4650 8700 5650
@@
 Wire Wire Line
 	7750 5350 7750 4300
-$Comp
-L Device:R R6
-U 1 1 61032E6F
-P 6850 3500
-F 0 "R6" H 6920 3546 50  0000 L CNN
-F 1 "100" H 6920 3455 50  0000 L CNN
-F 2 "Resistor_SMD:R_0805_2012Metric" V 6780 3500 50  0001 C CNN
-F 3 "~" H 6850 3500 50  0001 C CNN
-F 4 "311-100CRCT-ND" H 6850 3500 50  0001 C CNN "Digikey"
-	1    6850 3500
-	1    0    0    -1
-$EndComp
-Wire Wire Line
-	6850 3350 6750 3350
-$Comp
-L power:GND #PWR0117
-U 1 1 61034B7D
-P 6850 3650
-F 0 "#PWR0117" H 6850 3400 50  0001 C CNN
-F 1 "GND" H 6855 3477 50  0000 C CNN
-F 2 "" H 6850 3650 50  0001 C CNN
-F 3 "" H 6850 3650 50  0001 C CNN
-	1    6850 3650
-	1    0    0    -1
-$EndComp
 Text Label 9600 5550 0    50   ~ 0
 ~xray_protect
-Text Label 6850 3250 0    50   ~ 0
-eht_current
-Wire Wire Line
-	6850 3250 6850 3350
-Connection ~ 6850 3350
 Text Label 3250 1650 0    50   ~ 0
 ~xray_protect
@@
 $EndComp
 Connection ~ 1700 3850
-NoConn ~ 6750 3950
+NoConn ~ 6950 3950
 $Comp
 L Device:C C7
@@
 P 4950 3500
 F 0 "C7" H 5065 3546 50  0000 L CNN
-F 1 "470pF 2000V NP0" H 5065 3455 50  0000 L CNN
-F 2 "Capacitor_SMD:C_1812_4532Metric" H 4988 3350 50  0001 C CNN
+F 1 "47pF 2000V NP0" H 5065 3455 50  0000 L CNN
+F 2 "Capacitor_SMD:C_1206_3216Metric" H 4988 3350 50  0001 C CNN
 F 3 "~" H 4950 3500 50  0001 C CNN
-F 4 "399-17981-1-ND" H 4950 3500 50  0001 C CNN "Digikey"
+F 4 "1276-3272-1-ND‎" H 4950 3500 50  0001 C CNN "Digikey"
 	1    4950 3500
 	1    0    0    -1
@@
 P 4950 3800
 F 0 "R10" H 5020 3846 50  0000 L CNN
-F 1 "20k" H 5020 3755 50  0000 L CNN
-F 2 "Resistor_SMD:R_1206_3216Metric" V 4880 3800 50  0001 C CNN
+F 1 "3k" H 5020 3755 50  0000 L CNN
+F 2 "Resistor_SMD:R_2512_6332Metric" V 4880 3800 50  0001 C CNN
 F 3 "~" H 4950 3800 50  0001 C CNN
-F 4 "311-20.0KCRCT-ND" H 4950 3800 50  0001 C CNN "Digikey"
+F 4 "13-RC2512JK-073KLCT-ND‎" H 4950 3800 50  0001 C CNN "Digikey"
 	1    4950 3800
 	1    0    0    -1
@@
 L Device:R_POT_TRIM RV2
 U 1 1 61008162
-P 6750 4350
-F 0 "RV2" H 6680 4396 50  0000 R CNN
-F 1 "1k" H 6680 4305 50  0000 R CNN
-F 2 "Potentiometer_SMD:Potentiometer_Bourns_3314G_Vertical" H 6750 4350 50  0001 C CNN
-F 3 "~" H 6750 4350 50  0001 C CNN
-F 4 "3314G-1-102E" H 6750 4350 50  0001 C CNN "Digikey"
-	1    6750 4350
+P 6950 4350
+F 0 "RV2" H 6880 4396 50  0000 R CNN
+F 1 "1k" H 6880 4305 50  0000 R CNN
+F 2 "Potentiometer_SMD:Potentiometer_Bourns_3314G_Vertical" H 6950 4350 50  0001 C CNN
+F 3 "~" H 6950 4350 50  0001 C CNN
+F 4 "3314G-1-102E" H 6950 4350 50  0001 C CNN "Digikey"
+	1    6950 4350
 	1    0    0    -1
 $EndComp
@@
 L power:GND #PWR0109
 U 1 1 60FEDDEA
-P 6750 4800
-F 0 "#PWR0109" H 6750 4550 50  0001 C CNN
-F 1 "GND" H 6755 4627 50  0000 C CNN
-F 2 "" H 6750 4800 50  0001 C CNN
-F 3 "" H 6750 4800 50  0001 C CNN
-	1    6750 4800
-	1    0    0    -1
-$EndComp
-Wire Wire Line
-	6750 4200 6750 4150
-Wire Wire Line
-	6750 4500 6900 4500
-Wire Wire Line
-	6900 4500 6900 4350
-Connection ~ 6750 4500
-Wire Wire Line
-	6900 4500 7500 4500
+P 6950 4800
+F 0 "#PWR0109" H 6950 4550 50  0001 C CNN
+F 1 "GND" H 6955 4627 50  0000 C CNN
+F 2 "" H 6950 4800 50  0001 C CNN
+F 3 "" H 6950 4800 50  0001 C CNN
+	1    6950 4800
+	1    0    0    -1
+$EndComp
+Wire Wire Line
+	6950 4500 7100 4500
+Wire Wire Line
+	7100 4500 7100 4350
+Connection ~ 6950 4500
+Wire Wire Line
+	7100 4500 7500 4500
 Wire Wire Line
 	7500 3350 7500 4500
-Connection ~ 6900 4500
+Connection ~ 7100 4500
+Wire Wire Line
+	8700 4650 8950 4650
+Wire Wire Line
+	8800 5450 8800 4850
+Connection ~ 8800 4850
+Wire Wire Line
+	8800 4850 8200 4850
+Wire Wire Line
+	6950 4150 6950 4200
+Text Label 7000 3350 0    50   ~ 0
+eht_current
+$Comp
+L power:GND #PWR0117
+U 1 1 61034B7D
+P 7250 3650
+F 0 "#PWR0117" H 7250 3400 50  0001 C CNN
+F 1 "GND" H 7255 3477 50  0000 C CNN
+F 2 "" H 7250 3650 50  0001 C CNN
+F 3 "" H 7250 3650 50  0001 C CNN
+	1    7250 3650
+	1    0    0    -1
+$EndComp
+$Comp
+L Device:R R6
+U 1 1 61032E6F
+P 7250 3500
+F 0 "R6" H 7320 3546 50  0000 L CNN
+F 1 "100" H 7320 3455 50  0000 L CNN
+F 2 "Resistor_SMD:R_0805_2012Metric" V 7180 3500 50  0001 C CNN
+F 3 "~" H 7250 3500 50  0001 C CNN
+F 4 "311-100CRCT-ND" H 7250 3500 50  0001 C CNN "Digikey"
+	1    7250 3500
+	1    0    0    -1
+$EndComp
+$Comp
+L td-hv:053X0528-001 L1
+U 1 1 60FCCF60
+P 6550 3300
+F 0 "L1" H 6550 3645 50  0000 C CNN
+F 1 "053X0528-001" H 6550 3554 50  0000 C CNN
+F 2 "td-hv:053X0528-001" V 6550 3350 50  0001 C CNN
+F 3 "~" V 6550 3350 50  0001 C CNN
+	1    6550 3300
+	1    0    0    -1
+$EndComp
+Wire Wire Line
+	6950 3350 7250 3350
+$Comp
+L Device:R R4
+U 1 1 60FD3507
+P 4500 4100
+F 0 "R4" H 4570 4146 50  0000 L CNN
+F 1 "4.7" H 4570 4055 50  0000 L CNN
+F 2 "Resistor_SMD:R_1206_3216Metric" V 4430 4100 50  0001 C CNN
+F 3 "~" H 4500 4100 50  0001 C CNN
+F 4 "RNCP1206FTD4R70" H 4500 4100 50  0001 C CNN "Digikey"
+	1    4500 4100
+	1    0    0    -1
+$EndComp
 $EndSCHEMATC

Commit message: td-hv improvements
Parts:
- removed D4: BAS21, Package_TO_SOT_SMD:SOT-23, symbol Diode:BAS21
- removed D5: SMAJ400ALFCT-ND, Diode_SMD:D_SMA, symbol Device:D_Zener
- added C11: 10000pF, Capacitor_SMD:C_0805_2012Metric, symbol Device:C
- added C12: 0.01uF, Capacitor_SMD:C_0805_2012Metric, symbol Device:C
- added L2: L, Inductor_SMD:L_Bourns_SRR1260, symbol Device:L
- added R15: R, Resistor_THT:R_Radial_Power_L13.0mm_W9.0mm_P5.00mm, symbol Device:R
- added R16, R17: 10k, Resistor_SMD:R_0805_2012Metric, symbol Device:R
- R14: value 50 -> 10k; footprint Resistor_SMD:R_1206_3216Metric -> Resistor_SMD:R_0805_2012Metric
- RV2: value 1k -> 10k
- U2: footprint (none) -> Package_SO:SOIC-8_3.9x4.9mm_P1.27mm
Connections:
- net GND: now also L1.5, C12.2; no longer L1.3, R10.2
- net VBUS: now also L2.1, R15.1; no longer L1.2
- net comp: now also R14.1, C11.1; no longer R1.1
- net cs: now also C12.1, R17.2; no longer Q1.2 (DS), Q1.3 (S), Q1.4 (S), Q1.5 (S), Q1.6 (S), Q1.7 (S), R4.1
- net fb: now also R14.2; no longer C1.2, R1.2, U1.2 (FB)
- net sw: now also C7.2; no longer C7.1, R14.2
- net at D1.1 (K): now also L1.3; no longer L1.4
- net at C6.1, R7.1, RV1.1: now also R16.2; no longer D1.3 (K)
- net snubber_node: no longer names the net of R10.1
- net snubber_node: now also L1.2, L2.2, R15.2; no longer C7.2
- new net: Q1.3 (S), Q1.4 (S), Q1.5 (S), Q1.6 (S), Q1.7 (S), R17.1, R4.1
- new net: C1.2, R1.2, U1.2 (FB)
- new net: C11.2, R1.1
- new net: D1.3 (K), R16.1
- new net: C7.1, R10.2
- no-connect marks 4 -> 5
Other:
- note added: "turn-off damping"
- note added: "turn-on damping"
- moved on the sheet: C4, C5, C7, D1, R10, R9
