File: td-hv/td-hv.kicad_pcb (KiCad board)
At the start: 2 copper layers, 90 x 71 mm, 56 parts, among them J1 Conn_01x14, Q1 BSZ42DN25NS3GATMA1, Q12 G3R450MT17J, Q2 BSZ42DN25NS3GATMA1, U1 74HC00, U13 MCP1416, U2 LM2903, U4 2ED2101S06FXUMA1, U7 MIC5504-3.3YM5

Commit message: small bom changes
Parts:
- D2: value ES1G-13-F -> DNP; footprint Diode_THT:D_DO-41_SOD81_P10.16mm_Horizontal -> Diode_SMD:D_SMA
Changed lines of the file:
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@@
     (property "ki_keywords" "cap capacitor")
     (attr smd)
-    (fp_text reference "C1" (at 0 -1.68) (layer "F.SilkS")
+    (fp_text reference "C1" (at 0 -1.5) (layer "F.SilkS")
         (effects (font (size 1 1) (thickness 0.15)))
     )
@@
     (property "ki_keywords" "cap capacitor")
     (attr smd)
-    (fp_text reference "C4" (at -0.05 1.75 -90) (layer "F.SilkS")
+    (fp_text reference "C4" (at -4.05 -0.25 -90) (layer "F.SilkS")
         (effects (font (size 1 1) (thickness 0.15)))
     )
@@
     (property "ki_keywords" "R res resistor")
     (attr smd)
-    (fp_text reference "R5" (at -0.6 1.5 90) (layer "F.SilkS")
+    (fp_text reference "R5" (at -0.0875 2 90) (layer "F.SilkS")
         (effects (font (size 1 1) (thickness 0.15)))
     )
@@
     )
   )
-  (footprint "Diode_THT:D_DO-41_SOD81_P10.16mm_Horizontal" (layer "F.Cu")
+  (footprint "Diode_SMD:D_SMA" (layer "F.Cu")
     (at 116 72 180)
-    (descr "Diode, DO-41_SOD81 series, Axial, Horizontal, pin pitch=10.16mm, , length*diameter=5.2*2.7mm^2, , http://www.diodes.com/_files/packages/DO-41%20(Plastic).pdf")
-    (tags "Diode DO-41_SOD81 series Axial Horizontal pin pitch 10.16mm  length 5.2mm diameter 2.7mm")
+    (descr "Diode SMA (DO-214AC)")
+    (tags "Diode SMA (DO-214AC)")
     (property "Digikey" "ES1G-FDICT-ND")
     (property "Field2" "")
@@
     (property "Sim.Device" "D")
     (property "Sim.Pins" "1=K 2=A")
-    (property "ki_description" "400V 1A Fast recovery Rectifier Diode, DO-41")
+    (property "ki_description" "400V, 1A, General Purpose Rectifier Diode, SMA(DO-214AC)")
     (property "ki_keywords" "diode")
-    (attr through_hole)
-    (fp_text reference "D2" (at 5.08 -2.47 180) (layer "F.SilkS")
-        (effects (font (size 1 1) (thickness 0.15)))
-    )
-    (fp_text value "ES1G-13-F" (at 5.08 2.47 180) (layer "F.Fab")
-        (effects (font (size 1 1) (thickness 0.15)))
-    )
-    (fp_text user "K" (at 0 -2.1 180) (layer "F.SilkS")
+    (attr smd)
+    (fp_text reference "D2" (at 1 2.5 180) (layer "F.SilkS")
         (effects (font (size 1 1) (thickness 0.15)))
     )
-    (fp_text user "${REFERENCE}" (at 5.47 0 180) (layer "F.Fab")
+    (fp_text value "DNP" (at 0 2.6 180) (layer "F.Fab")
         (effects (font (size 1 1) (thickness 0.15)))
     )
-    (fp_text user "K" (at 0 -2.1 180) (layer "F.Fab")
+    (fp_text user "${REFERENCE}" (at 0 -2.5 180) (layer "F.Fab")
         (effects (font (size 1 1) (thickness 0.15)))
     )
-    (fp_line (start 1.34 0) (end 2.36 0)
-      (stroke (width 0.12) (type solid)) (layer "F.SilkS"))
-    (fp_line (start 2.36 -1.47) (end 2.36 1.47)
-      (stroke (width 0.12) (type solid)) (layer "F.SilkS"))
-    (fp_line (start 2.36 1.47) (end 7.8 1.47)
+    (fp_line (start -3.51 -1.65) (end -3.51 1.65)
       (stroke (width 0.12) (type solid)) (layer "F.SilkS"))
-    (fp_line (start 3.14 -1.47) (end 3.14 1.47)
+    (fp_line (start -3.51 -1.65) (end 2 -1.65)
       (stroke (width 0.12) (type solid)) (layer "F.SilkS"))
-    (fp_line (start 3.26 -1.47) (end 3.26 1.47)
+    (fp_line (start -3.51 1.65) (end 2 1.65)
       (stroke (width 0.12) (type solid)) (layer "F.SilkS"))
-    (fp_line (start 3.38 -1.47) (end 3.38 1.47)
-      (stroke (width 0.12) (type solid)) (layer "F.SilkS"))
-    (fp_line (start 7.8 -1.47) (end 2.36 -1.47)
-      (stroke (width 0.12) (type solid)) (layer "F.SilkS"))
-    (fp_line (start 7.8 1.47) (end 7.8 -1.47)
-      (stroke (width 0.12) (type solid)) (layer "F.SilkS"))
-    (fp_line (start 8.82 0) (end 7.8 0)
-      (stroke (width 0.12) (type solid)) (layer "F.SilkS"))
-    (fp_line (start -1.35 -1.6) (end -1.35 1.6)
+    (fp_line (start -3.5 -1.75) (end 3.5 -1.75)
       (stroke (width 0.05) (type solid)) (layer "F.CrtYd"))
-    (fp_line (start -1.35 1.6) (end 11.51 1.6)
+    (fp_line (start -3.5 1.75) (end -3.5 -1.75)
       (stroke (width 0.05) (type solid)) (layer "F.CrtYd"))
-    (fp_line (start 11.51 -1.6) (end -1.35 -1.6)
+    (fp_line (start 3.5 -1.75) (end 3.5 1.75)
       (stroke (width 0.05) (type solid)) (layer "F.CrtYd"))
-    (fp_line (start 11.51 1.6) (end 11.51 -1.6)
+    (fp_line (start 3.5 1.75) (end -3.5 1.75)
       (stroke (width 0.05) (type solid)) (layer "F.CrtYd"))
-    (fp_line (start 0 0) (end 2.48 0)
+    (fp_line (start -2.3 1.5) (end -2.3 -1.5)
       (stroke (width 0.1) (type solid)) (layer "F.Fab"))
-    (fp_line (start 2.48 -1.35) (end 2.48 1.35)
+    (fp_line (start -0.64944 -0.79908) (end -0.64944 0.80112)
       (stroke (width 0.1) (type solid)) (layer "F.Fab"))
-    (fp_line (start 2.48 1.35) (end 7.68 1.35)
+    (fp_line (start -0.64944 0.00102) (end -1.55114 0.00102)
       (stroke (width 0.1) (type solid)) (layer "F.Fab"))
-    (fp_line (start 3.16 -1.35) (end 3.16 1.35)
+    (fp_line (start -0.64944 0.00102) (end 0.50118 -0.79908)
       (stroke (width 0.1) (type solid)) (layer "F.Fab"))
-    (fp_line (start 3.26 -1.35) (end 3.26 1.35)
+    (fp_line (start -0.64944 0.00102) (end 0.50118 0.75032)
       (stroke (width 0.1) (type solid)) (layer "F.Fab"))
-    (fp_line (start 3.36 -1.35) (end 3.36 1.35)
+    (fp_line (start 0.50118 0.00102) (end 1.4994 0.00102)
       (stroke (width 0.1) (type solid)) (layer "F.Fab"))
-    (fp_line (start 7.68 -1.35) (end 2.48 -1.35)
+    (fp_line (start 0.50118 0.75032) (end 0.50118 -0.79908)
       (stroke (width 0.1) (type solid)) (layer "F.Fab"))
-    (fp_line (start 7.68 1.35) (end 7.68 -1.35)
+    (fp_line (start 2.3 -1.5) (end -2.3 -1.5)
       (stroke (width 0.1) (type solid)) (layer "F.Fab"))
-    (fp_line (start 10.16 0) (end 7.68 0)
+    (fp_line (start 2.3 -1.5) (end 2.3 1.5)
       (stroke (width 0.1) (type solid)) (layer "F.Fab"))
-    (pad "1" thru_hole rect (at 0 0 180) (size 2.2 2.2) (drill 1.1) (layers "*.Cu" "*.Mask")
+    (fp_line (start 2.3 1.5) (end -2.3 1.5)
+      (stroke (width 0.1) (type solid)) (layer "F.Fab"))
+    (pad "1" smd roundrect (at -2 0 180) (size 2.5 1.8) (layers "F.Cu" "F.Paste" "F.Mask") (roundrect_rratio 0.1388888889)
       (net 5 "Net-(D2-K)") (pinfunction "K") (pintype "passive"))
-    (pad "2" thru_hole oval (at 10.16 0 180) (size 2.2 2.2) (drill 1.1) (layers "*.Cu" "*.Mask")
+    (pad "2" smd roundrect (at 2 0 180) (size 2.5 1.8) (layers "F.Cu" "F.Paste" "F.Mask") (roundrect_rratio 0.1388888889)
       (net 3 "+12V") (pinfunction "A") (pintype "passive"))
-    (model "${KICAD6_3DMODEL_DIR}/Diode_THT.3dshapes/D_DO-41_SOD81_P10.16mm_Horizontal.wrl"
+    (model "${KICAD6_3DMODEL_DIR}/Diode_SMD.3dshapes/D_SMA.wrl"
       (offset (xyz 0 0 0))
       (scale (xyz 1 1 1))
@@
     (property "ki_keywords" "schottky diode")
     (attr smd)
-    (fp_text reference "D3" (at 0 -2.4) (layer "F.SilkS")
+    (fp_text reference "D3" (at 0 2.75) (layer "F.SilkS")
         (effects (font (size 1 1) (thickness 0.15)))
     )
@@
     (property "ki_keywords" "mosfet gate driver")
     (attr smd)
-    (fp_text reference "U13" (at 0 -2.4) (layer "F.SilkS")
+    (fp_text reference "U13" (at -2.8625 -3.55) (layer "F.SilkS")
         (effects (font (size 1 1) (thickness 0.15)))
     )
@@
     (effects (font (size 1 1) (thickness 0.15)) (justify left))
   )
+  (gr_text "High Voltage" (at 92 83.5 90) (layer "F.SilkS")
+    (effects (font (size 1 1) (thickness 0.15)))
+  )
   (gr_text "gnd" (at 100.5 96.5) (layer "F.SilkS")
     (effects (font (size 1 1) (thickness 0.15)) (justify left))
@@
   (segment (start 121.675 81.105) (end 119.475 78.905) (width 0.25) (layer "F.Cu") (net 33))
   (segment (start 115.25 124.65) (end 115.85 124.65) (width 0.25) (layer "F.Cu") (net 34))
-  (segment (start 117.85 122.35) (end 118 122.5) (width 0.25) (layer "F.Cu") (net 34))
   (segment (start 115.85 124.65) (end 118 122.5) (width 0.25) (layer "F.Cu") (net 34))
   (segment (start 140 73) (end 138.1 73) (width 0.75) (layer "F.Cu") (net 35))
