File: td-hv/td-hv.kicad_sch (KiCad schematic)
At the start: 8 parts, among them J1 Conn_01x14, U7 MIC5504-3.3YM5

Commit message: small bom changes
Parts:
- U7: value MIC5504-3.3YM5 -> AP2205; symbol Regulator_Linear:MIC5504-3.3YM5 -> Regulator_Linear:AP2204K-3.3; Digikey (none) -> 31-AP2205-33W5-7CT-ND
Changed lines of the file:
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@@
 (kicad_sch (version 20230121) (generator eeschema)
   (paper "A4")
+  (junction (at 106.68 81.28) (diameter 0) (color 0 0 0 0)
+  )
   (junction (at 114.3 91.44) (diameter 0) (color 0 0 0 0)
   )
@@
   (junction (at 128.27 81.28) (diameter 0) (color 0 0 0 0)
   )
-  (junction (at 99.06 86.36) (diameter 0) (color 0 0 0 0)
-  )
   (junction (at 99.06 81.28) (diameter 0) (color 0 0 0 0)
   )
@@
   )
   (no_connect (at 177.8 132.08))
-  (wire (pts (xy 99.06 81.28) (xy 104.14 81.28))
+  (wire (pts (xy 99.06 81.28) (xy 106.68 81.28))
     (stroke (width 0) (type default))
   )
@@
     (stroke (width 0) (type default))
   )
-  (wire (pts (xy 124.46 81.28) (xy 128.27 81.28))
+  (wire (pts (xy 121.92 81.28) (xy 128.27 81.28))
     (stroke (width 0) (type default))
   )
@@
     (stroke (width 0) (type default))
   )
+  (wire (pts (xy 106.68 81.28) (xy 106.68 83.82))
+    (stroke (width 0) (type default))
+  )
   (wire (pts (xy 128.27 91.44) (xy 128.27 88.9))
-    (stroke (width 0) (type default))
-  )
-  (wire (pts (xy 104.14 86.36) (xy 99.06 86.36))
     (stroke (width 0) (type default))
   )
@@
     )
   )
-  (symbol (lib_id "Regulator_Linear:MIC5504-3.3YM5") (at 114.3 83.82 0) (unit 1)
+  (symbol (lib_id "Regulator_Linear:AP2204K-3.3") (at 114.3 83.82 0) (unit 1)
     (in_bom yes) (on_board yes) (dnp no) (fields_autoplaced)
     (property "Reference" "U7" (at 114.3 74.5957 0)
       (effects (font (size 1.27 1.27)))
     )
-    (property "Value" "MIC5504-3.3YM5" (at 114.3 77.0199 0)
-      (effects (font (size 1.27 1.27)))
-    )
-    (property "Footprint" "Package_TO_SOT_SMD:SOT-23-5" (at 114.3 93.98 0)
-      (effects (font (size 1.27 1.27)) hide)
-    )
-    (property "Datasheet" "http://ww1.microchip.com/downloads/en/DeviceDoc/MIC550X.pdf" (at 107.95 77.47 0)
-      (effects (font (size 1.27 1.27)) hide)
-    )
+    (property "Value" "AP2205" (at 114.3 77.0199 0)
+      (effects (font (size 1.27 1.27)))
+    )
+    (property "Footprint" "Package_TO_SOT_SMD:SOT-23-5" (at 114.3 75.565 0)
+      (effects (font (size 1.27 1.27)) hide)
+    )
+    (property "Datasheet" "https://www.diodes.com/assets/Datasheets/AP2204.pdf" (at 114.3 81.28 0)
+      (effects (font (size 1.27 1.27)) hide)
+    )
+    (property "Digikey" "31-AP2205-33W5-7CT-ND" (at 114.3 83.82 0)
+      (effects (font (size 1.27 1.27)) hide)
+    )
