File: td-rgbinput/color_channel.sch (KiCad schematic (older format))
At the start: 13 parts, among them Q1 2N7002NXBKR, Q2 2N7002NXBKR, U6 AD8337

Commit message: add todos
Other:
- note added: "todo: bias impedance is not constant"
Changed lines of the file:
@@
 Text GLabel 6000 3300 0    50   Input ~ 0
 bias_buffered
+Text Notes 6050 4000 0    50   ~ 0
+todo: bias impedance is not constant
 $EndSCHEMATC
