File: td-rgbinput/td-rgbinput.sch (KiCad schematic (older format))
At the start: 57 parts, among them J5 DB15_Female_HighDensity_Mount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, Q4 2N7002NXBKR, Q5 2N7002NXBKR, Q6 2N7002NXBKR, U11 LM2664M4, U3 ADA4861-3, U5 AT24CS01-SSHM

Commit message: more rgbinput changes
Parts:
- removed C38, C40: 1uF, Capacitor_SMD:C_0805_2012Metric, symbol Device:C
- removed JP?: Jumper_2_Bridged, symbol Jumper:Jumper_2_Bridged
- removed Q4, Q6, Q?: 2N7002NXBKR, Package_TO_SOT_SMD:SOT-23, symbol Transistor_FET:2N7002
- removed R10, R17, R19, R8: 75, Resistor_SMD:R_0805_2012Metric, symbol Device:R
- removed R11, R13: 330, Resistor_SMD:R_0805_2012Metric, symbol Device:R
- removed R14, R16: 1k, Resistor_SMD:R_0805_2012Metric, symbol Device:R
- removed R53, R59: 10k, Resistor_SMD:R_0805_2012Metric, symbol Device:R
- removed R?: 1k, symbol Device:R
- removed unit 2 of U3
- removed unit 3 of U3
- removed U?: LM1117-5.0, symbol Regulator_Linear:LM1117-5.0
- added C? (x2): 1uF, symbol Device:C
- added C? (x3): 0.1uF, symbol Device:C
- added C? (x2): 2.2uF, symbol Device:C
- added J?: Conn_01x07_Male, symbol Connector:Conn_01x07_Male
- added Q? (x3): 2N7002NXBKR, Package_TO_SOT_SMD:SOT-23, symbol Transistor_FET:2N7002
- added R? (x2): 10k, symbol Device:R
- added R?: 100k, Resistor_SMD:R_0805_2012Metric, symbol Device:R
- added R? (x2): 1k, symbol Device:R
- added RV?: 1k, symbol Device:R_POT
- added U?: ADP7142AUJZ-5.0, Package_TO_SOT_SMD:TSOT-23-5, symbol Regulator_Linear:ADP7142AUJZ-5.0
- added U? (x3): 74HC00, symbol 74xx:74HC00
- C?: value C -> 0.1uF
- R54: value 10k -> 100k
Connections:
- net +5V: now also C?.1, J?.2 (Pin_2), R?.1, U?.2, U?.2, U?.4 (SENSE/ADJ), U?.5 (VOUT); no longer U3.1 (~DISABLE)
- net GND: now also C?.2, C?.2, C?.2, C?.2, C?.2, J?.1 (Pin_1), Q?.2 (S), Q?.2 (S), R?.2, R?.2, RV?.3, U?.2 (GND); no longer Q5.2 (S), R54.2
- net bias_buffered: no longer RV?.1
- net blank: now also Q?.1 (G), U?.1, U?.3; no longer U?.9 (BPOUT)
- net clamp: now also U?.9 (BPOUT), U?.1
- net csync: now also U?.1
- net hsync: now also J?.3 (Pin_3)
- net oddeven: now also J?.6 (Pin_6)
- net vga_hsync: no longer J5.13
- net vsync: now also J?.4 (Pin_4)
- net at U3.5 (+): now also C?.1, Q?.3 (D), R?.1; no longer RV?.2
- net at U?.1: now also R?.2
- net at RV?.2, U?.7 (GAIN): now also C?.1
- net at U?.1 (Rext): now also R?.1
- net at U?.4 (Vin): now also C?.1
- net vga_vsync renamed vsync_vga
- net vsync_vga: now also J?.5 (Pin_5)
- new net: C?.1, Q?.2 (S), RV?.2
- new net: C?.2, Q?.3 (D), R?.1
- new net: Q?.1 (G), Q?.3 (D), R?.2
- new net: R?.2, RV?.1
- new net +12V: C?.1, R?.1, U3.1 (~DISABLE), U?.1 (VIN), U?.3 (EN)
- new net black_ref: C?.1, Q5.2 (S), R54.2, RV?.2
- new net global_bias: RV?.1
- new net hsync_vga: C?.2, J5.13
- new net uc_blank: J?.7 (Pin_7), U?.2
- new net ~blank: U?.3
- new net ~clamp: Q?.1 (G), U?.3
- no-connect marks 2 -> 3
Other:
- moved on the sheet: C28, C30, C31, C39, C?, Q5, R12, R15, R18, R54, R9, R?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

Commit message: td-rgbinput
Parts:
- removed C39: 1uF, Capacitor_SMD:C_0805_2012Metric, symbol Device:C
- removed C? (x2): 1uF, symbol Device:C
- removed C? (x2): 0.1uF, symbol Device:C
- removed Q5, Q? (x3): 2N7002NXBKR, Package_TO_SOT_SMD:SOT-23, symbol Transistor_FET:2N7002
- removed R54, R?: 100k, Resistor_SMD:R_0805_2012Metric, symbol Device:R
- removed R9: 75, Resistor_SMD:R_0805_2012Metric, symbol Device:R
- removed R? (x2): 470, symbol Device:R
- removed R? (x2): 10k, symbol Device:R
- removed R?: 1k, symbol Device:R
- removed RV? (x2): 1k, symbol Device:R_POT
- removed U?: AD8337, symbol td-rgbinput:AD8337
- removed U?: LMH1980, Package_SO:VSSOP-10_3x3mm_P0.5mm, symbol td-deflect:LMH1980
- added C11: 0.1uF, Capacitor_SMD:C_0805_2012Metric, symbol Device:C
- added H1, H2, H3, H4: MountingHole_Pad, MountingHole:MountingHole_3.2mm_M3_Pad_Via, symbol Mechanical:MountingHole_Pad
- added J1: Conn_01x06_Male, Connector_JST:JST_EH_B6B-EH-A_1x06_P2.50mm_Vertical, symbol Connector:Conn_01x06_Male
- added J3: Conn_01x06_Male, Connector_JST:JST_XH_B6B-XH-AM_1x06_P2.50mm_Vertical, symbol Connector:Conn_01x06_Male
- added JP1: Jumper_NC_Small, Jumper:SolderJumper-2_P1.3mm_Bridged_Pad1.0x1.5mm, symbol Device:Jumper_NC_Small
- added R11, R13: 10k, Resistor_SMD:R_0805_2012Metric, symbol Device:R
- added R19, R28, R29, R30: 470, Resistor_SMD:R_0805_2012Metric, symbol Device:R
- added R31, R32: 47, Resistor_SMD:R_0805_2012Metric, symbol Device:R
- added unit 4 of U3
- added unit 2 of U3
- added unit 3 of U3
- C1, C2: renamed from C?; footprint (none) -> Capacitor_SMD:C_0805_2012Metric; Digikey (none) -> 13-CC0805KPX7R9BB103CT-ND
- C3, C4, C5, C6: renamed from C?; footprint (none) -> Capacitor_SMD:C_0805_2012Metric; Digikey (none) -> 1276-2444-1-ND
- C8, C9: renamed from C?; footprint (none) -> Capacitor_SMD:C_0805_2012Metric; Digikey (none) -> 490-14467-1-ND
- J2: renamed from J?; footprint (none) -> Connector_JST:JST_XH_B7B-XH-AM_1x07_P2.50mm_Vertical; Digikey (none) -> 1175-51025-07-0100-01-ND
- J5: footprint td-io:DSUB-15-HD_Female_Horizontal_P2.29x2.5mm_EdgePinOffset8.35mm_Housed_MountingHolesOffset10.89mm -> td-deflect:DSUB-15-HD_Female_Horizontal_P2.29x2.5mm_EdgePinOffset8.35mm_Housed_MountingHolesOffset10.89mm
- R1, R6: renamed from R?; value R -> 1k; footprint (none) -> Resistor_SMD:R_0805_2012Metric; Digikey (none) -> 311-1.00KCRCT-ND
- R10: renamed from R?; footprint (none) -> Resistor_SMD:R_0805_2012Metric; Digikey (none) -> 311-1.00KCRCT-ND
- R12: Digikey 311-330CRCT-ND -> YAG3733CT-ND
- R15: Digikey 311-1.00KCRCT-ND -> YAG3733CT-ND
- R18: Digikey 311-75.0CRCT-ND -> 311-47.0CRCT-ND
- R2, R3, R4, R5: renamed from R?; footprint (none) -> Resistor_SMD:R_0805_2012Metric; Digikey (none) -> 13-RT0805FRE0775RLCT-ND
- R7, R8: renamed from R?; footprint (none) -> Resistor_SMD:R_0805_2012Metric; Digikey (none) -> YAG3690CT-ND
- RV1, RV2, RV3: renamed from RV?; footprint (none) -> Potentiometer_THT:Potentiometer_Bourns_3386P_Vertical; Digikey (none) -> 3386P-102TLF-ND
- SW1: renamed from SW?; Digikey (none) -> CT2064-ND
- U1: renamed from U?; footprint (none) -> Package_SO:SOIC-8_3.9x4.9mm_P1.27mm; Digikey (none) -> 296-1309-1-ND
- U2: renamed from U?; Digikey (none) -> ADP7142ARDZ-5.0
- U4: renamed from U?; value 74HC00 -> 74HCT00; footprint (none) -> Package_SO:SOIC-14_3.9x8.7mm_P1.27mm; Digikey (none) -> 296-14542-1-ND
Connections:
- net hsync_vga is gone; now on net vga_hsync: J5.13
- net vsync is gone; now on net vga_hsync: J2.4 (Pin_4)
- net +12V: now also J2.2 (Pin_2), C11.1, J3.6 (Pin_6), U3.2 (~DISABLE), U3.3 (~DISABLE), U3.4 (V+)
- net +5V: now also U4.10; no longer J2.2 (Pin_2), U4.2
- net GND: now also C11.2, H1.1, H2.1, H3.1, H4.1, J1.4 (Pin_4), J3.1 (Pin_1), J3.2 (Pin_2), JP1.2, R11.2, R13.2, R19.1, R28.1, U3.11 (V-)
- net blank: now also U4.6, U4.9; no longer U4.1, U4.3
- net clamp: now also J2.5 (Pin_5)
- net neck_red: now also J3.5 (Pin_5)
- net uc_blank: now also U4.5, R13.1; no longer U4.2
- net vga_blue: now also SW1.6, J1.3 (Pin_3); no longer SW1.3
- net vga_green: now also SW1.7, J1.2 (Pin_2); no longer SW1.2
- net vga_hsync: now also SW1.5, J1.5 (Pin_5); no longer SW1.4
- net vga_red: now also SW1.8, J1.1 (Pin_1); no longer SW1.1
- net ~blank: now also U4.8; no longer U4.3
- net mixed_red: now reaches U3.5 (+)
- net at R5.1: now also SW1.4; no longer SW1.5
- net at R4.1: now also SW1.3; no longer SW1.6
- net at R3.1: now also SW1.2; no longer SW1.7
- net at R2.1: now also SW1.1; no longer SW1.8
- net black_ref renamed black_level
- net black_level: now also JP1.1
- removed net csync: U4.1
- net hsync renamed vga_vsync
- net vga_vsync: now also J5.14, J1.6 (Pin_6)
- net oddeven renamed sync_blank
- net sync_blank: now also U4.4, R11.1
- removed net vsync_vga: J2.5 (Pin_5), J5.14
- new net: R29.1, R31.2, U3.14
- new net: R30.1, R32.2, U3.8
- new net blue_fb: R28.2, R30.2, U3.9 (-)
- new net green_fb: R19.2, R29.2, U3.13 (-)
- new net mixed_blue: U3.10 (+)
- new net mixed_green: U3.12 (+)
- new net neck_blue: J3.3 (Pin_3), R32.1
- new net neck_green: J3.4 (Pin_4), R31.1
- no-connect marks 3 -> 4
Other:
- note added: "ms9 compatible rgb input connector"
- moved on the sheet: R12, R15, R18, U3A

Commit message: add todos
Other:
- note added: "todo: switch gain knob to -5V\nadd power to global opamp\nadd power to 7400\nchange linear regulator footprint\nreduce paste on ad8337\nreverse pinout on output connector\nswitch digikey pn on dip sw"
Changed lines of the file:
@@
 NoConn ~ 7250 6900
 NoConn ~ 8100 7750
+Text Notes 5550 1500 0    50   ~ 0
+todo: switch gain knob to -5V\nadd power to global opamp\nadd power to 7400\nchange linear regulator footprint\nreduce paste on ad8337\nreverse pinout on output connector\nswitch digikey pn on dip sw
 $EndSCHEMATC
