File: td-rgbinput/td-rgbinput.kicad_pcb (KiCad board)
At the start: 2 copper layers, 180 x 50 mm, 91 parts, among them J1 Conn_01x06_Male, J2 Conn_01x07_Male, J3 Conn_01x06_Male, J5 DB15_Female_HighDensity_Mount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, Q1 2N7002NXBKR, Q2 2N7002NXBKR, Q3 2N7002NXBKR, Q4 2N7002NXBKR, Q5 2N7002NXBKR, Q6 2N7002NXBKR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

Commit message: finish pcb
Parts:
- removed C22: 0.1uF, Capacitor_SMD:C_0805_2012Metric
- removed R10: 1k, Resistor_SMD:R_0805_2012Metric
- removed RV3: 1k, Potentiometer_THT:Potentiometer_Bourns_3386P_Vertical
- added C23: 0.1uF, Capacitor_SMD:C_0805_2012Metric, F.Cu at (181.0, 84.0)
- added C24: 0.1uF, Capacitor_SMD:C_0805_2012Metric, F.Cu at (205.0, 83.5)
- added C25: 0.1uF, Capacitor_SMD:C_0805_2012Metric, F.Cu at (183.0, 95.5)
- added C26: 0.1uF, Capacitor_SMD:C_0805_2012Metric, F.Cu at (181.0, 69.0)
- added C27: 0.1uF, Capacitor_SMD:C_0805_2012Metric, F.Cu at (205.0, 68.5)
- added C29: 0.1uF, Capacitor_SMD:C_0805_2012Metric, F.Cu at (183.0, 80.5)
- added C32: 0.1uF, Capacitor_SMD:C_0805_2012Metric, F.Cu at (181.0, 54.0)
- added C33: 0.1uF, Capacitor_SMD:C_0805_2012Metric, F.Cu at (205.0, 53.5)
- added C34: 0.1uF, Capacitor_SMD:C_0805_2012Metric, F.Cu at (183.0, 65.5)
- added R33: 1k, Resistor_SMD:R_0805_2012Metric, F.Cu at (195.0, 95.5)
- added R34: 1k, Resistor_SMD:R_0805_2012Metric, F.Cu at (190.0, 95.5)
- added R35: 1k, Resistor_SMD:R_0805_2012Metric, F.Cu at (205.0, 86.5)
- added R36: 1k, Resistor_SMD:R_0805_2012Metric, F.Cu at (205.0, 89.5)
- added R37: 1k, Resistor_SMD:R_0805_2012Metric, F.Cu at (195.0, 83.5)
- added R38: 10, Resistor_SMD:R_0805_2012Metric, F.Cu at (179.1, 93.0)
- added R39: 1k, Resistor_SMD:R_0805_2012Metric, F.Cu at (183.0, 93.0)
- added R40: 1k, Resistor_SMD:R_0805_2012Metric, F.Cu at (195.0, 80.5)
- added R41: 1k, Resistor_SMD:R_0805_2012Metric, F.Cu at (190.0, 80.5)
- added R42: 1k, Resistor_SMD:R_0805_2012Metric, F.Cu at (205.0, 71.5)
- added R43: 1k, Resistor_SMD:R_0805_2012Metric, F.Cu at (205.0, 74.5)
- added R44: 1k, Resistor_SMD:R_0805_2012Metric, F.Cu at (195.0, 68.5)
- added R45: 10, Resistor_SMD:R_0805_2012Metric, F.Cu at (179.1, 78.0)
- added R46: 1k, Resistor_SMD:R_0805_2012Metric, F.Cu at (183.0, 78.0)
- added R47: 1k, Resistor_SMD:R_0805_2012Metric, F.Cu at (195.0, 65.5)
- added R48: 1k, Resistor_SMD:R_0805_2012Metric, F.Cu at (190.0, 65.5)
- added R49: 1k, Resistor_SMD:R_0805_2012Metric, F.Cu at (205.0, 56.5)
- added R50: 1k, Resistor_SMD:R_0805_2012Metric, F.Cu at (205.0, 59.5)
- added R51: 1k, Resistor_SMD:R_0805_2012Metric, F.Cu at (195.0, 53.5)
- added R52: 10, Resistor_SMD:R_0805_2012Metric, F.Cu at (179.1, 63.0)
- added R53: 1k, Resistor_SMD:R_0805_2012Metric, F.Cu at (183.0, 63.0)
- added U12: TLC272, Package_SO:SOIC-8_3.9x4.9mm_P1.27mm, F.Cu at (181.0, 89.0)
- added U13: TLC272, Package_SO:SOIC-8_3.9x4.9mm_P1.27mm, F.Cu at (181.0, 74.0)
- added U14: TLC272, Package_SO:SOIC-8_3.9x4.9mm_P1.27mm, F.Cu at (181.0, 59.0)
- U11: value LM2664M4 -> MAX1720EUT
- U2: value ADP7142AUJZ-5.0 -> ADP7142ARDZ-5.0; footprint Package_TO_SOT_SMD:TSOT-23-5 -> Package_SO:SOIC-8-1EP_3.9x4.9mm_P1.27mm_EP2.29x3mm
- U6, U7, U8: footprint Package_CSP:LFCSP-8-1EP_3x3mm_P0.5mm_EP1.45x1.74mm -> td-deflect:LFCSP-8-1EP_3x3mm_P0.5mm_AD8337
- moved C18 93.5 mm to (126.5, 92.0), turned to 180 degrees
- moved C14 82.4 mm to (139.0, 83.0)
- moved RV8 23.3 mm to (159.0, 91.5)
- moved RV9 23.3 mm to (171.0, 91.5)
- moved RV6 23.1 mm to (159.0, 76.5)
- moved RV7 23.1 mm to (171.0, 76.5)
- moved RV4 23.0 mm to (159.0, 61.5)
- moved RV5 23.0 mm to (171.0, 61.5)
- moved C2 21.3 mm to (145.5, 90.5)
- moved C4 20.9 mm to (145.5, 83.0)
- moved R6 20.7 mm to (145.5, 85.5)
- moved C1 20.4 mm to (133.1, 89.5)
- moved C3 20.4 mm to (133.0, 81.9)
- moved R1 20.4 mm to (133.0, 85.7)
- moved R7 20.4 mm to (133.1, 92.7)
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Connections:
- net /~blank renamed /~{blank}
- net /~clamp renamed /~{clamp}
- C12 pad 2: /vga_red -> Net-(C12-Pad2)
- C14 pad 1: Net-(C14-Pad1) -> +5V
- C14 pad 2: GND -> -5V
- C16 pad 2: /vga_green -> Net-(C16-Pad2)
- C18 pad 1: Net-(C18-Pad1) -> +5V
- C20 pad 2: /vga_blue -> Net-(C20-Pad2)
- J3 pad 1: GND -> +12V
- J3 pad 2: GND -> /neck_red
- J3 pad 3: /neck_blue -> /neck_green
- J3 pad 4: /neck_green -> /neck_blue
- J3 pad 5: /neck_red -> GND
- J3 pad 6: +12V -> GND
- J5 pad 11: Net-(J5-Pad11) -> unconnected-(J5-Pad11)
- J5 pad 4: Net-(J5-Pad4) -> unconnected-(J5-Pad4)
- RV1 pad 3: GND -> -5V
- RV4 pad 1: gain_buffered -> +5V
- RV4 pad 2: Net-(C14-Pad1) -> Net-(RV4-Pad2)
- RV4 pad 3: GND -> -5V
- RV5 pad 1: bias_buffered -> +5V
- RV5 pad 2: /mixed_red -> Net-(RV5-Pad2)
- RV6 pad 1: gain_buffered -> +5V
- RV6 pad 2: Net-(C18-Pad1) -> Net-(RV6-Pad2)
- RV6 pad 3: GND -> -5V
- RV7 pad 1: bias_buffered -> +5V
- RV7 pad 2: /mixed_green -> Net-(RV7-Pad2)
- RV8 pad 1: gain_buffered -> +5V
- RV8 pad 2: Net-(C22-Pad1) -> Net-(RV8-Pad2)
- RV8 pad 3: GND -> -5V
- RV9 pad 1: bias_buffered -> +5V
- RV9 pad 2: /mixed_blue -> Net-(RV9-Pad2)
- U1 pad 4: (no net) -> -5V
- U1 pad 8: (no net) -> +5V
- U11 pad 1: GND -> -5V
- U11 pad 2: -5V -> +5V
- U11 pad 4: +5V -> GND
- U2 pad 1: +12V -> +5V
- U2 pad 2: GND -> +5V
- U2 pad 3: +12V -> +5V
- U2 pad 4: +5V -> GND
- U2 pad 5: +5V -> +12V
- U4 pad 14: (no net) -> +5V
- U4 pad 7: (no net) -> GND
- U6 pad 7: Net-(C14-Pad1) -> Net-(U6-Pad7)
- U7 pad 7: Net-(C18-Pad1) -> Net-(U7-Pad7)
- U8 pad 7: Net-(C22-Pad1) -> Net-(U8-Pad7)
Routing:
- net +5V: track 220.7 -> 463.3 mm, vias 6 -> 8
- net -5V: track 141.6 -> 334.2 mm, vias 4 -> 13
- net gain_buffered: track 72.4 -> 137.5 mm, vias 1 -> 4
- net Net-(C18-Pad1): track 43.9 -> 0.00 mm
- net Net-(C22-Pad1): track 43.6 -> 0.00 mm
- net Net-(C14-Pad1): track 43.5 -> 0.00 mm
- net bias_buffered: track 68.6 -> 106.6 mm, vias 0 -> 4
- net black_level: track 110.1 -> 146.8 mm, vias 3 -> 6
- net Net-(RV1-Pad2): track 54.0 -> 31.3 mm, vias 2 -> 1
- net Net-(RV4-Pad2): track 0.00 -> 18.0 mm
- net Net-(RV8-Pad2): track 0.00 -> 18.0 mm
- net Net-(RV6-Pad2): track 0.00 -> 18.0 mm
- net Net-(R21-Pad2): track 16.4 -> 32.8 mm
- net Net-(R25-Pad2): track 16.4 -> 32.8 mm
- net Net-(RV2-Pad2): track 47.8 -> 31.4 mm, vias 2 -> 1
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Other:
- board size 180 x 50 mm -> 165 x 50 mm
- net class Default removed
- board text removed: "sub bias"

Commit message: fill a few extra areas
Routing:
- net GND: vias 47 -> 52
Changed lines of the file:
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@@
   (via (at 144.75 81.5) (size 0.8) (drill 0.4) (layers "F.Cu" "B.Cu") (free) (net 5))
   (via (at 192.5 86.5) (size 0.8) (drill 0.4) (layers "F.Cu" "B.Cu") (free) (net 5))
+  (via (at 146.75 76.5) (size 0.8) (drill 0.4) (layers "F.Cu" "B.Cu") (free) (net 5))
   (via (at 223 72.5) (size 0.8) (drill 0.4) (layers "F.Cu" "B.Cu") (net 5))
   (via (at 135.5 68.5) (size 0.8) (drill 0.4) (layers "F.Cu" "B.Cu") (net 5))
@@
   (via (at 130.5 84.5) (size 0.8) (drill 0.4) (layers "F.Cu" "B.Cu") (net 5))
   (via (at 192.5 95.5) (size 0.8) (drill 0.4) (layers "F.Cu" "B.Cu") (free) (net 5))
+  (via (at 152.75 92.75) (size 0.8) (drill 0.4) (layers "F.Cu" "B.Cu") (free) (net 5))
   (via (at 185.5 95.5) (size 0.8) (drill 0.4) (layers "F.Cu" "B.Cu") (free) (net 5))
   (via (at 207.25 68.5) (size 0.8) (drill 0.4) (layers "F.Cu" "B.Cu") (free) (net 5))
@@
   (via (at 122.5 80.5) (size 0.8) (drill 0.4) (layers "F.Cu" "B.Cu") (net 5))
   (via (at 192.5 65.5) (size 0.8) (drill 0.4) (layers "F.Cu" "B.Cu") (free) (net 5))
+  (via (at 165 65.25) (size 0.8) (drill 0.4) (layers "F.Cu" "B.Cu") (free) (net 5))
   (via (at 192.5 80.5) (size 0.8) (drill 0.4) (layers "F.Cu" "B.Cu") (free) (net 5))
   (via (at 207.25 59.5) (size 0.8) (drill 0.4) (layers "F.Cu" "B.Cu") (free) (net 5))
@@
   (via (at 185.5 65.5) (size 0.8) (drill 0.4) (layers "F.Cu" "B.Cu") (free) (net 5))
   (via (at 192 75.25) (size 0.8) (drill 0.4) (layers "F.Cu" "B.Cu") (free) (net 5))
+  (via (at 148 94) (size 0.8) (drill 0.4) (layers "F.Cu" "B.Cu") (free) (net 5))
+  (via (at 165.25 80.75) (size 0.8) (drill 0.4) (layers "F.Cu" "B.Cu") (free) (net 5))
   (segment (start 180.71548 82.75048) (end 181.965 84) (width 0.75) (layer "F.Cu") (net 6))
   (segment (start 157.770489 55.944506) (end 160.964515 52.75048) (width 0.75) (layer "F.Cu") (net 6))
@@
   (segment (start 154.5 67) (end 154.674511 66.825489) (width 0.25) (layer "F.Cu") (net 12))
   (segment (start 192.777011 66.825489) (end 194.1025 65.5) (width 0.25) (layer "F.Cu") (net 12))
+  (segment (start 160.994536 94.925988) (end 179.974522 94.925988) (width 0.25) (layer "F.Cu") (net 13))
   (segment (start 85.77 75.928) (end 92.572 75.928) (width 0.25) (layer "F.Cu") (net 13))
+  (segment (start 118.820138 74.928436) (end 121.071564 74.928436) (width 0.25) (layer "F.Cu") (net 13))
+  (segment (start 117.866692 73.97499) (end 118.820138 74.928436) (width 0.25) (layer "F.Cu") (net 13))
+  (segment (start 104.45001 73.97499) (end 117.866692 73.97499) (width 0.25) (layer "F.Cu") (net 13))
+  (segment (start 142.068548 76) (end 160.994536 94.925988) (width 0.25) (layer "F.Cu") (net 13))
+  (segment (start 124.5 76) (end 142.068548 76) (width 0.25) (layer "F.Cu") (net 13))
+  (segment (start 181.548533 96.499999) (end 193.102501 96.499999) (width 0.25) (layer "F.Cu") (net 13))
+  (segment (start 93 75) (end 102.5 75) (width 0.25) (layer "F.Cu") (net 13))
   (segment (start 179.974522 94.925988) (end 181.548533 96.499999) (width 0.25) (layer "F.Cu") (net 13))
-  (segment (start 118.820138 74.928436) (end 121.071564 74.928436) (width 0.25) (layer "F.Cu") (net 13))
-  (segment (start 124.5 76) (end 134.535474 76) (width 0.25) (layer "F.Cu") (net 13))
-  (segment (start 117.866692 73.97499) (end 118.820138 74.928436) (width 0.25) (layer "F.Cu") (net 13))
-  (segment (start 139.035474 80.5) (end 146.568548 80.5) (width 0.25) (layer "F.Cu") (net 13))
-  (segment (start 104.45001 73.97499) (end 117.866692 73.97499) (width 0.25) (layer "F.Cu") (net 13))
-  (segment (start 134.535474 76) (end 139.035474 80.5) (width 0.25) (layer "F.Cu") (net 13))
   (segment (start 193.102501 96.499999) (end 194.1025 95.5) (width 0.25) (layer "F.Cu") (net 13))
-  (segment (start 146.568548 80.5) (end 160.994536 94.925988) (width 0.25) (layer "F.Cu") (net 13))
-  (segment (start 93 75) (end 102.5 75) (width 0.25) (layer "F.Cu") (net 13))
-  (segment (start 181.548533 96.499999) (end 193.102501 96.499999) (width 0.25) (layer "F.Cu") (net 13))
-  (segment (start 160.994536 94.925988) (end 179.974522 94.925988) (width 0.25) (layer "F.Cu") (net 13))
+  (segment (start 122.5 78) (end 124.5 76) (width 0.25) (layer "F.Cu") (net 13))
   (segment (start 92.572 75.928) (end 93 75.5) (width 0.25) (layer "F.Cu") (net 13))
   (segment (start 121.071564 74.928436) (end 122.5 73.5) (width 0.25) (layer "F.Cu") (net 13))
   (segment (start 103.195 75.23) (end 104.45001 73.97499) (width 0.25) (layer "F.Cu") (net 13))
-  (segment (start 122.5 78) (end 124.5 76) (width 0.25) (layer "F.Cu") (net 13))
   (via (at 122.5 73.5) (size 0.8) (drill 0.4) (layers "F.Cu" "B.Cu") (net 13))
   (via (at 122.5 78) (size 0.8) (drill 0.4) (layers "F.Cu" "B.Cu") (net 13))
@@
   (segment (start 123.174511 77.325489) (end 122.5 78) (width 0.25) (layer "B.Cu") (net 13))
   (segment (start 109.615001 76.884999) (end 118.384999 76.884999) (width 0.25) (layer "F.Cu") (net 14))
-  (segment (start 181.825489 81.825489) (end 192.777011 81.825489) (width 0.25) (layer "F.Cu") (net 14))
-  (segment (start 122.5 77) (end 124.10048 75.39952) (width 0.25) (layer "F.Cu") (net 14))
-  (segment (start 192.777011 81.825489) (end 194.1025 80.5) (width 0.25) (layer "F.Cu") (net 14))
   (segment (start 103.195 77.77) (end 93.27 77.77) (width 0.25) (layer "F.Cu") (net 14))
   (segment (start 92.286 78.214) (end 93 77.5) (width 0.25) (layer "F.Cu") (net 14))
   (segment (start 108.73 77.77) (end 109.615001 76.884999) (width 0.25) (layer "F.Cu") (net 14))
+  (segment (start 85.643 78.214) (end 92.286 78.214) (width 0.25) (layer "F.Cu") (net 14))
+  (segment (start 124.10048 75.39952) (end 142.033062 75.39952) (width 0.25) (layer "F.Cu") (net 14))
+  (segment (start 122.5 77) (end 124.10048 75.39952) (width 0.25) (layer "F.Cu") (net 14))
+  (segment (start 119 77.5) (end 120 77.5) (width 0.25) (layer "F.Cu") (net 14))
+  (segment (start 120 77.5) (end 122.5 75) (width 0.25) (layer "F.Cu") (net 14))
+  (segment (start 142.033062 75.39952) (end 145.608062 78.97452) (width 0.25) (layer "F.Cu") (net 14))
+  (segment (start 192.777011 81.825489) (end 194.1025 80.5) (width 0.25) (layer "F.Cu") (net 14))
   (segment (start 178.97452 78.97452) (end 181.825489 81.825489) (width 0.25) (layer "F.Cu") (net 14))
-  (segment (start 85.643 78.214) (end 92.286 78.214) (width 0.25) (layer "F.Cu") (net 14))
-  (segment (start 124.10048 75.39952) (end 134.5 75.39952) (width 0.25) (layer "F.Cu") (net 14))
-  (segment (start 119 77.5) (end 120 77.5) (width 0.25) (layer "F.Cu") (net 14))
-  (segment (start 138.075 78.97452) (end 178.97452 78.97452) (width 0.25) (layer "F.Cu") (net 14))
-  (segment (start 120 77.5) (end 122.5 75) (width 0.25) (layer "F.Cu") (net 14))
-  (segment (start 134.5 75.39952) (end 138.075 78.97452) (width 0.25) (layer "F.Cu") (net 14))
+  (segment (start 181.825489 81.825489) (end 192.777011 81.825489) (width 0.25) (layer "F.Cu") (net 14))
   (segment (start 118.384999 76.884999) (end 119 77.5) (width 0.25) (layer "F.Cu") (net 14))
   (segment (start 103.195 77.77) (end 108.73 77.77) (width 0.25) (layer "F.Cu") (net 14))
+  (segment (start 145.608062 78.97452) (end 178.97452 78.97452) (width 0.25) (layer "F.Cu") (net 14))
   (via (at 122.5 75) (size 0.8) (drill 0.4) (layers "F.Cu" "B.Cu") (net 14))
   (via (at 122.5 77) (size 0.8) (drill 0.4) (layers "F.Cu" "B.Cu") (net 14))
