File: td-rgbinput/color_channel.kicad_sch (KiCad schematic)
At the start: 13 parts, among them Q1 2N7002NXBKR, Q2 2N7002NXBKR, U6 AD8337

Commit message: fix todos
Parts:
- removed C14: 0.1uF, Capacitor_SMD:C_0805_2012Metric, symbol Device:C
- added C? (x3): 0.1uF, Capacitor_SMD:C_0805_2012Metric, symbol Device:C
- added R? (x6): 1k, Resistor_SMD:R_0805_2012Metric, symbol Device:R
- added R?: 10, Resistor_SMD:R_0805_2012Metric, symbol Device:R
- added U? (x3): TLC272, symbol Amplifier_Operational:TLC272
- U6: footprint Package_CSP:LFCSP-8-1EP_3x3mm_P0.5mm_EP1.45x1.74mm -> td-deflect:LFCSP-8-1EP_3x3mm_P0.5mm_AD8337
Connections:
- net +5V: now also RV4.1, RV5.1, C?.1
- net -5V: now also RV4.3, C?.2
- net GND: now also C?.2, C?.2, R?.1, R?.2, U?.1, U?.2 (-); no longer RV4.3
- net bias_buffered: now also R?.2; no longer RV5.1
- net gain_buffered: now also R?.2; no longer RV4.1
- net input: now also R?.1; no longer C12.2
- net output: now also R?.1, R?.2; no longer RV5.2
- net at U6.7 (GAIN): now also C?.1, R?.1, R?.2; no longer RV4.2
- new net: C12.2, R?.1, R?.2
- new net: RV4.2, U?.3 (+)
- new net: RV5.2, U?.3 (+)
- new net: R?.2, U?.1, U?.2 (-)
- new net: C?.1, R?.1, R?.1
Other:
- note removed: "todo: bias impedance is not constant"
- moved on the sheet: RV4, RV5

Commit message: finish pcb
Parts:
- U12: renamed from U?; footprint (none) -> Package_SO:SOIC-8_3.9x4.9mm_P1.27mm
- gave numbers to parts that had none: 10
- renumbered C10 to C19, C12 to C20, C13 to C21, Q1 to Q5, Q2 to Q6, R9 to R24, R14 to R25, R16 to R26, R17 to R27, RV4 to RV8, RV5 to RV9, U6 to U8

Commit message: finish layout
Parts:
- U6: renamed from U8; Digikey AD8337BCPZ-WP -> 505-AD8337BCPZ-REELCT-ND
- renumbered C19 to C10, C20 to C12, C21 to C13, C23 to C32, C24 to C33, C25 to C34, Q5 to Q1, Q6 to Q2, R25 to R14, R26 to R16, R27 to R17, R33 to R47, R34 to R48, R35 to R49, R36 to R50, R37 to R51, R38 to R52, R39 to R53, R24 to R9, RV8 to RV4, RV9 to RV5, U12 to U14

Commit message: update td-rgbinput to reflect constructed circuit
Connections:
- net GND: no longer R50.1, U14.1, U14.2 (-)
- new net: R50.1, U14.1, U14.2 (-)
Changed lines of the file:
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@@
   (junction (at 128.27 43.18) (diameter 0) (color 0 0 0 0)
   )
-  (junction (at 115.57 33.02) (diameter 0) (color 0 0 0 0)
-  )
   (wire (pts (xy 148.59 67.31) (xy 156.21 67.31))
     (stroke (width 0) (type default) (color 0 0 0 0))
@@
   )
   (wire (pts (xy 130.81 82.55) (xy 123.19 82.55))
-    (stroke (width 0) (type default) (color 0 0 0 0))
-  )
-  (wire (pts (xy 115.57 33.02) (xy 124.46 33.02))
     (stroke (width 0) (type default) (color 0 0 0 0))
   )
@@
       (effects (font (size 1.27 1.27)) hide)
     )
-    (pin "1")
-    (pin "2")
-    (pin "3")
+    (pin "5")
+    (pin "6")
+    (pin "7")
   )
   (symbol (lib_id "power:GND") (at 160.02 128.27 0)
@@
       (effects (font (size 1.27 1.27)) hide)
     )
-    (pin "1")
-    (pin "2")
-    (pin "3")
+    (pin "4")
+    (pin "8")
   )
   (symbol (lib_id "power:-5V") (at 31.75 39.37 180)
@@
     (pin "3")
   )
-  (symbol (lib_id "power:GND") (at 124.46 33.02 0)
-    (in_bom yes) (on_board yes)
-    (property "Reference" "#PWR0140" (id 0) (at 124.46 39.37 0)
-      (effects (font (size 1.27 1.27)) hide)
-    )
-    (property "Value" "GND" (id 1) (at 124.587 37.4142 0))
-    (property "Footprint" "" (id 2) (at 124.46 33.02 0)
-      (effects (font (size 1.27 1.27)) hide)
-    )
-    (property "Datasheet" "" (id 3) (at 124.46 33.02 0)
-      (effects (font (size 1.27 1.27)) hide)
-    )
-    (pin "1")
-  )
   (symbol (lib_id "power:+5V") (at 31.75 24.13 0)
