File: td-rgbinput-lm1205/rgb.kicad_sch (KiCad schematic)
At the start: 48 parts, among them J1 Conn_01x10_Socket, J16 Conn_01x06_Male, J17 Conn_01x06_Male, J5 DB15_Female_HighDensity, U11 24LC08, U18 LM1205, U19 LMH1980, U26 MCP4728, U27 MCP4728, U29 MCP6001U

Commit message: update lm1205 to v1.0
Parts:
- added C1: 0.1uF, Capacitor_SMD:C_0805_2012Metric, symbol Device:C
- C47, C48, C49: Digikey (none) -> 490-10516-1-ND
- J1: Digikey (none) -> 455-B10B-XH-A-ND
- R1, R58, R59, R60, R61, R62, R63: Digikey (none) -> 311-1.00KCRCT-ND
- R111, R51, R52, R53: Digikey (none) -> 311-30.0CRCT-ND
- R2, R3, R4: Digikey (none) -> 311-220CRCT-ND
- R54, R55: Digikey (none) -> 311-100CRCT-ND
- R86, R87, R88: Digikey (none) -> 311-75.0CRCT-ND
- R89: Digikey 311-1.00CRCT-ND -> 311-1.00KCRCT-ND
- U26, U27: Digikey (none) -> MCP4728T-E/UNCT-ND
- U29: footprint Package_SO:SOIC-8_3.9x4.9mm_P1.27mm -> Package_TO_SOT_SMD:SOT-23-5; Digikey (none) -> MCP6001UT-I/OTCT-ND
Connections:
- net backporch is gone; now on net SEP_BP: R55.1
- net GND: now also C1.2
- net globalbias: now also C1.1
- net +3V3 renamed +3.3V
Other:
- moved on the sheet: C47, C48, C49, C56, R51, R52, R53, U26, U27
