File: td-rgbinput-lm1205/rgb.kicad_sch (KiCad schematic)
At the start: 49 parts, among them J1 Conn_01x10_Socket, J16 Conn_01x06_Male, J17 Conn_01x06_Male, J5 DB15_Female_HighDensity, U11 24LC08, U18 LM1205, U19 LMH1980, U26 MCP4728, U27 MCP4728, U29 MCP6001U

Commit message: Update td-rgbinput-lm1205 to add decoupling caps etc
Parts:
- added C10, C6, C7: 1uF, Capacitor_SMD:C_0805_2012Metric, symbol Device:C
- added C2, C3, C4, C5: 0.1uF, Capacitor_SMD:C_0805_2012Metric, symbol Device:C
- added U2: 74HCT14, Package_SO:SOIC-14_3.9x8.7mm_P1.27mm, symbol 74xx:74HC14
- C1, C50, C51, C52, C53, C54, C55, C56, C90: Digikey (none) -> 1276-1099-1-ND
- C91: value 0.1uF -> 1uF; Digikey 1276-1099-1-ND -> 1276-1066-1-ND
- J5: footprint td-io:DSUB-15-HD_Female_Horizontal_P2.29x2.5mm_EdgePinOffset8.35mm_Housed_MountingHolesOffset10.89mm -> Connector_Dsub:DSUB-15-HD_Socket_Horizontal_P2.29x2.54mm_EdgePinOffset8.35mm_Housed_MountingHolesOffset10.89mm; symbol Connector:DB15_Female_HighDensity -> Connector:DE15_Socket_HighDensity_MountingHoles
- U26, U27: now not fitted
Connections:
- net hsync_vga is gone; now on net vga_hsync: C57.2, R1.2
- net +12V: now also C10.1, C6.1, C7.1
- net +3.3VA: now also U2.14 (VCC)
- net GND: now also J5.0, C10.2, C2.2, C3.2, C4.2, C5.2, C6.2, C7.2, U2.11, U2.13, U2.5, U2.7 (GND), U2.9
- net bgain: now also C2.1
- net ggain: now also C4.1
- net globalgain: now also C3.1
- net rgain: now also C5.1
- net vga_hsync: now also U2.1
- new net: U2.2, U2.3
- new net PLAIN_HSYNC: U2.4
- no-connect marks 6 -> 10
Other:
- moved on the sheet: J1, R90, R91, R92
