File: td-rgbinput-lm1205/td-rgbinput-lm1205.kicad_pcb (KiCad board)
At the start: 2 copper layers, 120 x 50 mm, 58 parts, among them J1 Conn_01x10_Socket, J16 Conn_01x06_Male, J17 Conn_01x06_Male, J2 Conn_01x07_Male, J3 Conn_01x05_Pin, J4 Conn_01x06_Male, J5 DB15_Female_HighDensity, U1 AP2204K-3.3, U11 24LC08, U18 LM1205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

Commit message: update lm1205 to v1.0
Parts:
- added C1: 0.1uF, Capacitor_SMD:C_0805_2012Metric, F.Cu at (130.9, 79.5)
- J2: footprint Connector_JST:JST_XH_B7B-XH-AM_1x07_P2.50mm_Vertical -> Connector_JST:JST_XH_B7B-XH-A_1x07_P2.50mm_Vertical
- U29: footprint Package_SO:SOIC-8_3.9x4.9mm_P1.27mm -> Package_TO_SOT_SMD:SOT-23-5
- moved J16 81.2 mm to (93.0, 83.3)
- moved R2 68.9 mm to (100.7, 66.8), turned to 0 degrees
- moved R4 68.6 mm to (100.7, 82.0), turned to 0 degrees
- moved R3 68.1 mm to (100.7, 79.5)
- moved J4 65.0 mm to (158.0, 91.5)
- moved R59 40.4 mm to (135.0, 61.5), turned to 180 degrees
- moved J2 32.7 mm to (109.3, 53.8)
- moved J17 31.0 mm to (157.8, 71.5)
- moved U27 24.0 mm to (141.0, 65.0)
- moved U26 22.5 mm to (140.8, 75.0)
- moved C92 21.4 mm to (141.0, 70.0)
- moved H3 20.0 mm to (167.0, 56.0)
- moved H4 20.0 mm to (167.0, 96.0)
- moved J3 10.5 mm to (150.0, 85.0), turned to -90 degrees
- moved C56 10.1 mm to (130.9, 77.0)
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Connections:
- C58 pad 1: +3V3 -> +3.3V
- J16 pad 5: /rgb/vga_hsync -> vga_hsync
- J16 pad 6: /rgb/vga_vsync -> vga_vsync
- J17 pad 2: /rgb/r_yoke -> r_yoke
- J17 pad 3: /rgb/g_yoke -> g_yoke
- J17 pad 4: /rgb/b_yoke -> b_yoke
- J2 pad 3: /vga_vsync -> vga_vsync
- J4 pad 1: /vga_red -> r_yoke
- J4 pad 2: /vga_green -> g_yoke
- J4 pad 3: /vga_blue -> b_yoke
- J4 pad 5: /vga_hsync -> vga_hsync
- J4 pad 6: /vga_vsync -> vga_vsync
- J5 pad 13: /rgb/vga_hsync -> vga_hsync
- J5 pad 14: /rgb/vga_vsync -> vga_vsync
- R1 pad 1: +3V3 -> +3.3V
- R55 pad 1: /rgb/backporch -> SEP_BP
- R86 pad 1: /rgb/r_yoke -> r_yoke
- R87 pad 1: /rgb/g_yoke -> g_yoke
- R88 pad 1: /rgb/b_yoke -> b_yoke
- U19 pad 3: +3V3 -> +3.3V
Routing:
- net vga_hsync: track 0.00 -> 133.5 mm, vias 0 -> 1
- net +12V: track 0.00 -> 127.5 mm, vias 0 -> 2
- net vga_vsync: track 0.00 -> 127.1 mm
- net +3.3V: track 0.00 -> 102.5 mm, vias 0 -> 3
- net /rgb/globalgain: track 0.00 -> 69.9 mm, vias 0 -> 2
- net /rgb/bgain: track 0.00 -> 64.4 mm, vias 0 -> 2
- net LM1205_BLANK: track 0.00 -> 57.6 mm, vias 0 -> 2
- net /rgb/ggain: track 0.00 -> 55.8 mm, vias 0 -> 2
- net g_yoke: track 0.00 -> 54.3 mm, vias 0 -> 2
- net r_yoke: track 0.00 -> 53.8 mm, vias 0 -> 1
- net b_yoke: track 0.00 -> 52.3 mm
- net /rgb/rbias: track 0.00 -> 49.2 mm, vias 0 -> 1
- net GAIN_LOAD: track 0.00 -> 44.0 mm, vias 0 -> 2
- net /rgb/gbias: track 0.00 -> 43.7 mm, vias 0 -> 3
- net /rgb/bbias: track 0.00 -> 43.6 mm, vias 0 -> 3
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Other:
- board size 120 x 50 mm -> 100 x 50 mm
- board text added: "bias"
- board text added: "digital"
- board text added: "gain"
- board text added: "locked"
- board text added: "ms8 in"
- board text added: "remote"
- board text added: "scl"
- board text added: "sda"
- board text added: "sync"
