File: td-rgbinput-lm1205/td-rgbinput-lm1205.kicad_sch (KiCad schematic)
At the start: 16 parts, among them J2 Conn_01x07_Male, J3 Conn_01x05_Pin, J4 Conn_01x06_Male, U1 AP2205-33W5-7, U3 AZ1117-ADJ

Commit message: small notes
Other:
- note added: "fix 10k resistor part numbers"
